File: frank_pro_m2/gamepad.kicad_sch (KiCad schematic)
At the start: 3 parts, among them J14 GP2

Commit message: Board updates
Parts:
- D3: footprint FRANK:D_SOD-323 -> FRANK:D_miniMELF
Changed lines of the file:
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@@
 			)
 		)
-		(property "Footprint" "FRANK:D_SOD-323"
+		(property "Footprint" "FRANK:D_miniMELF"
 			(at 147.32 109.22 0)
 			(hide yes)

Commit message: FRANK Pro 1.01 HW Release
Parts:
- D3: footprint FRANK:D_miniMELF -> FRANK:D_MiniMELF; symbol Device:D_Zener -> FRANK:D_Zener
Changed lines of the file:
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@@
 	)
 	(symbol
-		(lib_id "power:GND")
+		(lib_id "FRANK:GND")
 		(at 147.32 113.03 0)
 		(unit 1)
@@
 	)
 	(symbol
-		(lib_id "Device:D_Zener")
+		(lib_id "FRANK:D_Zener")
 		(at 147.32 109.22 270)
 		(unit 1)
@@
 			)
 		)
-		(property "Footprint" "FRANK:D_miniMELF"
+		(property "Footprint" "FRANK:D_MiniMELF"
 			(at 147.32 109.22 0)
 			(hide yes)
@@
 	)
 	(symbol
-		(lib_id "power:VBUS")
+		(lib_id "FRANK:VBUS")
 		(at 160.02 106.68 180)
 		(unit 1)
@@
 	)
 	(symbol
-		(lib_id "power:GND")
+		(lib_id "FRANK:GND")
 		(at 161.29 96.52 270)
 		(unit 1)
