File: frank_pro_m2/sd.kicad_sch (KiCad schematic)
At the start: 2 parts, among them J16 104031-0811

Commit message: FRANK Pro 1.01 HW Release
Parts:
- J16: symbol Connector:Micro_SD_Card -> FRANK:Micro_SD_Card
Changed lines of the file:
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@@
 	)
 	(symbol
-		(lib_id "power:+3V3")
+		(lib_id "FRANK:+3V3")
 		(at 162.56 120.65 180)
 		(unit 1)
@@
 	)
 	(symbol
-		(lib_id "power:GND")
+		(lib_id "FRANK:GND")
 		(at 148.59 115.57 270)
 		(unit 1)
@@
 	)
 	(symbol
-		(lib_id "power:GND")
+		(lib_id "FRANK:GND")
 		(at 175.26 120.65 270)
 		(unit 1)
@@
 	)
 	(symbol
-		(lib_id "Connector:Micro_SD_Card")
+		(lib_id "FRANK:Micro_SD_Card")
 		(at 198.12 115.57 0)
 		(unit 1)
