File: frank_pro_m2/frank_pro_m2.kicad_sch (KiCad schematic)
At the start: 18 parts, among them J1 UART, J2 DEBUG, J3 PWR

Commit message: Board updates
Parts:
- removed S2: RP Reset, FRANK:Button_SMD_TS1234VW, symbol FRANK:SW_Push_1234VW
- removed S3: RP BOOT, FRANK:Button_SMD_TS1234VW, symbol FRANK:SW_Push_1234VW
- removed S4: RP Reset, FRANK:Button_SMD_3x4x2mm, symbol KMR221G_LFS:KMR221G_LFS
- removed S5: RP BOOT, FRANK:Button_SMD_3x4x2mm, symbol KMR221G_LFS:KMR221G_LFS
- removed S6: ESP Reset, FRANK:Button_SMD_TS1234VW, symbol FRANK:SW_Push_1234VW
Connections:
- net GND: now also J1.MP
- net MONO_L renamed Audio/MONO_L
- net MONO_R renamed Audio/MONO_R
- net SHND renamed Audio/SHND
Other:
- added sheet Boot Select (bootsel.kicad_sch)
- added sheet ESP Reset (esp_reset.kicad_sch)
- added sheet RP Reset (reset.kicad_sch)
- moved on the sheet: H1, H2, H3, H4, J2, J3, JP1, R1, R2, R3, R4, S1

Commit message: FRANK Pro 1.01 HW Release
Parts:
- H1, H2, H3, H4: symbol Mechanical:MountingHole -> FRANK:MountingHole
- J1: symbol Connector:Conn_01x04_Pin -> FRANK:Conn_01x04_Pin
- J2, J3: symbol Connector:Conn_01x03_Pin -> FRANK:Conn_01x03_Pin
- JP1: symbol DS05-127-2-04BK-SMT-TR:DS05-127-2-04BK-SMT-TR -> FRANK:DS05-127-2-04BK-SMT-TR
- S1: symbol MSK12C02:MSK12C02 -> FRANK:MSK12C02
Changed lines of the file:
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@@
 	)
 	(symbol
-		(lib_id "power:GND")
+		(lib_id "FRANK:GND")
 		(at 105.41 45.72 270)
 		(mirror x)
@@
 	)
 	(symbol
-		(lib_id "power:GND")
+		(lib_id "FRANK:GND")
 		(at 134.62 165.1 90)
 		(unit 1)
@@
 	)
 	(symbol
-		(lib_id "power:GND")
+		(lib_id "FRANK:GND")
 		(at 114.3 50.8 0)
 		(mirror x)
@@
 	)
 	(symbol
-		(lib_id "MSK12C02:MSK12C02")
+		(lib_id "FRANK:MSK12C02")
 		(at 148.59 95.25 0)
 		(mirror y)
@@
 	)
 	(symbol
-		(lib_id "DS05-127-2-04BK-SMT-TR:DS05-127-2-04BK-SMT-TR")
+		(lib_id "FRANK:DS05-127-2-04BK-SMT-TR")
 		(at 97.79 138.43 0)
 		(unit 1)
@@
 	)
 	(symbol
-		(lib_id "power:GND")
+		(lib_id "FRANK:GND")
 		(at 138.43 100.33 270)
 		(mirror x)
@@
 	)
 	(symbol
-		(lib_id "power:GND")
+		(lib_id "FRANK:GND")
 		(at 129.54 143.51 90)
 		(unit 1)
@@
 	)
 	(symbol
-		(lib_id "Connector:Conn_01x03_Pin")
+		(lib_id "FRANK:Conn_01x03_Pin")
 		(at 120.65 184.15 0)
 		(unit 1)
@@
 	)
 	(symbol
-		(lib_id "power:VBUS")
+		(lib_id "FRANK:VBUS")
 		(at 129.54 138.43 270)
 		(unit 1)
@@
 	)
 	(symbol
-		(lib_id "Connector:Conn_01x03_Pin")
+		(lib_id "FRANK:Conn_01x03_Pin")
 		(at 129.54 165.1 0)
 		(unit 1)
@@
 	)
 	(symbol
-		(lib_id "power:VBUS")
+		(lib_id "FRANK:VBUS")
 		(at 134.62 167.64 270)
 		(unit 1)
@@
 	)
 	(symbol
-		(lib_id "power:+3V3")
+		(lib_id "FRANK:+3V3")
 		(at 105.41 48.26 90)
 		(mirror x)
@@
 	)
 	(symbol
-		(lib_id "power:VBUS")
+		(lib_id "FRANK:VBUS")
 		(at 66.04 180.34 270)
 		(unit 1)
@@
 	)
 	(symbol
-		(lib_id "Connector:Conn_01x04_Pin")
+		(lib_id "FRANK:Conn_01x04_Pin")
 		(at 110.49 48.26 0)
 		(mirror y)
@@
 	)
 	(symbol
-		(lib_id "Mechanical:MountingHole")
+		(lib_id "FRANK:MountingHole")
 		(at 267.97 156.21 0)
 		(unit 1)
@@
 	)
 	(symbol
-		(lib_id "Mechanical:MountingHole")
+		(lib_id "FRANK:MountingHole")
 		(at 267.97 151.13 0)
 		(unit 1)
@@
 	)
 	(symbol
-		(lib_id "power:GND")
+		(lib_id "FRANK:GND")
 		(at 125.73 184.15 90)
 		(unit 1)
@@
 	)
 	(symbol
-		(lib_id "Mechanical:MountingHole")
+		(lib_id "FRANK:MountingHole")
 		(at 267.97 161.29 0)
 		(unit 1)
@@
 	)
 	(symbol
-		(lib_id "power:+3V3")
+		(lib_id "FRANK:+3V3")
 		(at 83.82 48.26 270)
 		(mirror x)
@@
 	)
 	(symbol
-		(lib_id "power:+3V3")
+		(lib_id "FRANK:+3V3")
 		(at 83.82 45.72 270)
 		(mirror x)
@@
 	)
 	(symbol
-		(lib_id "Mechanical:MountingHole")
+		(lib_id "FRANK:MountingHole")
 		(at 267.97 146.05 0)
 		(unit 1)
@@
 	)
 	(symbol
-		(lib_id "power:+3V3")
+		(lib_id "FRANK:+3V3")
 		(at 134.62 162.56 270)
 		(unit 1)
@@
 	)
 	(symbol
-		(lib_id "power:+3V3")
+		(lib_id "FRANK:+3V3")
 		(at 129.54 140.97 270)
 		(unit 1)
@@
 	)
 	(symbol
-		(lib_id "power:VBUS")
+		(lib_id "FRANK:VBUS")
 		(at 138.43 92.71 90)
 		(mirror x)

Commit message: Board updates
Parts:
- removed J1: UART, FRANK:JST_SH_1x04_P1.00mm_Vertical, symbol FRANK:Conn_01x04_Pin
- added J1: UART, FRANK:JST_SH_1x03_P1.00mm_Vertical, symbol FRANK:Conn_01x03_Pin
Connections:
- net GND: now also J1.2 (Pin_2)
- net PGPIO0: now also J1.1 (Pin_1)
- net PGPIO1: now also J1.3 (Pin_3)
- net PSWCLK: now also J2.3 (Pin_3); no longer J2.1 (Pin_1)
- net PSWDIO: now also J2.1 (Pin_1); no longer J2.3 (Pin_3)
