File: nyx2b/nyx.kicad_sch (KiCad schematic)
At the start: 3 parts

Commit message: Nyx WIP
Connections:
- net VS: no longer names the net of J1.39
Other:
- sheet RP2350B ports: added none; removed GPIO25
- moved on the sheet: J1, J2, J3
