File: frank_m2/amp.kicad_sch (KiCad schematic)
At the start: 30 parts, among them U10 LM358, U9 PAM8403D

Commit message: Board updates
Parts:
- C36: value 47u -> 100u; footprint FRANK:C_0805_2012Metric -> FRANK:C_Radial_D6.3mm_P2.50mm; symbol FRANK:C_Small -> FRANK:C_Polarized_Small
Changed lines of the file:
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@@
 	)
 	(symbol
-		(lib_id "FRANK:C_Small")
+		(lib_id "FRANK:C_Polarized_Small")
 		(at 198.12 73.66 90)
 		(unit 1)
@@
 			)
 		)
-		(property "Value" "47u"
+		(property "Value" "100u"
 			(at 198.374 76.454 90)
 			(show_name no)
@@
 			)
 		)
-		(property "Footprint" "FRANK:C_0805_2012Metric"
+		(property "Footprint" "FRANK:C_Radial_D6.3mm_P2.50mm"
 			(at 198.12 73.66 0)
 			(hide yes)
@@
 			)
 		)
-		(property "Description" "Unpolarized capacitor, small symbol"
+		(property "Description" "Polarized capacitor, small symbol"
 			(at 198.12 73.66 0)
 			(hide yes)
