File: frank_m2/esp01s.kicad_sch (KiCad schematic)
At the start: 1 part, among them U1 ESP-01v090

Commit message: Board updates
Connections:
- net CH_PD: no longer names the net of U1.3 (CH_PD)
- net GPIO0: no longer names the net of U1.6 (GPIO0)
- net GPIO2: no longer names the net of U1.4 (GPIO2)
- no-connect marks 0 -> 3
Changed lines of the file:
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@@
 		(comment 1 "https://github.com/rh1tech/frank")
 	)
-	(hierarchical_label "GPIO0"
-		(shape input)
-		(at 175.26 101.6 0)
-		(effects
-			(font
-				(size 1.27 1.27)
-			)
-			(justify left)
-		)
+	(no_connect
+		(at 175.26 101.6)
+	)
+	(no_connect
+		(at 175.26 99.06)
+	)
+	(no_connect
+		(at 127 99.06)
 	)
 	(hierarchical_label "RX"
@@
 		)
 	)
-	(hierarchical_label "CH_PD"
-		(shape input)
-		(at 127 99.06 180)
-		(effects
-			(font
-				(size 1.27 1.27)
-			)
-			(justify right)
-		)
-	)
-	(hierarchical_label "GPIO2"
-		(shape input)
-		(at 175.26 99.06 0)
-		(effects
-			(font
-				(size 1.27 1.27)
-			)
-			(justify left)
-		)
-	)
