File: frank_m2/power.kicad_sch (KiCad schematic)
At the start: 28 parts, among them J4 USB4215-03-A, J5 DC-005-5A-2.0, U2 MP1584EN-LF-Z, U3 AMS1117 3.3

Commit message: Board updates
Parts:
- added J2: PWR, FRANK:PinHeader_1x03_P2.54mm, symbol FRANK:Conn_01x03_Pin
- D1: footprint FRANK:D_SMA_SS34 -> FRANK:D_SMA
Connections:
- net +3V3: now also J2.1 (Pin_1)
- net GND: now also J2.2 (Pin_2)
- net VBUS: now also J2.3 (Pin_3)
- net EN: no longer names the net of R7.1, R8.1, U2.2 (EN)
