File: tinyfrank_m2p2/tinyfrank_m2p2.kicad_sch (KiCad schematic)
At the start: 8 parts, among them J1 UART, J2 DEBUG, J3 PWR

Commit message: Board updates
Parts:
- removed J1: UART, TinyFRANK:JST_SH_1x04_P1.00mm_Vertical, symbol TinyFRANK:Conn_01x04_Pin
- added J9: DEBUG, TinyFRANK:JST_SH_1x03_P1.00mm_Vertical, symbol TinyFRANK:Conn_01x03_Pin
Connections:
- net GND: now also J9.2 (Pin_2); no longer J2.MP (Shield)
- net RP2350A/GPIO0: now also J9.1 (Pin_1)
- net RP2350A/GPIO1: now also J9.3 (Pin_3)
- net RP2350A/SWCLK: now also J2.3 (Pin_3); no longer J2.1 (Pin_1)
- net RP2350A/SWD: now also J2.1 (Pin_1); no longer J2.3 (Pin_3)
