File: minifrank_m2p2/minifrank_m2p2.kicad_pcb (KiCad board)
At the start: 4 copper layers, 85.6 x 54 mm, 136 parts, among them J1 PWR, J10 VGA, J11 PJ-320D, J12 104031-0811, J2 UART, J3 DEBUG, J4 SS-52100-004, J5 USB4215-03-A, J6 MDC-036, J7 PJ-320D, J8 DC3RX19JA2, J9 GP2, U1 TS3USB221RSER, U10 ESP-01v090, U11 TDA1387T, U12 LM358, U2 USBLC6-2SC6, U3 MW7211A, U4 NCP1117-3.3_SOT223, U5 TXS0104ERGYR, U6 ESP-PSRAM32, U7 W25Q128JVS, U8 CD4069UBM, U9 RP2350, Y1 ASE-12MHz

Commit message: Board updates
Parts:
- J2: footprint FRANK:JST_SH_BM04B-SRSS-TB_1x04-1MP_P1.00mm_Vertical -> FRANK:JST_SH_BM03B-SRSS-TB_1x03-1MP_P1.00mm_Vertical
- moved J2 0.60 mm to (172.5, 100.7)
- moved S1 0.14 mm to (172.9, 96.1)
Connections:
- net /ESP_CH_PD renamed /ESP01/CH_PD
- net /ESP_GPIO0 renamed /ESP01/GPIO0
- net /ESP_GPIO2 renamed /ESP01/GPIO2
- net /GPIO23 renamed /RP2350A/GPIO23
- net /GPIO24 renamed /RP2350A/GPIO24
- net /GPIO27 renamed /RP2350A/GPIO27
- net /GPIO28 renamed /RP2350A/GPIO28
- net /GPIO29 renamed /RP2350A/GPIO29
- net /GPIO8 renamed /RP2350A/GPIO8
- J12 pad 9: unconnected-(J12-SHIELD-Pad9) -> (no net)
- J2 pad 1: GND -> /GPIO0
- J2 pad 2: +3V3 -> GND
- J2 pad 3: /GPIO0 -> /GPIO1
- J3 pad 1: /SWCLK -> /RP2350A/SWD
- J3 pad 3: /SWD -> /RP2350A/SWCLK
- J4 pad 9: GND -> (no net)
- U9 pad 24: /SWCLK -> /RP2350A/SWCLK
- U9 pad 25: /SWD -> /RP2350A/SWD
Routing:
- net /SWD: track 25.9 -> 0.00 mm, vias 2 -> 0
- net /RP2350A/SWCLK: track 0.00 -> 22.4 mm, vias 0 -> 2
- net /RP2350A/SWD: track 0.00 -> 21.7 mm, vias 0 -> 2
- net /SWCLK: track 20.1 -> 0.00 mm, vias 2 -> 0
- net +3V3: track 79.9 -> 78.6 mm, vias 28 -> 27
- net /ESP_RST: track 22.0 -> 22.6 mm
- net GND: vias 17 -> 18
