File: minifrank_m2p2/minifrank_m2p2.kicad_sch (KiCad schematic)
At the start: 15 parts, among them J1 PWR, J2 UART, J3 DEBUG

Commit message: Board updates
Parts:
- removed S1: ESP Reset, FRANK:KMR_2, symbol KMR221G_LFS:KMR221G_LFS
- removed S2: RP Reset, FRANK:KMR_2, symbol KMR221G_LFS:KMR221G_LFS
- removed S3: RP Reset, FRANK:TS-1234VW, symbol FRANK:SW_Push_1234VW
- J2: footprint FRANK:JST_SH_BM04B-SRSS-TB_1x04-1MP_P1.00mm_Vertical -> FRANK:JST_SH_BM03B-SRSS-TB_1x03-1MP_P1.00mm_Vertical; symbol Connector:Conn_01x04_Pin -> Connector:Conn_01x03_Pin
Connections:
- net +3V3: no longer J2.2 (Pin_2)
- net GND: now also J2.2 (Pin_2); no longer J2.1 (Pin_1)
- net GPIO0: now also J2.1 (Pin_1); no longer J2.3 (Pin_3)
- net GPIO1: now also J2.3 (Pin_3); no longer J2.4 (Pin_4)
- net SWCLK renamed RP2350A/SWD
- net SWD renamed RP2350A/SWCLK
- no-connect marks 11 -> 13
Other:
- added sheet ESP Reset (reset_esp.kicad_sch)
- added sheet RP Reset (reset_rp.kicad_sch)
- moved on the sheet: J1, J3, R1, R2, R3, R4, S4
