File: xt8086/pc_speaker.kicad_sch (KiCad schematic)
At the start: 7 parts, among them J5 SJ1-3525N, Q1 2N7000, U3 CMT-7525-80-SMT-TR

Commit message: Board updates
Parts:
- added JP6: Dir, Jumper:SolderJumper-2_P1.3mm_Open_Pad1.0x1.5mm, symbol xt8086:Conn_01x02_Pin
- added R27: 22R, xt8086:R_0805_2012Metric, symbol xt8086:R
- J: renamed from U3; value CMT-7525-80-SMT-TR -> GENERIC BUZZER
- Q1: value 2N7000 -> BC847
- R4: value 20K -> 1K
Connections:
- net GND: no longer R4.2
- net SPEAKER: now also JP6.2 (Pin_2)
- net SPK_IN: no longer Q1.2 (B)
- net at D1.2 (A), J.2 (-): now also JP6.1 (Pin_1), R27.1; no longer Q1.1 (C)
- new net: Q1.1 (C), R27.2
- new net: Q1.2 (B), R4.2
- no-connect marks 4 -> 2
Other:
- moved on the sheet: D1, J5, JP1, JP2

Commit message: xt8086 WIP
Parts:
- removed JP1: Jck, xt8086:PinHeader_1x02_P2.54mm, symbol xt8086:Conn_01x02_Pin
- removed JP2: Spk, xt8086:PinHeader_1x02_P2.54mm, symbol xt8086:Conn_01x02_Pin
- added SW1: SW_DIP_x02, Button_Switch_THT:SW_DIP_SPSTx02_Slide_9.78x7.26mm_W7.62mm_P2.54mm, symbol Switch:SW_DIP_x02
- J4: renamed from J; footprint xt8086:Buzzer_SMD_7.5x7.5mm -> xt8086:Buzzer_12x8.5RM6.5
- renumbered J5 to J6, JP6 to JP1, R4 to R5, R27 to R6
Connections:
- net JACK_IN: now also SW1.2
- net SPEAKER: now also SW1.3, SW1.4
- net SPK_IN: now also SW1.1
Other:
- moved on the sheet: D1, J4, J6, JP1, Q1, R5, R6

Commit message: xt8086 WIP
Parts:
- JP1: footprint Jumper:SolderJumper-2_P1.3mm_Open_Pad1.0x1.5mm -> xt8086:SolderJumper-2_P1.3mm_Open_Pad1.0x1.5mm
- SW1: footprint Button_Switch_THT:SW_DIP_SPSTx02_Slide_9.78x7.26mm_W7.62mm_P2.54mm -> xt8086:SW_DIP_SPSTx02_Slide_9.78x7.26mm_W7.62mm_P2.54mm
Changed lines of the file:
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@@
 			)
 		)
-		(property "Footprint" "Jumper:SolderJumper-2_P1.3mm_Open_Pad1.0x1.5mm"
+		(property "Footprint" "xt8086:SolderJumper-2_P1.3mm_Open_Pad1.0x1.5mm"
 			(at 133.35 115.57 0)
 			(hide yes)
@@
 			)
 		)
-		(property "Footprint" "Button_Switch_THT:SW_DIP_SPSTx02_Slide_9.78x7.26mm_W7.62mm_P2.54mm"
+		(property "Footprint" "xt8086:SW_DIP_SPSTx02_Slide_9.78x7.26mm_W7.62mm_P2.54mm"
 			(at 185.42 114.3 0)
 			(hide yes)

Commit message: xt8086 1.03
Parts:
- added R6: 300R, xt8086:R_0805_2012Metric, symbol xt8086:R
- J6: renamed from J4; value GENERIC BUZZER -> Buzzer
- JP1: value Dir -> Direct
- renumbered J6 to J8, R6 to R7, SW1 to S4
Connections:
- net VBUS: now also R6.1
- net at D1.2 (A), J6.2 (-), JP1.1 (Pin_1)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: now also R6.2
