File: xt8086/xt8086.kicad_sch (KiCad schematic)
At the start: 19 parts, among them J1 UART, J2 Ext Connector, J3 DEBUG, U1 SN74LS04, U2 SN74LS74

Commit message: xt8086 WIP
Parts:
- removed J1: UART, xt8086:JST_SH_1x04_P1.00mm_Vertical, symbol xt8086:Conn_01x04_Pin
- added J1: UART, xt8086:JST_SH_1x03_P1.00mm_Vertical, symbol xt8086:Conn_01x03_Pin
- added S1: SS12D00, xt8086:Switch_Slide_SS12D00, symbol xt8086:SS12D00
- renumbered J3 to J2, J2 to J3, S1 to S2, S2 to S3
Connections:
- net GND: now also J1.2 (Pin_2); no longer J2.MP
- net SWCLK: now also J2.3 (Pin_3); no longer J2.1 (Pin_1)
- net SWDIO: now also J2.1 (Pin_1); no longer J2.3 (Pin_3)
- net UART0_RX: now also J1.3 (Pin_3)
- net UART0_TX: now also J1.1 (Pin_1)
- net VBUS: now also S1.2
- new net USB/SW: S1.1
- no-connect marks 25 -> 26
Other:
- sheet USB ports: added SW; removed none
- moved on the sheet: J3, S2, S3

Commit message: xt8086 WIP
Parts:
- removed J3: Ext Connector, xt8086:PinHeader_2x20_P2.54mm_Vertical, symbol xt8086:Conn_02x20_Odd_Even
- added J12: 8086_Pins_Right, xt8086:PinSocket_1x20_P2.54mm_Vertical, symbol xt8086:Conn_01x20_Pin
- added J3: 8086_Pins_Left, xt8086:PinSocket_1x20_P2.54mm_Vertical, symbol xt8086:Conn_01x20_Pin
Connections:
- net A16/GP16: now also J3.18 (Pin_18)
- net A17/GP17: now also J3.17 (Pin_17)
- net A18/GP18: now also J3.16 (Pin_16)
- net A19/GP19: now also J3.15 (Pin_15)
- net AD0/GP0: now also J12.5 (Pin_5)
- net AD10/GP10: now also J12.15 (Pin_15)
- net AD11/GP11: now also J12.16 (Pin_16)
- net AD12/GP12: now also J12.17 (Pin_17)
- net AD13/GP13: now also J12.18 (Pin_18)
- net AD14/GP14: now also J12.19 (Pin_19)
- net AD15/GP15: now also J3.19 (Pin_19)
- net AD1/GP1: now also J12.6 (Pin_6)
- net AD2/GP2: now also J12.7 (Pin_7)
- net AD3/GP3: now also J12.8 (Pin_8)
- net AD4/GP4: now also J12.9 (Pin_9)
- net AD5/GP5: now also J12.10 (Pin_10)
- net AD6/GP6: now also J12.11 (Pin_11)
- net AD7/GP7: now also J12.12 (Pin_12)
- net AD8/GP8: now also J12.13 (Pin_13)
- net AD9/GP9: now also J12.14 (Pin_14)
- net ALE/GP20: now also J3.5 (Pin_5)
- net BHE/GP25: now also J3.14 (Pin_14)
- net CLK/GP29: now also J12.2 (Pin_2)
- net GND: now also J12.1 (Pin_1), J12.20 (Pin_20), J12.4 (Pin_4), J3.11 (Pin_11)
- net INTA/GP23: now also J3.4 (Pin_4)
- net INTR/GP26: now also J12.3 (Pin_3)
- net MIO/GP24: now also J3.8 (Pin_8)
- net RD/GP21: now also J3.12 (Pin_12)
- net READY: now also J3.2 (Pin_2)
- net RESET/GP28: now also J3.1 (Pin_1)
- net VBUS: now also J3.20 (Pin_20)
- net WR/GP22: now also J3.9 (Pin_9)
- net 8086/MN/MX renamed MN/MX
- net MN/MX: now also J3.13 (Pin_13)
- net 8086/TEST renamed TEST
- net TEST: now also J3.3 (Pin_3)
- new net DEN: J3.6 (Pin_6)
- new net DT/R: J3.7 (Pin_7)
- new net HLDA: J3.10 (Pin_10)
- no-connect marks 26 -> 23
Other:
- moved on the sheet: R1, R2

Commit message: xt8086 1.03
Parts:
- added J1: PWR, xt8086:PinHeader_1x03_P2.54mm_Vertical, symbol xt8086:Conn_01x03_Pin
- J5: renamed from J2; value DEBUG -> Debug
- S2: value BOOT -> Boot
- S3: value RESET -> Reset
- renumbered J1 to J2, J12 to J4, R2 to R1, R1 to R2
Connections:
- net +3V3: now also J1.3 (Pin_3)
- net GND: now also J1.2 (Pin_2)
- net VBUS: now also J1.1 (Pin_1)
Other:
- moved on the sheet: C1, C2, C3, C4, J2, J3, J4, J5, LD1, R1, R2, R3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
