File: frank_mega/frank_mega.kicad_pcb (KiCad board)
At the start: 2 copper layers, 149.9 x 99.5 mm, 236 parts, among them J1 PWR, J10 SJ1-3525N, J11 PAM L, J12 PAM R, J13 SJ1-3525N, J14 GP2, J15 GP2, J16 104031-0811, J17 SS-52100-004, J18 VGA, J19 Conn_02x20_Odd_Even, J2 UART, J3 DEBUG, J4 DC-005-5A-2.0, J5 USB4215-03-A, J6 MDC-036, J7 DC3RX19JA2, J8 RCA-103, J9 Pin Header 1x08, Q1 BC850, U1 MP1584EN-LF-Z, U10 MW7211A, U11 Pimoroni PGA2350, U12 74HC4052D, U13 ESP-01v090, U14 CD4069UBM, U15 TDA1387T, U16 PAM8403D, U17 LM358, U18 74HC4052D, U2 USBLC6-2SC6, U3 AMS1117 3.3, U4 TXS0104EDR, U5 JFC95101, U6 74HC74, U7 JFC95101, U8 74HC595, U9 74HC595, X1 3.58 MHz

Commit message: FRANK_MEGA WIP
Parts:
- moved J19 48.2 mm to (134.8, 104.5), turned to 90 degrees
Routing:
- net +3V3: track 347.7 -> 338.5 mm

Commit message: FRANK MEGA WIP
Parts:
- removed S1: MSK12C02, FRANK:Switch_Slide_MSK12C02
- added S9: SK12D07VG3NS, FRANK:Switch_Slide_SK12D07VG3NS, F.Cu at (222.7, 61.3)
- moved S6 56.5 mm to (223.2, 113.0)
- moved S7 0.09 mm to (223.2, 124.1)
Routing:
- net /PGPIO10: track 0.00 -> 181.8 mm, vias 0 -> 5
- net /PGPIO9: track 0.00 -> 175.0 mm, vias 0 -> 3
- net /PGPIO11: track 0.00 -> 149.5 mm, vias 0 -> 3
- net /PGPIO0: track 0.00 -> 133.1 mm, vias 0 -> 5
- net /PGPIO20: track 0.00 -> 121.8 mm, vias 0 -> 2
- net /Audio/TS/R_IN: track 0.00 -> 119.7 mm, vias 0 -> 3
- net /PGPIO21: track 0.00 -> 111.2 mm
- net /PGPIO1: track 0.00 -> 99.6 mm, vias 0 -> 3
- net /PGPIO27: track 0.00 -> 97.4 mm, vias 0 -> 3
- net /MONO_R: track 0.00 -> 94.0 mm, vias 0 -> 2
- net /PGPIO2: track 0.00 -> 90.8 mm, vias 0 -> 2
- net /PGPIO3: track 0.00 -> 88.3 mm, vias 0 -> 3
- net /Audio/TS/YM_CS2: track 0.00 -> 80.2 mm, vias 0 -> 2
- net /Audio Multiplexer/SW_TDA: track 0.00 -> 79.2 mm, vias 0 -> 1
- net /MONO_L: track 0.00 -> 78.6 mm, vias 0 -> 1
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