File: frank_mega/display.kicad_sch (KiCad schematic)
At the start: 1 part, among them J9 Pin Header 1x08

Commit message: New boards WIP
Parts:
- renumbered J9 to J10
Changed lines of the file:
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@@
 		(dnp no)
 		(fields_autoplaced yes)
-		(property "Reference" "#PWR0117"
+		(property "Reference" "#PWR0121"
 			(at 166.37 95.25 0)
 			(hide yes)
@@
 			(project "frank_mega"
 				(path "/8c0b3d8b-46d3-4173-ab1e-a61765f77d61/3504beb8-2939-46b0-9c32-2648908a1056"
-					(reference "#PWR0117")
+					(reference "#PWR0121")
 					(unit 1)
 				)
@@
 		(dnp no)
 		(fields_autoplaced yes)
-		(property "Reference" "#PWR0116"
+		(property "Reference" "#PWR0120"
 			(at 156.21 92.71 0)
 			(hide yes)
@@
 			(project "frank_mega"
 				(path "/8c0b3d8b-46d3-4173-ab1e-a61765f77d61/3504beb8-2939-46b0-9c32-2648908a1056"
-					(reference "#PWR0116")
+					(reference "#PWR0120")
 					(unit 1)
 				)
@@
 		(dnp no)
 		(fields_autoplaced yes)
-		(property "Reference" "J9"
+		(property "Reference" "J10"
 			(at 135.255 87.63 0)
 			(show_name no)
@@
 			(project "frank_mega"
 				(path "/8c0b3d8b-46d3-4173-ab1e-a61765f77d61/3504beb8-2939-46b0-9c32-2648908a1056"
-					(reference "J9")
+					(reference "J10")
 					(unit 1)
 				)

Commit message: FRANK MEGA WIP
Parts:
- renumbered J10 to J11
Changed lines of the file:
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@@
 		(dnp no)
 		(fields_autoplaced yes)
-		(property "Reference" "#PWR0133"
+		(property "Reference" "#PWR0136"
 			(at 166.37 95.25 0)
 			(hide yes)
@@
 			(project "frank_mega"
 				(path "/8c0b3d8b-46d3-4173-ab1e-a61765f77d61/3504beb8-2939-46b0-9c32-2648908a1056"
-					(reference "#PWR0133")
+					(reference "#PWR0136")
 					(unit 1)
 				)
@@
 		(dnp no)
 		(fields_autoplaced yes)
-		(property "Reference" "#PWR0132"
+		(property "Reference" "#PWR0135"
 			(at 156.21 92.71 0)
 			(hide yes)
@@
 			(project "frank_mega"
 				(path "/8c0b3d8b-46d3-4173-ab1e-a61765f77d61/3504beb8-2939-46b0-9c32-2648908a1056"
-					(reference "#PWR0132")
+					(reference "#PWR0135")
 					(unit 1)
 				)
@@
 		(dnp no)
 		(fields_autoplaced yes)
-		(property "Reference" "J10"
+		(property "Reference" "J11"
 			(at 135.255 87.63 0)
 			(show_name no)
@@
 			(project "frank_mega"
 				(path "/8c0b3d8b-46d3-4173-ab1e-a61765f77d61/3504beb8-2939-46b0-9c32-2648908a1056"
-					(reference "J10")
+					(reference "J11")
 					(unit 1)
 				)
