File: frank_mega/hdmi.kicad_sch (KiCad schematic)
At the start: 11 parts, among them J7 DC3RX19JA2

Commit message: FRANK_MEGA WIP
Parts:
- renumbered C21 to C22
Changed lines of the file:
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@@
 		(in_pos_files yes)
 		(dnp no)
-		(property "Reference" "C21"
+		(property "Reference" "C22"
 			(at 162.6616 82.169 0)
 			(show_name no)
@@
 			(project "frank_mega"
 				(path "/8c0b3d8b-46d3-4173-ab1e-a61765f77d61/db853a64-9343-4a36-b5b8-71001392b936"
-					(reference "C21")
+					(reference "C22")
 					(unit 1)
 				)

Commit message: New boards WIP
Parts:
- renumbered C22 to C23, J7 to J8
Changed lines of the file:
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@@
 		(dnp no)
 		(fields_autoplaced yes)
-		(property "Reference" "#PWR090"
+		(property "Reference" "#PWR094"
 			(at 151.13 74.93 0)
 			(hide yes)
@@
 			(project "frank_mega"
 				(path "/8c0b3d8b-46d3-4173-ab1e-a61765f77d61/db853a64-9343-4a36-b5b8-71001392b936"
-					(reference "#PWR090")
+					(reference "#PWR094")
 					(unit 1)
 				)
@@
 		(in_pos_files yes)
 		(dnp no)
-		(property "Reference" "C22"
+		(property "Reference" "C23"
 			(at 162.6616 82.169 0)
 			(show_name no)
@@
 			(project "frank_mega"
 				(path "/8c0b3d8b-46d3-4173-ab1e-a61765f77d61/db853a64-9343-4a36-b5b8-71001392b936"
-					(reference "C22")
+					(reference "C23")
 					(unit 1)
 				)
@@
 		(dnp no)
 		(fields_autoplaced yes)
-		(property "Reference" "#PWR089"
+		(property "Reference" "#PWR093"
 			(at 139.7 144.78 0)
 			(hide yes)
@@
 			(project "frank_mega"
 				(path "/8c0b3d8b-46d3-4173-ab1e-a61765f77d61/db853a64-9343-4a36-b5b8-71001392b936"
-					(reference "#PWR089")
+					(reference "#PWR093")
 					(unit 1)
 				)
@@
 		(dnp no)
 		(fields_autoplaced yes)
-		(property "Reference" "#PWR091"
+		(property "Reference" "#PWR095"
 			(at 173.99 85.09 0)
 			(hide yes)
@@
 			(project "frank_mega"
 				(path "/8c0b3d8b-46d3-4173-ab1e-a61765f77d61/db853a64-9343-4a36-b5b8-71001392b936"
-					(reference "#PWR091")
+					(reference "#PWR095")
 					(unit 1)
 				)
@@
 		(dnp no)
 		(fields_autoplaced yes)
-		(property "Reference" "J7"
+		(property "Reference" "J8"
 			(at 115.57 99.0599 0)
 			(show_name no)
@@
 			(project "frank_mega"
 				(path "/8c0b3d8b-46d3-4173-ab1e-a61765f77d61/db853a64-9343-4a36-b5b8-71001392b936"
-					(reference "J7")
-					(unit 1)
-				)
+					(reference "J8")
+					(unit 1)
+				)

Commit message: FRANK MEGA WIP
Parts:
- renumbered C23 to C24, R56 to R59, R57 to R60, R58 to R61, R59 to R62, R60 to R63, R61 to R64, R62 to R65, R63 to R66
Changed lines of the file:
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@@
 		(in_pos_files yes)
 		(dnp no)
-		(property "Reference" "R59"
+		(property "Reference" "R62"
 			(at 162.56 111.76 90)
 			(show_name no)
@@
 			(project "frank_mega"
 				(path "/8c0b3d8b-46d3-4173-ab1e-a61765f77d61/db853a64-9343-4a36-b5b8-71001392b936"
-					(reference "R59")
+					(reference "R62")
 					(unit 1)
 				)
@@
 		(in_pos_files yes)
 		(dnp no)
-		(property "Reference" "R63"
+		(property "Reference" "R66"
 			(at 172.72 119.38 90)
 			(show_name no)
@@
 			(project "frank_mega"
 				(path "/8c0b3d8b-46d3-4173-ab1e-a61765f77d61/db853a64-9343-4a36-b5b8-71001392b936"
-					(reference "R63")
+					(reference "R66")
 					(unit 1)
 				)
@@
 		(in_pos_files yes)
 		(dnp no)
-		(property "Reference" "R58"
+		(property "Reference" "R61"
 			(at 162.56 99.06 90)
 			(show_name no)
@@
 			(project "frank_mega"
 				(path "/8c0b3d8b-46d3-4173-ab1e-a61765f77d61/db853a64-9343-4a36-b5b8-71001392b936"
-					(reference "R58")
+					(reference "R61")
 					(unit 1)
 				)
@@
 		(dnp no)
 		(fields_autoplaced yes)
-		(property "Reference" "#PWR094"
+		(property "Reference" "#PWR099"
 			(at 151.13 74.93 0)
 			(hide yes)
@@
 			(project "frank_mega"
 				(path "/8c0b3d8b-46d3-4173-ab1e-a61765f77d61/db853a64-9343-4a36-b5b8-71001392b936"
-					(reference "#PWR094")
+					(reference "#PWR099")
 					(unit 1)
 				)
@@
 		(in_pos_files yes)
 		(dnp no)
-		(property "Reference" "R60"
+		(property "Reference" "R63"
 			(at 162.56 114.3 90)
 			(show_name no)
@@
 			(project "frank_mega"
 				(path "/8c0b3d8b-46d3-4173-ab1e-a61765f77d61/db853a64-9343-4a36-b5b8-71001392b936"
-					(reference "R60")
+					(reference "R63")
 					(unit 1)
 				)
@@
 		(in_pos_files yes)
 		(dnp no)
-		(property "Reference" "C23"
+		(property "Reference" "C24"
 			(at 162.6616 82.169 0)
 			(show_name no)
@@
 			(project "frank_mega"
 				(path "/8c0b3d8b-46d3-4173-ab1e-a61765f77d61/db853a64-9343-4a36-b5b8-71001392b936"
-					(reference "C23")
+					(reference "C24")
 					(unit 1)
 				)
@@
 		(in_pos_files yes)
 		(dnp no)
-		(property "Reference" "R56"
+		(property "Reference" "R59"
 			(at 152.4 106.68 90)
 			(show_name no)
@@
 			(project "frank_mega"
 				(path "/8c0b3d8b-46d3-4173-ab1e-a61765f77d61/db853a64-9343-4a36-b5b8-71001392b936"
-					(reference "R56")
+					(reference "R59")
 					(unit 1)
 				)
@@
 		(dnp no)
 		(fields_autoplaced yes)
-		(property "Reference" "#PWR093"
+		(property "Reference" "#PWR098"
 			(at 139.7 144.78 0)
 			(hide yes)
@@
 			(project "frank_mega"
 				(path "/8c0b3d8b-46d3-4173-ab1e-a61765f77d61/db853a64-9343-4a36-b5b8-71001392b936"
-					(reference "#PWR093")
+					(reference "#PWR098")
 					(unit 1)
 				)
@@
 		(dnp no)
 		(fields_autoplaced yes)
-		(property "Reference" "#PWR095"
+		(property "Reference" "#PWR0100"
 			(at 173.99 85.09 0)
 			(hide yes)
@@
 			(project "frank_mega"
 				(path "/8c0b3d8b-46d3-4173-ab1e-a61765f77d61/db853a64-9343-4a36-b5b8-71001392b936"
-					(reference "#PWR095")
+					(reference "#PWR0100")
 					(unit 1)
 				)
@@
 		(in_pos_files yes)
 		(dnp no)
-		(property "Reference" "R62"
+		(property "Reference" "R65"
 			(at 172.72 104.14 90)
 			(show_name no)
@@
 			(project "frank_mega"
 				(path "/8c0b3d8b-46d3-4173-ab1e-a61765f77d61/db853a64-9343-4a36-b5b8-71001392b936"
-					(reference "R62")
+					(reference "R65")
 					(unit 1)
 				)
@@
 		(in_pos_files yes)
 		(dnp no)
-		(property "Reference" "R61"
+		(property "Reference" "R64"
 			(at 162.56 127 90)
 			(show_name no)
@@
 			(project "frank_mega"
 				(path "/8c0b3d8b-46d3-4173-ab1e-a61765f77d61/db853a64-9343-4a36-b5b8-71001392b936"
-					(reference "R61")
+					(reference "R64")
 					(unit 1)
 				)
@@
 		(in_pos_files yes)
 		(dnp no)
-		(property "Reference" "R57"
+		(property "Reference" "R60"
 			(at 152.4 121.92 90)
 			(show_name no)
@@
 			(project "frank_mega"
 				(path "/8c0b3d8b-46d3-4173-ab1e-a61765f77d61/db853a64-9343-4a36-b5b8-71001392b936"
-					(reference "R57")
+					(reference "R60")
 					(unit 1)
 				)

Commit message: FRANK MEGA WIP
Parts:
- renumbered R59 to R63, R60 to R64, R61 to R65, R62 to R66, R63 to R67, R64 to R68, R65 to R69, R66 to R70
Changed lines of the file:
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@@
 		(in_pos_files yes)
 		(dnp no)
-		(property "Reference" "R62"
+		(property "Reference" "R66"
 			(at 162.56 111.76 90)
 			(show_name no)
@@
 			(project "frank_mega"
 				(path "/8c0b3d8b-46d3-4173-ab1e-a61765f77d61/db853a64-9343-4a36-b5b8-71001392b936"
-					(reference "R62")
+					(reference "R66")
 					(unit 1)
 				)
@@
 		(in_pos_files yes)
 		(dnp no)
-		(property "Reference" "R66"
+		(property "Reference" "R70"
 			(at 172.72 119.38 90)
 			(show_name no)
@@
 			(project "frank_mega"
 				(path "/8c0b3d8b-46d3-4173-ab1e-a61765f77d61/db853a64-9343-4a36-b5b8-71001392b936"
-					(reference "R66")
+					(reference "R70")
 					(unit 1)
 				)
@@
 		(in_pos_files yes)
 		(dnp no)
-		(property "Reference" "R61"
+		(property "Reference" "R65"
 			(at 162.56 99.06 90)
 			(show_name no)
@@
 			(project "frank_mega"
 				(path "/8c0b3d8b-46d3-4173-ab1e-a61765f77d61/db853a64-9343-4a36-b5b8-71001392b936"
-					(reference "R61")
+					(reference "R65")
 					(unit 1)
 				)
@@
 		(dnp no)
 		(fields_autoplaced yes)
-		(property "Reference" "#PWR099"
+		(property "Reference" "#PWR0100"
 			(at 151.13 74.93 0)
 			(hide yes)
@@
 			(project "frank_mega"
 				(path "/8c0b3d8b-46d3-4173-ab1e-a61765f77d61/db853a64-9343-4a36-b5b8-71001392b936"
-					(reference "#PWR099")
+					(reference "#PWR0100")
 					(unit 1)
 				)
@@
 		(in_pos_files yes)
 		(dnp no)
-		(property "Reference" "R63"
+		(property "Reference" "R67"
 			(at 162.56 114.3 90)
 			(show_name no)
@@
 			(project "frank_mega"
 				(path "/8c0b3d8b-46d3-4173-ab1e-a61765f77d61/db853a64-9343-4a36-b5b8-71001392b936"
-					(reference "R63")
+					(reference "R67")
 					(unit 1)
 				)
@@
 		(in_pos_files yes)
 		(dnp no)
-		(property "Reference" "R59"
+		(property "Reference" "R63"
 			(at 152.4 106.68 90)
 			(show_name no)
@@
 			(project "frank_mega"
 				(path "/8c0b3d8b-46d3-4173-ab1e-a61765f77d61/db853a64-9343-4a36-b5b8-71001392b936"
-					(reference "R59")
+					(reference "R63")
 					(unit 1)
 				)
@@
 		(dnp no)
 		(fields_autoplaced yes)
-		(property "Reference" "#PWR098"
+		(property "Reference" "#PWR099"
 			(at 139.7 144.78 0)
 			(hide yes)
@@
 			(project "frank_mega"
 				(path "/8c0b3d8b-46d3-4173-ab1e-a61765f77d61/db853a64-9343-4a36-b5b8-71001392b936"
-					(reference "#PWR098")
+					(reference "#PWR099")
 					(unit 1)
 				)
@@
 		(dnp no)
 		(fields_autoplaced yes)
-		(property "Reference" "#PWR0100"
+		(property "Reference" "#PWR0101"
 			(at 173.99 85.09 0)
 			(hide yes)
@@
 			(project "frank_mega"
 				(path "/8c0b3d8b-46d3-4173-ab1e-a61765f77d61/db853a64-9343-4a36-b5b8-71001392b936"
-					(reference "#PWR0100")
+					(reference "#PWR0101")
 					(unit 1)
 				)
@@
 		(in_pos_files yes)
 		(dnp no)
-		(property "Reference" "R65"
+		(property "Reference" "R69"
 			(at 172.72 104.14 90)
 			(show_name no)
@@
 			(project "frank_mega"
 				(path "/8c0b3d8b-46d3-4173-ab1e-a61765f77d61/db853a64-9343-4a36-b5b8-71001392b936"
-					(reference "R65")
+					(reference "R69")
 					(unit 1)
 				)
@@
 		(in_pos_files yes)
 		(dnp no)
-		(property "Reference" "R64"
+		(property "Reference" "R68"
 			(at 162.56 127 90)
 			(show_name no)
@@
 			(project "frank_mega"
 				(path "/8c0b3d8b-46d3-4173-ab1e-a61765f77d61/db853a64-9343-4a36-b5b8-71001392b936"
-					(reference "R64")
+					(reference "R68")
 					(unit 1)
 				)
@@
 		(in_pos_files yes)
 		(dnp no)
-		(property "Reference" "R60"
+		(property "Reference" "R64"
 			(at 152.4 121.92 90)
 			(show_name no)
@@
 			(project "frank_mega"
 				(path "/8c0b3d8b-46d3-4173-ab1e-a61765f77d61/db853a64-9343-4a36-b5b8-71001392b936"
-					(reference "R60")
+					(reference "R64")
 					(unit 1)
 				)

Commit message: FRANK MEGA WIP
Parts:
- renumbered J8 to J9
Changed lines of the file:
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@@
 		(dnp no)
 		(fields_autoplaced yes)
-		(property "Reference" "#PWR0100"
+		(property "Reference" "#PWR0103"
 			(at 151.13 74.93 0)
 			(hide yes)
@@
 			(project "frank_mega"
 				(path "/8c0b3d8b-46d3-4173-ab1e-a61765f77d61/db853a64-9343-4a36-b5b8-71001392b936"
-					(reference "#PWR0100")
+					(reference "#PWR0103")
 					(unit 1)
 				)
@@
 		(dnp no)
 		(fields_autoplaced yes)
-		(property "Reference" "#PWR099"
+		(property "Reference" "#PWR0102"
 			(at 139.7 144.78 0)
 			(hide yes)
@@
 			(project "frank_mega"
 				(path "/8c0b3d8b-46d3-4173-ab1e-a61765f77d61/db853a64-9343-4a36-b5b8-71001392b936"
-					(reference "#PWR099")
+					(reference "#PWR0102")
 					(unit 1)
 				)
@@
 		(dnp no)
 		(fields_autoplaced yes)
-		(property "Reference" "#PWR0101"
+		(property "Reference" "#PWR0104"
 			(at 173.99 85.09 0)
 			(hide yes)
@@
 			(project "frank_mega"
 				(path "/8c0b3d8b-46d3-4173-ab1e-a61765f77d61/db853a64-9343-4a36-b5b8-71001392b936"
-					(reference "#PWR0101")
+					(reference "#PWR0104")
 					(unit 1)
 				)
@@
 		(dnp no)
 		(fields_autoplaced yes)
-		(property "Reference" "J8"
+		(property "Reference" "J9"
 			(at 115.57 99.0599 0)
 			(show_name no)
@@
 			(project "frank_mega"
 				(path "/8c0b3d8b-46d3-4173-ab1e-a61765f77d61/db853a64-9343-4a36-b5b8-71001392b936"
-					(reference "J8")
-					(unit 1)
-				)
+					(reference "J9")
+					(unit 1)
+				)
