File: frank_mega/tda.kicad_sch (KiCad schematic)
At the start: 7 parts, among them U15 TDA1387T

Commit message: FRANK_MEGA WIP
Parts:
- renumbered C29 to C30, C30 to C31, C31 to C32
Changed lines of the file:
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@@
 		(in_pos_files yes)
 		(dnp no)
-		(property "Reference" "C30"
+		(property "Reference" "C31"
 			(at 169.418 112.014 90)
 			(show_name no)
@@
 			(project "frank_mega"
 				(path "/8c0b3d8b-46d3-4173-ab1e-a61765f77d61/9d0ad236-240c-42bd-9e4a-79b0506e7ea9/0dccd710-fd54-4e53-9f08-059759dd7a75"
-					(reference "C30")
+					(reference "C31")
 					(unit 1)
 				)
@@
 		(in_pos_files yes)
 		(dnp no)
-		(property "Reference" "C31"
+		(property "Reference" "C32"
 			(at 179.578 108.204 90)
 			(show_name no)
@@
 			(project "frank_mega"
 				(path "/8c0b3d8b-46d3-4173-ab1e-a61765f77d61/9d0ad236-240c-42bd-9e4a-79b0506e7ea9/0dccd710-fd54-4e53-9f08-059759dd7a75"
-					(reference "C31")
+					(reference "C32")
 					(unit 1)
 				)
@@
 		(in_pos_files yes)
 		(dnp no)
-		(property "Reference" "C29"
+		(property "Reference" "C30"
 			(at 160.528 112.014 90)
 			(show_name no)
@@
 			(project "frank_mega"
 				(path "/8c0b3d8b-46d3-4173-ab1e-a61765f77d61/9d0ad236-240c-42bd-9e4a-79b0506e7ea9/0dccd710-fd54-4e53-9f08-059759dd7a75"
-					(reference "C29")
+					(reference "C30")
 					(unit 1)
 				)

Commit message: New boards WIP
Parts:
- renumbered C30 to C31, C31 to C32, C32 to C33
Changed lines of the file:
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@@
 		(dnp no)
 		(fields_autoplaced yes)
-		(property "Reference" "#PWR0132"
+		(property "Reference" "#PWR0136"
 			(at 166.37 73.66 0)
 			(hide yes)
@@
 			(project "frank_mega"
 				(path "/8c0b3d8b-46d3-4173-ab1e-a61765f77d61/9d0ad236-240c-42bd-9e4a-79b0506e7ea9/0dccd710-fd54-4e53-9f08-059759dd7a75"
-					(reference "#PWR0132")
+					(reference "#PWR0136")
 					(unit 1)
 				)
@@
 		(in_pos_files yes)
 		(dnp no)
-		(property "Reference" "C31"
+		(property "Reference" "C32"
 			(at 169.418 112.014 90)
 			(show_name no)
@@
 			(project "frank_mega"
 				(path "/8c0b3d8b-46d3-4173-ab1e-a61765f77d61/9d0ad236-240c-42bd-9e4a-79b0506e7ea9/0dccd710-fd54-4e53-9f08-059759dd7a75"
-					(reference "C31")
+					(reference "C32")
 					(unit 1)
 				)
@@
 		(dnp no)
 		(fields_autoplaced yes)
-		(property "Reference" "#PWR0136"
+		(property "Reference" "#PWR0140"
 			(at 186.69 109.22 0)
 			(hide yes)
@@
 			(project "frank_mega"
 				(path "/8c0b3d8b-46d3-4173-ab1e-a61765f77d61/9d0ad236-240c-42bd-9e4a-79b0506e7ea9/0dccd710-fd54-4e53-9f08-059759dd7a75"
-					(reference "#PWR0136")
+					(reference "#PWR0140")
 					(unit 1)
 				)
@@
 		(dnp no)
 		(fields_autoplaced yes)
-		(property "Reference" "#PWR0135"
+		(property "Reference" "#PWR0139"
 			(at 186.69 68.58 0)
 			(hide yes)
@@
 			(project "frank_mega"
 				(path "/8c0b3d8b-46d3-4173-ab1e-a61765f77d61/9d0ad236-240c-42bd-9e4a-79b0506e7ea9/0dccd710-fd54-4e53-9f08-059759dd7a75"
-					(reference "#PWR0135")
+					(reference "#PWR0139")
 					(unit 1)
 				)
@@
 		(dnp no)
 		(fields_autoplaced yes)
-		(property "Reference" "#PWR0130"
+		(property "Reference" "#PWR0134"
 			(at 116.84 109.22 0)
 			(hide yes)
@@
 			(project "frank_mega"
 				(path "/8c0b3d8b-46d3-4173-ab1e-a61765f77d61/9d0ad236-240c-42bd-9e4a-79b0506e7ea9/0dccd710-fd54-4e53-9f08-059759dd7a75"
-					(reference "#PWR0130")
+					(reference "#PWR0134")
 					(unit 1)
 				)
@@
 		(in_pos_files yes)
 		(dnp no)
-		(property "Reference" "#PWR0133"
+		(property "Reference" "#PWR0137"
 			(at 166.37 121.92 0)
 			(hide yes)
@@
 			(project "frank_mega"
 				(path "/8c0b3d8b-46d3-4173-ab1e-a61765f77d61/9d0ad236-240c-42bd-9e4a-79b0506e7ea9/0dccd710-fd54-4e53-9f08-059759dd7a75"
-					(reference "#PWR0133")
+					(reference "#PWR0137")
 					(unit 1)
 				)
@@
 		(in_pos_files yes)
 		(dnp no)
-		(property "Reference" "C32"
+		(property "Reference" "C33"
 			(at 179.578 108.204 90)
 			(show_name no)
@@
 			(project "frank_mega"
 				(path "/8c0b3d8b-46d3-4173-ab1e-a61765f77d61/9d0ad236-240c-42bd-9e4a-79b0506e7ea9/0dccd710-fd54-4e53-9f08-059759dd7a75"
-					(reference "C32")
+					(reference "C33")
 					(unit 1)
 				)
@@
 		(dnp no)
 		(fields_autoplaced yes)
-		(property "Reference" "#PWR0131"
+		(property "Reference" "#PWR0135"
 			(at 157.48 121.92 0)
 			(hide yes)
@@
 			(project "frank_mega"
 				(path "/8c0b3d8b-46d3-4173-ab1e-a61765f77d61/9d0ad236-240c-42bd-9e4a-79b0506e7ea9/0dccd710-fd54-4e53-9f08-059759dd7a75"
-					(reference "#PWR0131")
+					(reference "#PWR0135")
 					(unit 1)
 				)
@@
 		(in_pos_files yes)
 		(dnp no)
-		(property "Reference" "C30"
+		(property "Reference" "C31"
 			(at 160.528 112.014 90)
 			(show_name no)
@@
 			(project "frank_mega"
 				(path "/8c0b3d8b-46d3-4173-ab1e-a61765f77d61/9d0ad236-240c-42bd-9e4a-79b0506e7ea9/0dccd710-fd54-4e53-9f08-059759dd7a75"
-					(reference "C30")
+					(reference "C31")
 					(unit 1)
 				)
@@
 		(dnp no)
 		(fields_autoplaced yes)
-		(property "Reference" "#PWR0134"
+		(property "Reference" "#PWR0138"
 			(at 176.53 121.92 0)
 			(hide yes)
@@
 			(project "frank_mega"
 				(path "/8c0b3d8b-46d3-4173-ab1e-a61765f77d61/9d0ad236-240c-42bd-9e4a-79b0506e7ea9/0dccd710-fd54-4e53-9f08-059759dd7a75"
-					(reference "#PWR0134")
+					(reference "#PWR0138")
 					(unit 1)
 				)

Commit message: FRANK MEGA WIP
Parts:
- renumbered C31 to C33, C32 to C34, C33 to C35, R91 to R94, R92 to R95, R93 to R96, U15 to U18
Changed lines of the file:
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@@
 		(dnp no)
 		(fields_autoplaced yes)
-		(property "Reference" "#PWR0136"
+		(property "Reference" "#PWR0147"
 			(at 166.37 73.66 0)
 			(hide yes)
@@
 			(project "frank_mega"
 				(path "/8c0b3d8b-46d3-4173-ab1e-a61765f77d61/9d0ad236-240c-42bd-9e4a-79b0506e7ea9/0dccd710-fd54-4e53-9f08-059759dd7a75"
-					(reference "#PWR0136")
+					(reference "#PWR0147")
 					(unit 1)
 				)
@@
 		(in_pos_files yes)
 		(dnp no)
-		(property "Reference" "R91"
+		(property "Reference" "R94"
 			(at 163.83 78.74 90)
 			(show_name no)
@@
 			(project "frank_mega"
 				(path "/8c0b3d8b-46d3-4173-ab1e-a61765f77d61/9d0ad236-240c-42bd-9e4a-79b0506e7ea9/0dccd710-fd54-4e53-9f08-059759dd7a75"
-					(reference "R91")
+					(reference "R94")
 					(unit 1)
 				)
@@
 		(dnp no)
 		(fields_autoplaced yes)
-		(property "Reference" "U15"
+		(property "Reference" "U18"
 			(at 140.97 76.2 0)
 			(show_name no)
@@
 			(project "frank_mega"
 				(path "/8c0b3d8b-46d3-4173-ab1e-a61765f77d61/9d0ad236-240c-42bd-9e4a-79b0506e7ea9/0dccd710-fd54-4e53-9f08-059759dd7a75"
-					(reference "U15")
+					(reference "U18")
 					(unit 1)
 				)
@@
 		(in_pos_files yes)
 		(dnp no)
-		(property "Reference" "C32"
+		(property "Reference" "C34"
 			(at 169.418 112.014 90)
 			(show_name no)
@@
 			(project "frank_mega"
 				(path "/8c0b3d8b-46d3-4173-ab1e-a61765f77d61/9d0ad236-240c-42bd-9e4a-79b0506e7ea9/0dccd710-fd54-4e53-9f08-059759dd7a75"
-					(reference "C32")
+					(reference "C34")
 					(unit 1)
 				)
@@
 		(in_pos_files yes)
 		(dnp no)
-		(property "Reference" "R93"
+		(property "Reference" "R96"
 			(at 184.15 97.79 90)
 			(show_name no)
@@
 			(project "frank_mega"
 				(path "/8c0b3d8b-46d3-4173-ab1e-a61765f77d61/9d0ad236-240c-42bd-9e4a-79b0506e7ea9/0dccd710-fd54-4e53-9f08-059759dd7a75"
-					(reference "R93")
+					(reference "R96")
 					(unit 1)
 				)
@@
 		(dnp no)
 		(fields_autoplaced yes)
-		(property "Reference" "#PWR0140"
+		(property "Reference" "#PWR0151"
 			(at 186.69 109.22 0)
 			(hide yes)
@@
 			(project "frank_mega"
 				(path "/8c0b3d8b-46d3-4173-ab1e-a61765f77d61/9d0ad236-240c-42bd-9e4a-79b0506e7ea9/0dccd710-fd54-4e53-9f08-059759dd7a75"
-					(reference "#PWR0140")
+					(reference "#PWR0151")
 					(unit 1)
 				)
@@
 		(dnp no)
 		(fields_autoplaced yes)
-		(property "Reference" "#PWR0139"
+		(property "Reference" "#PWR0150"
 			(at 186.69 68.58 0)
 			(hide yes)
@@
 			(project "frank_mega"
 				(path "/8c0b3d8b-46d3-4173-ab1e-a61765f77d61/9d0ad236-240c-42bd-9e4a-79b0506e7ea9/0dccd710-fd54-4e53-9f08-059759dd7a75"
-					(reference "#PWR0139")
+					(reference "#PWR0150")
 					(unit 1)
 				)
@@
 		(in_pos_files yes)
 		(dnp no)
-		(property "Reference" "R92"
+		(property "Reference" "R95"
 			(at 184.15 80.01 90)
 			(show_name no)
@@
 			(project "frank_mega"
 				(path "/8c0b3d8b-46d3-4173-ab1e-a61765f77d61/9d0ad236-240c-42bd-9e4a-79b0506e7ea9/0dccd710-fd54-4e53-9f08-059759dd7a75"
-					(reference "R92")
+					(reference "R95")
 					(unit 1)
 				)
@@
 		(dnp no)
 		(fields_autoplaced yes)
-		(property "Reference" "#PWR0134"
+		(property "Reference" "#PWR0145"
 			(at 116.84 109.22 0)
 			(hide yes)
@@
 			(project "frank_mega"
 				(path "/8c0b3d8b-46d3-4173-ab1e-a61765f77d61/9d0ad236-240c-42bd-9e4a-79b0506e7ea9/0dccd710-fd54-4e53-9f08-059759dd7a75"
-					(reference "#PWR0134")
+					(reference "#PWR0145")
 					(unit 1)
 				)
@@
 		(in_pos_files yes)
 		(dnp no)
-		(property "Reference" "#PWR0137"
+		(property "Reference" "#PWR0148"
 			(at 166.37 121.92 0)
 			(hide yes)
@@
 			(project "frank_mega"
 				(path "/8c0b3d8b-46d3-4173-ab1e-a61765f77d61/9d0ad236-240c-42bd-9e4a-79b0506e7ea9/0dccd710-fd54-4e53-9f08-059759dd7a75"
-					(reference "#PWR0137")
+					(reference "#PWR0148")
 					(unit 1)
 				)
@@
 		(in_pos_files yes)
 		(dnp no)
-		(property "Reference" "C33"
+		(property "Reference" "C35"
 			(at 179.578 108.204 90)
 			(show_name no)
@@
 			(project "frank_mega"
 				(path "/8c0b3d8b-46d3-4173-ab1e-a61765f77d61/9d0ad236-240c-42bd-9e4a-79b0506e7ea9/0dccd710-fd54-4e53-9f08-059759dd7a75"
-					(reference "C33")
+					(reference "C35")
 					(unit 1)
 				)
@@
 		(dnp no)
 		(fields_autoplaced yes)
-		(property "Reference" "#PWR0135"
+		(property "Reference" "#PWR0146"
 			(at 157.48 121.92 0)
 			(hide yes)
@@
 			(project "frank_mega"
 				(path "/8c0b3d8b-46d3-4173-ab1e-a61765f77d61/9d0ad236-240c-42bd-9e4a-79b0506e7ea9/0dccd710-fd54-4e53-9f08-059759dd7a75"
-					(reference "#PWR0135")
+					(reference "#PWR0146")
 					(unit 1)
 				)
@@
 		(in_pos_files yes)
 		(dnp no)
-		(property "Reference" "C31"
+		(property "Reference" "C33"
 			(at 160.528 112.014 90)
 			(show_name no)
@@
 			(project "frank_mega"
 				(path "/8c0b3d8b-46d3-4173-ab1e-a61765f77d61/9d0ad236-240c-42bd-9e4a-79b0506e7ea9/0dccd710-fd54-4e53-9f08-059759dd7a75"
-					(reference "C31")
+					(reference "C33")
 					(unit 1)
 				)
@@
 		(dnp no)
 		(fields_autoplaced yes)
-		(property "Reference" "#PWR0138"
+		(property "Reference" "#PWR0149"
 			(at 176.53 121.92 0)
 			(hide yes)
@@
 			(project "frank_mega"
 				(path "/8c0b3d8b-46d3-4173-ab1e-a61765f77d61/9d0ad236-240c-42bd-9e4a-79b0506e7ea9/0dccd710-fd54-4e53-9f08-059759dd7a75"
-					(reference "#PWR0138")
+					(reference "#PWR0149")
 					(unit 1)
 				)

Commit message: FRANK MEGA WIP
Parts:
- renumbered R96 to R100, R94 to R98, R95 to R99
Changed lines of the file:
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@@
 		(dnp no)
 		(fields_autoplaced yes)
-		(property "Reference" "#PWR0147"
+		(property "Reference" "#PWR0148"
 			(at 166.37 73.66 0)
 			(hide yes)
@@
 			(project "frank_mega"
 				(path "/8c0b3d8b-46d3-4173-ab1e-a61765f77d61/9d0ad236-240c-42bd-9e4a-79b0506e7ea9/0dccd710-fd54-4e53-9f08-059759dd7a75"
-					(reference "#PWR0147")
+					(reference "#PWR0148")
 					(unit 1)
 				)
@@
 		(in_pos_files yes)
 		(dnp no)
-		(property "Reference" "R94"
+		(property "Reference" "R98"
 			(at 163.83 78.74 90)
 			(show_name no)
@@
 			(project "frank_mega"
 				(path "/8c0b3d8b-46d3-4173-ab1e-a61765f77d61/9d0ad236-240c-42bd-9e4a-79b0506e7ea9/0dccd710-fd54-4e53-9f08-059759dd7a75"
-					(reference "R94")
+					(reference "R98")
 					(unit 1)
 				)
@@
 		(in_pos_files yes)
 		(dnp no)
-		(property "Reference" "R96"
+		(property "Reference" "R100"
 			(at 184.15 97.79 90)
 			(show_name no)
@@
 			(project "frank_mega"
 				(path "/8c0b3d8b-46d3-4173-ab1e-a61765f77d61/9d0ad236-240c-42bd-9e4a-79b0506e7ea9/0dccd710-fd54-4e53-9f08-059759dd7a75"
-					(reference "R96")
+					(reference "R100")
 					(unit 1)
 				)
@@
 		(dnp no)
 		(fields_autoplaced yes)
-		(property "Reference" "#PWR0151"
+		(property "Reference" "#PWR0152"
 			(at 186.69 109.22 0)
 			(hide yes)
@@
 			(project "frank_mega"
 				(path "/8c0b3d8b-46d3-4173-ab1e-a61765f77d61/9d0ad236-240c-42bd-9e4a-79b0506e7ea9/0dccd710-fd54-4e53-9f08-059759dd7a75"
-					(reference "#PWR0151")
+					(reference "#PWR0152")
 					(unit 1)
 				)
@@
 		(dnp no)
 		(fields_autoplaced yes)
-		(property "Reference" "#PWR0150"
+		(property "Reference" "#PWR0151"
 			(at 186.69 68.58 0)
 			(hide yes)
@@
 			(project "frank_mega"
 				(path "/8c0b3d8b-46d3-4173-ab1e-a61765f77d61/9d0ad236-240c-42bd-9e4a-79b0506e7ea9/0dccd710-fd54-4e53-9f08-059759dd7a75"
-					(reference "#PWR0150")
+					(reference "#PWR0151")
 					(unit 1)
 				)
@@
 		(in_pos_files yes)
 		(dnp no)
-		(property "Reference" "R95"
+		(property "Reference" "R99"
 			(at 184.15 80.01 90)
 			(show_name no)
@@
 			(project "frank_mega"
 				(path "/8c0b3d8b-46d3-4173-ab1e-a61765f77d61/9d0ad236-240c-42bd-9e4a-79b0506e7ea9/0dccd710-fd54-4e53-9f08-059759dd7a75"
-					(reference "R95")
+					(reference "R99")
 					(unit 1)
 				)
@@
 		(dnp no)
 		(fields_autoplaced yes)
-		(property "Reference" "#PWR0145"
+		(property "Reference" "#PWR0146"
 			(at 116.84 109.22 0)
 			(hide yes)
@@
 			(project "frank_mega"
 				(path "/8c0b3d8b-46d3-4173-ab1e-a61765f77d61/9d0ad236-240c-42bd-9e4a-79b0506e7ea9/0dccd710-fd54-4e53-9f08-059759dd7a75"
-					(reference "#PWR0145")
+					(reference "#PWR0146")
 					(unit 1)
 				)
@@
 		(in_pos_files yes)
 		(dnp no)
-		(property "Reference" "#PWR0148"
+		(property "Reference" "#PWR0149"
 			(at 166.37 121.92 0)
 			(hide yes)
@@
 			(project "frank_mega"
 				(path "/8c0b3d8b-46d3-4173-ab1e-a61765f77d61/9d0ad236-240c-42bd-9e4a-79b0506e7ea9/0dccd710-fd54-4e53-9f08-059759dd7a75"
-					(reference "#PWR0148")
+					(reference "#PWR0149")
 					(unit 1)
 				)
@@
 		(dnp no)
 		(fields_autoplaced yes)
-		(property "Reference" "#PWR0146"
+		(property "Reference" "#PWR0147"
 			(at 157.48 121.92 0)
 			(hide yes)
@@
 			(project "frank_mega"
 				(path "/8c0b3d8b-46d3-4173-ab1e-a61765f77d61/9d0ad236-240c-42bd-9e4a-79b0506e7ea9/0dccd710-fd54-4e53-9f08-059759dd7a75"
-					(reference "#PWR0146")
+					(reference "#PWR0147")
 					(unit 1)
 				)
@@
 		(dnp no)
 		(fields_autoplaced yes)
-		(property "Reference" "#PWR0149"
+		(property "Reference" "#PWR0150"
 			(at 176.53 121.92 0)
 			(hide yes)
@@
 			(project "frank_mega"
 				(path "/8c0b3d8b-46d3-4173-ab1e-a61765f77d61/9d0ad236-240c-42bd-9e4a-79b0506e7ea9/0dccd710-fd54-4e53-9f08-059759dd7a75"
-					(reference "#PWR0149")
+					(reference "#PWR0150")
 					(unit 1)
 				)
