File: protea/esp32-flash.kicad_sch (KiCad schematic)
At the start: 2 parts, among them U8 W25Q32JVSIQ

Commit message: Protea 2.00 WIP
Parts:
- C23: renamed from C29; footprint FRANK:C_0603_1608Metric_HandSolder -> Protea:C_0603_1608Metric_HandSolder; symbol FRANK:C -> Protea:C
- U4: renamed from U8; footprint FRANK:SOIC-8 -> Protea:SOIC-8_Longer; symbol FRANK:Flash_W25Q128JVS -> Protea:Flash_W25Q128JVS
Changed lines of the file:
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@@
 		(rev "${VERSION}")
 		(company "Mikhail Matveev")
-		(comment 1 "https://github.com/xtremespb/frank")
+		(comment 1 "https://github.com/rh1tech/protea")
 	)
 	(junction
@@
 	)
 	(symbol
-		(lib_id "FRANK:Flash_W25Q128JVS")
+		(lib_id "Protea:Flash_W25Q128JVS")
 		(at 162.56 100.33 0)
 		(unit 1)
@@
 		(in_pos_files yes)
 		(dnp no)
-		(property "Reference" "U8"
+		(property "Reference" "U4"
 			(at 156.21 88.265 0)
 			(show_name no)
@@
 			)
 		)
-		(property "Footprint" "FRANK:SOIC-8"
+		(property "Footprint" "Protea:SOIC-8_Longer"
 			(at 162.56 100.33 0)
 			(hide yes)
@@
 			)
 		)
-		(property "Datasheet" "http://www.winbond.com/resource-files/w25q128jv_dtr%20revc%2003272018%20plus.pdf"
+		(property "Datasheet" "https://www.winbond.com/resource-files/w25q128jv_dtr%20revc%2003272018%20plus.pdf"
 			(at 162.56 100.33 0)
 			(hide yes)
@@
 			(project "protea"
 				(path "/8c0b3d8b-46d3-4173-ab1e-a61765f77d61/6ffc8eb2-26a4-4e0a-a8e8-79eef59e436d/3907d691-16c9-46b9-8e1c-0399c2dec8f4"
-					(reference "U8")
+					(reference "U4")
 					(unit 1)
 				)
@@
 	(symbol
 		(lib_name "GND_10")
-		(lib_id "FRANK:GND")
+		(lib_id "Protea:GND")
 		(at 162.56 113.03 0)
 		(unit 1)
@@
 		(in_pos_files yes)
 		(dnp no)
-		(property "Reference" "#PWR083"
+		(property "Reference" "#PWR052"
 			(at 162.56 119.38 0)
 			(hide yes)
@@
 			(project "protea"
 				(path "/8c0b3d8b-46d3-4173-ab1e-a61765f77d61/6ffc8eb2-26a4-4e0a-a8e8-79eef59e436d/3907d691-16c9-46b9-8e1c-0399c2dec8f4"
-					(reference "#PWR083")
+					(reference "#PWR052")
 					(unit 1)
 				)
@@
 	)
 	(symbol
-		(lib_id "FRANK:C")
+		(lib_id "Protea:C")
 		(at 175.26 83.82 90)
 		(unit 1)
@@
 		(in_pos_files yes)
 		(dnp no)
-		(property "Reference" "C29"
+		(property "Reference" "C23"
 			(at 177.038 80.264 90)
 			(show_name no)
@@
 			)
 		)
-		(property "Footprint" "FRANK:C_0603_1608Metric_HandSolder"
+		(property "Footprint" "Protea:C_0603_1608Metric_HandSolder"
 			(at 179.07 82.8548 0)
 			(hide yes)
@@
 			(project "protea"
 				(path "/8c0b3d8b-46d3-4173-ab1e-a61765f77d61/6ffc8eb2-26a4-4e0a-a8e8-79eef59e436d/3907d691-16c9-46b9-8e1c-0399c2dec8f4"
-					(reference "C29")
+					(reference "C23")
 					(unit 1)
 				)
@@
 	)
 	(symbol
-		(lib_id "FRANK:GND")
+		(lib_id "Protea:GND")
 		(at 179.07 83.82 90)
 		(unit 1)
@@
 		(in_pos_files yes)
 		(dnp no)
-		(property "Reference" "#PWR084"
+		(property "Reference" "#PWR053"
 			(at 185.42 83.82 0)
 			(hide yes)
@@
 			(project "protea"
 				(path "/8c0b3d8b-46d3-4173-ab1e-a61765f77d61/6ffc8eb2-26a4-4e0a-a8e8-79eef59e436d/3907d691-16c9-46b9-8e1c-0399c2dec8f4"
-					(reference "#PWR084")
+					(reference "#PWR053")
 					(unit 1)
 				)
