File: protea/esp_flash.kicad_sch (KiCad schematic)
At the start: 2 parts

Commit message: Protea 2.00 WIP
Parts:
- S4: renamed from S6; footprint FRANK:KMR_2 -> Protea:KMR_2; symbol FRANK:KMR221G_LFS -> Protea:KMR221G_LFS
- S5: renamed from S7; footprint FRANK:KMR_2 -> Protea:KMR_2; symbol FRANK:KMR221G_LFS -> Protea:KMR221G_LFS
Changed lines of the file:
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@@
 		(rev "${VERSION}")
 		(company "Mikhail Matveev")
-		(comment 1 "https://github.com/rh1tech/frank")
+		(comment 1 "https://github.com/rh1tech/protea")
 	)
 	(hierarchical_label "ESP_FLASH"
@@
 	)
 	(symbol
-		(lib_id "FRANK:GND")
+		(lib_id "Protea:GND")
 		(at 170.18 121.92 90)
 		(unit 1)
@@
 		(in_pos_files yes)
 		(dnp no)
-		(property "Reference" "#PWR090"
+		(property "Reference" "#PWR059"
 			(at 176.53 121.92 0)
 			(hide yes)
@@
 			(project "protea"
 				(path "/8c0b3d8b-46d3-4173-ab1e-a61765f77d61/6b6a9768-d263-48b1-b95b-0ebb6152887f"
-					(reference "#PWR090")
+					(reference "#PWR059")
 					(unit 1)
 				)
@@
 	)
 	(symbol
-		(lib_id "FRANK:GND")
+		(lib_id "Protea:GND")
 		(at 149.86 121.92 270)
 		(unit 1)
@@
 		(in_pos_files yes)
 		(dnp no)
-		(property "Reference" "#PWR088"
+		(property "Reference" "#PWR057"
 			(at 143.51 121.92 0)
 			(hide yes)
@@
 			(project "protea"
 				(path "/8c0b3d8b-46d3-4173-ab1e-a61765f77d61/6b6a9768-d263-48b1-b95b-0ebb6152887f"
-					(reference "#PWR088")
+					(reference "#PWR057")
 					(unit 1)
 				)
@@
 	)
 	(symbol
-		(lib_id "FRANK:GND")
+		(lib_id "Protea:GND")
 		(at 149.86 106.68 270)
 		(unit 1)
@@
 		(in_pos_files yes)
 		(dnp no)
-		(property "Reference" "#PWR087"
+		(property "Reference" "#PWR056"
 			(at 143.51 106.68 0)
 			(hide yes)
@@
 			(project "protea"
 				(path "/8c0b3d8b-46d3-4173-ab1e-a61765f77d61/6b6a9768-d263-48b1-b95b-0ebb6152887f"
-					(reference "#PWR087")
+					(reference "#PWR056")
 					(unit 1)
 				)
@@
 	)
 	(symbol
-		(lib_id "FRANK:GND")
+		(lib_id "Protea:GND")
 		(at 170.18 106.68 90)
 		(unit 1)
@@
 		(in_pos_files yes)
 		(dnp no)
-		(property "Reference" "#PWR089"
+		(property "Reference" "#PWR058"
 			(at 176.53 106.68 0)
 			(hide yes)
@@
 			(project "protea"
 				(path "/8c0b3d8b-46d3-4173-ab1e-a61765f77d61/6b6a9768-d263-48b1-b95b-0ebb6152887f"
-					(reference "#PWR089")
+					(reference "#PWR058")
 					(unit 1)
 				)
@@
 	)
 	(symbol
-		(lib_id "FRANK:KMR221G_LFS")
+		(lib_id "Protea:KMR221G_LFS")
 		(at 149.86 119.38 0)
 		(unit 1)
@@
 		(in_pos_files yes)
 		(dnp no)
-		(property "Reference" "S7"
+		(property "Reference" "S5"
 			(at 160.02 113.03 0)
 			(show_name no)
@@
 			)
 		)
-		(property "Footprint" "FRANK:KMR_2"
+		(property "Footprint" "Protea:KMR_2"
 			(at 166.37 214.3 0)
 			(hide yes)
@@
 			(project "protea"
 				(path "/8c0b3d8b-46d3-4173-ab1e-a61765f77d61/6b6a9768-d263-48b1-b95b-0ebb6152887f"
-					(reference "S7")
+					(reference "S5")
 					(unit 1)
 				)
@@
 	)
 	(symbol
-		(lib_id "FRANK:KMR221G_LFS")
+		(lib_name "KMR221G_LFS_1")
+		(lib_id "Protea:KMR221G_LFS")
 		(at 149.86 104.14 0)
 		(unit 1)
@@
 		(in_pos_files yes)
 		(dnp no)
-		(property "Reference" "S6"
+		(property "Reference" "S4"
 			(at 160.02 97.79 0)
 			(show_name no)
@@
 			)
 		)
-		(property "Footprint" "FRANK:KMR_2"
+		(property "Footprint" "Protea:KMR_2"
 			(at 166.37 199.06 0)
 			(hide yes)
@@
 			(project "protea"
 				(path "/8c0b3d8b-46d3-4173-ab1e-a61765f77d61/6b6a9768-d263-48b1-b95b-0ebb6152887f"
-					(reference "S6")
+					(reference "S4")
 					(unit 1)
 				)
