File: protea/power.kicad_sch (KiCad schematic)
At the start: 17 parts, among them J5 USB4215-03-A, U3 USBLC6-2SC6, U6 AMS1117-3.3

Commit message: Protea 2.00 WIP
Parts:
- removed C9: 100n, FRANK:C_0603_1608Metric, symbol FRANK:C
- removed JP3: VBUS_IN Dbg, FRANK:SolderJumper-2_P1.3mm_Open_RoundedPad1.0x1.5mm, symbol FRANK:SolderJumper_2_Open
- removed L1: 330R, FRANK:L_0603_1608Metric, symbol FRANK:Ferrite_Bead
- removed S5: SK12D07VG3NS, FRANK:SK12D07VG3NS_PWR, symbol FRANK:SK12D07VG3NS
- added C2: 100n, Protea:C_0603_1608Metric, symbol Protea:C
- added L1: 330R, Protea:L_0603_1608Metric, symbol Protea:Ferrite_Bead
- added S3: SK12D07VG3NS, Protea:SK12D07VG3NS_PWR, symbol Protea:SK12D07VG3NS
- C1: renamed from C6; footprint FRANK:CP_Tantalum_3528-12 -> Protea:CP_Tantalum_3528-12; symbol FRANK:C_Polarized_Small -> Protea:C_Polarized_Small
- C3: renamed from C7; footprint FRANK:C_0603_1608Metric -> Protea:C_0603_1608Metric; symbol FRANK:C_Small -> Protea:C_Small
- C4: renamed from C10; footprint FRANK:CP_Tantalum_3528-12 -> Protea:CP_Tantalum_3528-12; symbol FRANK:C_Polarized_Small -> Protea:C_Polarized_Small
- C5: renamed from C11; footprint FRANK:C_0603_1608Metric -> Protea:C_0603_1608Metric; symbol FRANK:C_Small -> Protea:C_Small
- J4: renamed from J5; footprint FRANK:USB_C_Receptacle -> Protea:USB_C_Receptacle; symbol FRANK:USB_C -> Protea:USB_C
- LD2: renamed from LD4; footprint FRANK:LED_0603_1608Metric -> Protea:LED_0603_1608Metric; symbol FRANK:LED -> Protea:LED
- R5: renamed from R21; footprint FRANK:R_0603_1608Metric -> Protea:R_0603_1608Metric; symbol FRANK:R_Small -> Protea:R_Small
- R6: renamed from R22; footprint FRANK:R_0603_1608Metric -> Protea:R_0603_1608Metric; symbol FRANK:R_Small -> Protea:R_Small
- R7: renamed from R24; footprint FRANK:R_0603_1608Metric -> Protea:R_0603_1608Metric; symbol FRANK:R -> Protea:R
- R8: renamed from R25; footprint FRANK:R_0603_1608Metric -> Protea:R_0603_1608Metric; symbol FRANK:R -> Protea:R
- R9: renamed from R27; footprint FRANK:R_0603_1608Metric -> Protea:R_0603_1608Metric; symbol FRANK:R -> Protea:R
- U1: renamed from U3; footprint FRANK:SOT-23-6 -> Protea:SOT-23-6; symbol FRANK:USBLC6-2SC6 -> Protea:USBLC6-2SC6
- U2: renamed from U6; footprint FRANK:SOT-89-3 -> Protea:SOT-89-3; symbol FRANK:AMS1117-3.3 -> Protea:AMS1117-3.3
Connections:
- net GND: now also C2.2
- net VBUS: now also L1.1
- net VBUS_IN: now also J4.11 (VBUS), J4.2 (VBUS), S3.2
- new net: C2.1, L1.2, S3.1
