File: minifrank/power.kicad_sch (KiCad schematic)
At the start: 28 parts, among them J4 SS-52100-004, J5 USB4215-03-A, U1 TS3USB221RSER, U2 USBLC6-2SC6, U3 MW7211A, U4 AMS1117-3.3

Commit message: Board updates
Parts:
- C4, C7: footprint FRANK:Capacitor (3528, tantalum, polar) -> FRANK:CP_EIA-3528-12_Kemet-T
- J4: footprint FRANK:USB Type A (stacked) -> FRANK:USB_A_Stacked
- J5: footprint FRANK:USB Type C -> FRANK:USB_C_Receptacle
Changed lines of the file:
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@@
 			)
 		)
-		(property "Footprint" "FRANK:USB Type A (stacked)"
+		(property "Footprint" "FRANK:USB_A_Stacked"
 			(at 40.64 66.04 0)
 			(hide yes)
@@
 			)
 		)
-		(property "Footprint" "FRANK:Capacitor (3528, tantalum, polar)"
+		(property "Footprint" "FRANK:CP_EIA-3528-12_Kemet-T"
 			(at 214.63 40.64 0)
 			(hide yes)
@@
 			)
 		)
-		(property "Footprint" "FRANK:USB Type C"
+		(property "Footprint" "FRANK:USB_C_Receptacle"
 			(at 125.73 74.93 0)
 			(hide yes)
@@
 			)
 		)
-		(property "Footprint" "FRANK:Capacitor (3528, tantalum, polar)"
+		(property "Footprint" "FRANK:CP_EIA-3528-12_Kemet-T"
 			(at 242.57 40.64 0)
 			(hide yes)
