File: minifrank/vga.kicad_sch (KiCad schematic)
At the start: 9 parts, among them J11 VGA

Commit message: Board updates
Parts:
- J11: footprint FRANK:D-SUB (15 pin, female) -> FRANK:DSUB-15_Female
Changed lines of the file:
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@@
 			)
 		)
-		(property "Footprint" "FRANK:D-SUB (15 pin, female)"
+		(property "Footprint" "FRANK:DSUB-15_Female"
 			(at 133.35 92.71 0)
 			(hide yes)
