File: hecate/power.kicad_sch (KiCad schematic)
At the start: 15 parts, among them J4 USB4215-03-A, U4 USBLC6-2SC6, U5 AMS1117-3.3

Commit message: Hecate 3.00
Parts:
- removed C22: 100n, Hecate:C_0603_1608Metric, symbol Hecate:C
- removed C23, C25: 22u, Hecate:CP_EIA-3528-12_Kemet-T, symbol Hecate:C_Polarized_Small
- removed L1: 330R, Hecate:L_0603_1608Metric, symbol Hecate:FerriteBead
- removed U4: USBLC6-2SC6, Hecate:SOT-23-6, symbol Hecate:USBLC6-2SC6
- added C22: 100n, Hecate:C_0603_1608Metric, symbol Hecate:C_Small
- added C23, C25: 10u, Hecate:C_0603_1608Metric, symbol Hecate:C_Small
- renumbered R13 to R12, R14 to R13, R12 to R14
Connections:
- net VBUS_IN is gone; now on net VBUS: J4.11 (VBUS), J4.2 (VBUS)
- net +3V3: now also C25.2
- net D+: now also R13.1
- net D-: now also R12.1
- net GND: now also C22.1, C23.1, C25.1
- net VBUS: now also C22.2, C23.2
Other:
- title: ${NAME} ${MODEL} -> ${NAME}
- moved on the sheet: LD2, R14
