File: hecate/rp2040.kicad_sch (KiCad schematic)
At the start: 25 parts, among them U2 RP2040, U3 W25Q128JVSIQ, Y1 12 MHz

Commit message: Hecate 3.00
Other:
- title: ${NAME} ${MODEL} -> ${NAME}
Changed lines of the file:
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@@
 	(paper "A4")
 	(title_block
-		(title "${NAME} ${MODEL}")
+		(title "${NAME}")
 		(date "${DATE}")
 		(rev "${VERSION}")
@@
 		(in_pos_files yes)
 		(dnp no)
-		(property "Reference" "#PWR023"
+		(property "Reference" "#PWR022"
 			(at 198.12 97.79 0)
 			(hide yes)
@@
 			(project "hecate"
 				(path "/8c0b3d8b-46d3-4173-ab1e-a61765f77d61/5ac0b842-e6f7-4e44-aa60-2e4205bcbaeb"
-					(reference "#PWR023")
+					(reference "#PWR022")
 					(unit 1)
 				)
@@
 		(dnp no)
 		(fields_autoplaced yes)
-		(property "Reference" "#PWR027"
+		(property "Reference" "#PWR026"
 			(at 242.57 130.81 0)
 			(hide yes)
@@
 			(project "hecate"
 				(path "/8c0b3d8b-46d3-4173-ab1e-a61765f77d61/5ac0b842-e6f7-4e44-aa60-2e4205bcbaeb"
-					(reference "#PWR027")
+					(reference "#PWR026")
 					(unit 1)
 				)
@@
 		(in_pos_files yes)
 		(dnp no)
-		(property "Reference" "#PWR029"
+		(property "Reference" "#PWR028"
 			(at 259.08 69.85 0)
 			(hide yes)
@@
 			(project "hecate"
 				(path "/8c0b3d8b-46d3-4173-ab1e-a61765f77d61/5ac0b842-e6f7-4e44-aa60-2e4205bcbaeb"
-					(reference "#PWR029")
+					(reference "#PWR028")
 					(unit 1)
 				)
@@
 		(in_pos_files yes)
 		(dnp no)
-		(property "Reference" "#PWR026"
+		(property "Reference" "#PWR025"
 			(at 236.22 104.14 0)
 			(hide yes)
@@
 			(project "hecate"
 				(path "/8c0b3d8b-46d3-4173-ab1e-a61765f77d61/5ac0b842-e6f7-4e44-aa60-2e4205bcbaeb"
-					(reference "#PWR026")
+					(reference "#PWR025")
 					(unit 1)
 				)
@@
 		(in_pos_files yes)
 		(dnp no)
-		(property "Reference" "#PWR024"
+		(property "Reference" "#PWR023"
 			(at 200.66 125.73 0)
 			(hide yes)
@@
 			(project "hecate"
 				(path "/8c0b3d8b-46d3-4173-ab1e-a61765f77d61/5ac0b842-e6f7-4e44-aa60-2e4205bcbaeb"
-					(reference "#PWR024")
+					(reference "#PWR023")
 					(unit 1)
 				)
@@
 		(in_pos_files yes)
 		(dnp no)
-		(property "Reference" "#PWR028"
+		(property "Reference" "#PWR027"
 			(at 245.11 76.2 0)
 			(hide yes)
@@
 			(project "hecate"
 				(path "/8c0b3d8b-46d3-4173-ab1e-a61765f77d61/5ac0b842-e6f7-4e44-aa60-2e4205bcbaeb"
-					(reference "#PWR028")
+					(reference "#PWR027")
 					(unit 1)
 				)
@@
 		(in_pos_files yes)
 		(dnp no)
-		(property "Reference" "#PWR025"
+		(property "Reference" "#PWR024"
 			(at 215.9 118.11 0)
 			(hide yes)
@@
 			(project "hecate"
 				(path "/8c0b3d8b-46d3-4173-ab1e-a61765f77d61/5ac0b842-e6f7-4e44-aa60-2e4205bcbaeb"
-					(reference "#PWR025")
+					(reference "#PWR024")
 					(unit 1)
 				)
