File: hecate/usbstack.kicad_sch (KiCad schematic)
At the start: 7 parts

Commit message: Hecate 3.00
Parts:
- renumbered USB1 to U4
Other:
- title: ${NAME} ${MODEL} -> ${NAME}
Changed lines of the file:
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@@
 	(paper "A3")
 	(title_block
-		(title "${NAME} ${MODEL}")
+		(title "${NAME}")
 		(date "${DATE}")
 		(rev "${VERSION}")
@@
 		(dnp no)
 		(fields_autoplaced yes)
-		(property "Reference" "USB1"
+		(property "Reference" "U4"
 			(at 196.85 111.76 0)
 			(show_name no)
@@
 			(project "hecate"
 				(path "/8c0b3d8b-46d3-4173-ab1e-a61765f77d61/0026ee43-61f7-4da2-b06e-4811e7b74caa"
-					(reference "USB1")
+					(reference "U4")
 					(unit 1)
 				)
@@
 		(in_pos_files yes)
 		(dnp no)
-		(property "Reference" "#PWR033"
+		(property "Reference" "#PWR032"
 			(at 210.82 121.92 0)
 			(hide yes)
@@
 			(project "hecate"
 				(path "/8c0b3d8b-46d3-4173-ab1e-a61765f77d61/0026ee43-61f7-4da2-b06e-4811e7b74caa"
-					(reference "#PWR033")
+					(reference "#PWR032")
 					(unit 1)
 				)
@@
 		(in_pos_files yes)
 		(dnp no)
-		(property "Reference" "#PWR035"
+		(property "Reference" "#PWR034"
 			(at 240.03 138.43 0)
 			(hide yes)
@@
 			(project "hecate"
 				(path "/8c0b3d8b-46d3-4173-ab1e-a61765f77d61/0026ee43-61f7-4da2-b06e-4811e7b74caa"
-					(reference "#PWR035")
+					(reference "#PWR034")
 					(unit 1)
 				)
@@
 		(in_pos_files yes)
 		(dnp no)
-		(property "Reference" "#PWR036"
+		(property "Reference" "#PWR035"
 			(at 251.46 138.43 0)
 			(hide yes)
@@
 			(project "hecate"
 				(path "/8c0b3d8b-46d3-4173-ab1e-a61765f77d61/0026ee43-61f7-4da2-b06e-4811e7b74caa"
-					(reference "#PWR036")
+					(reference "#PWR035")
 					(unit 1)
 				)
@@
 		(in_pos_files yes)
 		(dnp no)
-		(property "Reference" "#PWR034"
+		(property "Reference" "#PWR033"
 			(at 217.17 121.92 0)
 			(hide yes)
@@
 			(project "hecate"
 				(path "/8c0b3d8b-46d3-4173-ab1e-a61765f77d61/0026ee43-61f7-4da2-b06e-4811e7b74caa"
-					(reference "#PWR034")
+					(reference "#PWR033")
 					(unit 1)
 				)
@@
 		(dnp no)
 		(fields_autoplaced yes)
-		(property "Reference" "#PWR032"
+		(property "Reference" "#PWR031"
 			(at 196.85 154.94 0)
 			(hide yes)
@@
 			(project "hecate"
 				(path "/8c0b3d8b-46d3-4173-ab1e-a61765f77d61/0026ee43-61f7-4da2-b06e-4811e7b74caa"
-					(reference "#PWR032")
+					(reference "#PWR031")
 					(unit 1)
 				)
