File: easyfrank/pga2350.kicad_sch (KiCad schematic)
At the start: 3 parts, among them U1 Pimoroni PGA2350

Commit message: EasyFRANK WIP
Parts:
- added SW1: Reset, FRANK:SW_PUSH_6mm_H5mm, symbol FRANK:SW_Push
- added SW2: Boot, FRANK:SW_PUSH_6mm_H5mm, symbol FRANK:SW_Push
- renumbered R1 to R5
Connections:
- net BOOTSEL: now also SW2.1
- net GND: now also SW1.2, SW2.2
- net RUN: now also SW1.1
Other:
- moved on the sheet: LD1, R5, U1
