File: easyfrank/tda.kicad_sch (KiCad schematic)
At the start: 7 parts, among them U6 TDA1545A

Commit message: EasyFRANK WIP
Parts:
- renumbered C19 to C22, C20 to C23, R36 to R43, R37 to R44, R38 to R45, R39 to R46, U6 to U7
Changed lines of the file:
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@@
 		(in_pos_files yes)
 		(dnp no)
-		(property "Reference" "#PWR071"
+		(property "Reference" "#PWR087"
 			(at 166.37 81.28 0)
 			(hide yes)
@@
 			(project "easyfrank"
 				(path "/8c0b3d8b-46d3-4173-ab1e-a61765f77d61/c459dc46-a7cf-48ca-8577-a2dbbf1c0ae2/0dccd710-fd54-4e53-9f08-059759dd7a75"
-					(reference "#PWR071")
+					(reference "#PWR087")
 					(unit 1)
 				)
@@
 		(in_pos_files yes)
 		(dnp no)
-		(property "Reference" "R36"
+		(property "Reference" "R43"
 			(at 163.83 81.28 90)
 			(show_name no)
@@
 			(project "easyfrank"
 				(path "/8c0b3d8b-46d3-4173-ab1e-a61765f77d61/c459dc46-a7cf-48ca-8577-a2dbbf1c0ae2/0dccd710-fd54-4e53-9f08-059759dd7a75"
-					(reference "R36")
+					(reference "R43")
 					(unit 1)
 				)
@@
 		(dnp no)
 		(fields_autoplaced yes)
-		(property "Reference" "U6"
+		(property "Reference" "U7"
 			(at 140.97 76.2 0)
 			(show_name no)
@@
 			(project "easyfrank"
 				(path "/8c0b3d8b-46d3-4173-ab1e-a61765f77d61/c459dc46-a7cf-48ca-8577-a2dbbf1c0ae2/0dccd710-fd54-4e53-9f08-059759dd7a75"
-					(reference "U6")
+					(reference "U7")
 					(unit 1)
 				)
@@
 		(in_pos_files yes)
 		(dnp no)
-		(property "Reference" "C20"
+		(property "Reference" "C23"
 			(at 169.418 101.854 90)
 			(show_name no)
@@
 			(project "easyfrank"
 				(path "/8c0b3d8b-46d3-4173-ab1e-a61765f77d61/c459dc46-a7cf-48ca-8577-a2dbbf1c0ae2/0dccd710-fd54-4e53-9f08-059759dd7a75"
-					(reference "C20")
+					(reference "C23")
 					(unit 1)
 				)
@@
 		(in_pos_files yes)
 		(dnp no)
-		(property "Reference" "R39"
+		(property "Reference" "R46"
 			(at 184.15 97.79 90)
 			(show_name no)
@@
 			(project "easyfrank"
 				(path "/8c0b3d8b-46d3-4173-ab1e-a61765f77d61/c459dc46-a7cf-48ca-8577-a2dbbf1c0ae2/0dccd710-fd54-4e53-9f08-059759dd7a75"
-					(reference "R39")
+					(reference "R46")
 					(unit 1)
 				)
@@
 		(in_pos_files yes)
 		(dnp no)
-		(property "Reference" "#PWR075"
+		(property "Reference" "#PWR091"
 			(at 186.69 109.22 0)
 			(hide yes)
@@
 			(project "easyfrank"
 				(path "/8c0b3d8b-46d3-4173-ab1e-a61765f77d61/c459dc46-a7cf-48ca-8577-a2dbbf1c0ae2/0dccd710-fd54-4e53-9f08-059759dd7a75"
-					(reference "#PWR075")
+					(reference "#PWR091")
 					(unit 1)
 				)
@@
 		(dnp no)
 		(fields_autoplaced yes)
-		(property "Reference" "#PWR074"
+		(property "Reference" "#PWR090"
 			(at 186.69 69.85 0)
 			(hide yes)
@@
 			(project "easyfrank"
 				(path "/8c0b3d8b-46d3-4173-ab1e-a61765f77d61/c459dc46-a7cf-48ca-8577-a2dbbf1c0ae2/0dccd710-fd54-4e53-9f08-059759dd7a75"
-					(reference "#PWR074")
+					(reference "#PWR090")
 					(unit 1)
 				)
@@
 		(in_pos_files yes)
 		(dnp no)
-		(property "Reference" "R38"
+		(property "Reference" "R45"
 			(at 184.15 81.28 90)
 			(show_name no)
@@
 			(project "easyfrank"
 				(path "/8c0b3d8b-46d3-4173-ab1e-a61765f77d61/c459dc46-a7cf-48ca-8577-a2dbbf1c0ae2/0dccd710-fd54-4e53-9f08-059759dd7a75"
-					(reference "R38")
+					(reference "R45")
 					(unit 1)
 				)
@@
 		(in_pos_files yes)
 		(dnp no)
-		(property "Reference" "#PWR069"
+		(property "Reference" "#PWR084"
 			(at 115.57 93.98 0)
 			(hide yes)
@@
 			(project "easyfrank"
 				(path "/8c0b3d8b-46d3-4173-ab1e-a61765f77d61/c459dc46-a7cf-48ca-8577-a2dbbf1c0ae2/0dccd710-fd54-4e53-9f08-059759dd7a75"
-					(reference "#PWR069")
+					(reference "#PWR084")
 					(unit 1)
 				)
@@
 		(in_pos_files yes)
 		(dnp no)
-		(property "Reference" "#PWR072"
+		(property "Reference" "#PWR088"
 			(at 166.37 111.76 0)
 			(hide yes)
@@
 			(project "easyfrank"
 				(path "/8c0b3d8b-46d3-4173-ab1e-a61765f77d61/c459dc46-a7cf-48ca-8577-a2dbbf1c0ae2/0dccd710-fd54-4e53-9f08-059759dd7a75"
-					(reference "#PWR072")
+					(reference "#PWR088")
 					(unit 1)
 				)
@@
 		(in_pos_files yes)
 		(dnp no)
-		(property "Reference" "#PWR073"
+		(property "Reference" "#PWR089"
 			(at 176.53 96.52 0)
 			(hide yes)
@@
 			(project "easyfrank"
 				(path "/8c0b3d8b-46d3-4173-ab1e-a61765f77d61/c459dc46-a7cf-48ca-8577-a2dbbf1c0ae2/0dccd710-fd54-4e53-9f08-059759dd7a75"
-					(reference "#PWR073")
+					(reference "#PWR089")
 					(unit 1)
 				)
@@
 		(in_pos_files yes)
 		(dnp no)
-		(property "Reference" "#PWR070"
+		(property "Reference" "#PWR086"
 			(at 157.48 111.76 0)
 			(hide yes)
@@
 			(project "easyfrank"
 				(path "/8c0b3d8b-46d3-4173-ab1e-a61765f77d61/c459dc46-a7cf-48ca-8577-a2dbbf1c0ae2/0dccd710-fd54-4e53-9f08-059759dd7a75"
-					(reference "#PWR070")
+					(reference "#PWR086")
 					(unit 1)
 				)
@@
 		(in_pos_files yes)
 		(dnp no)
-		(property "Reference" "R37"
+		(property "Reference" "R44"
 			(at 173.99 97.79 90)
 			(show_name no)
@@
 			(project "easyfrank"
 				(path "/8c0b3d8b-46d3-4173-ab1e-a61765f77d61/c459dc46-a7cf-48ca-8577-a2dbbf1c0ae2/0dccd710-fd54-4e53-9f08-059759dd7a75"
-					(reference "R37")
+					(reference "R44")
 					(unit 1)
 				)
@@
 		(in_pos_files yes)
 		(dnp no)
-		(property "Reference" "C19"
+		(property "Reference" "C22"
 			(at 160.528 101.854 90)
 			(show_name no)
@@
 			(project "easyfrank"
 				(path "/8c0b3d8b-46d3-4173-ab1e-a61765f77d61/c459dc46-a7cf-48ca-8577-a2dbbf1c0ae2/0dccd710-fd54-4e53-9f08-059759dd7a75"
-					(reference "C19")
+					(reference "C22")
 					(unit 1)
 				)

Commit message: EasyFRANK WIP
Parts:
- renumbered R43 to R44, R44 to R45, R45 to R46, R46 to R47
Changed lines of the file:
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@@
 		(in_pos_files yes)
 		(dnp no)
-		(property "Reference" "#PWR087"
+		(property "Reference" "#PWR089"
 			(at 166.37 81.28 0)
 			(hide yes)
@@
 			(project "easyfrank"
 				(path "/8c0b3d8b-46d3-4173-ab1e-a61765f77d61/c459dc46-a7cf-48ca-8577-a2dbbf1c0ae2/0dccd710-fd54-4e53-9f08-059759dd7a75"
-					(reference "#PWR087")
+					(reference "#PWR089")
 					(unit 1)
 				)
@@
 		(in_pos_files yes)
 		(dnp no)
-		(property "Reference" "R43"
+		(property "Reference" "R44"
 			(at 163.83 81.28 90)
 			(show_name no)
@@
 			(project "easyfrank"
 				(path "/8c0b3d8b-46d3-4173-ab1e-a61765f77d61/c459dc46-a7cf-48ca-8577-a2dbbf1c0ae2/0dccd710-fd54-4e53-9f08-059759dd7a75"
-					(reference "R43")
+					(reference "R44")
 					(unit 1)
 				)
@@
 		(in_pos_files yes)
 		(dnp no)
-		(property "Reference" "R46"
+		(property "Reference" "R47"
 			(at 184.15 97.79 90)
 			(show_name no)
@@
 			(project "easyfrank"
 				(path "/8c0b3d8b-46d3-4173-ab1e-a61765f77d61/c459dc46-a7cf-48ca-8577-a2dbbf1c0ae2/0dccd710-fd54-4e53-9f08-059759dd7a75"
-					(reference "R46")
+					(reference "R47")
 					(unit 1)
 				)
@@
 		(in_pos_files yes)
 		(dnp no)
-		(property "Reference" "#PWR091"
+		(property "Reference" "#PWR093"
 			(at 186.69 109.22 0)
 			(hide yes)
@@
 			(project "easyfrank"
 				(path "/8c0b3d8b-46d3-4173-ab1e-a61765f77d61/c459dc46-a7cf-48ca-8577-a2dbbf1c0ae2/0dccd710-fd54-4e53-9f08-059759dd7a75"
-					(reference "#PWR091")
+					(reference "#PWR093")
 					(unit 1)
 				)
@@
 		(dnp no)
 		(fields_autoplaced yes)
-		(property "Reference" "#PWR090"
+		(property "Reference" "#PWR092"
 			(at 186.69 69.85 0)
 			(hide yes)
@@
 			(project "easyfrank"
 				(path "/8c0b3d8b-46d3-4173-ab1e-a61765f77d61/c459dc46-a7cf-48ca-8577-a2dbbf1c0ae2/0dccd710-fd54-4e53-9f08-059759dd7a75"
-					(reference "#PWR090")
+					(reference "#PWR092")
 					(unit 1)
 				)
@@
 		(in_pos_files yes)
 		(dnp no)
-		(property "Reference" "R45"
+		(property "Reference" "R46"
 			(at 184.15 81.28 90)
 			(show_name no)
@@
 			(project "easyfrank"
 				(path "/8c0b3d8b-46d3-4173-ab1e-a61765f77d61/c459dc46-a7cf-48ca-8577-a2dbbf1c0ae2/0dccd710-fd54-4e53-9f08-059759dd7a75"
-					(reference "R45")
+					(reference "R46")
 					(unit 1)
 				)
@@
 		(in_pos_files yes)
 		(dnp no)
-		(property "Reference" "#PWR084"
+		(property "Reference" "#PWR086"
 			(at 115.57 93.98 0)
 			(hide yes)
@@
 			(project "easyfrank"
 				(path "/8c0b3d8b-46d3-4173-ab1e-a61765f77d61/c459dc46-a7cf-48ca-8577-a2dbbf1c0ae2/0dccd710-fd54-4e53-9f08-059759dd7a75"
-					(reference "#PWR084")
+					(reference "#PWR086")
 					(unit 1)
 				)
@@
 		(in_pos_files yes)
 		(dnp no)
-		(property "Reference" "#PWR088"
+		(property "Reference" "#PWR090"
 			(at 166.37 111.76 0)
 			(hide yes)
@@
 			(project "easyfrank"
 				(path "/8c0b3d8b-46d3-4173-ab1e-a61765f77d61/c459dc46-a7cf-48ca-8577-a2dbbf1c0ae2/0dccd710-fd54-4e53-9f08-059759dd7a75"
-					(reference "#PWR088")
+					(reference "#PWR090")
 					(unit 1)
 				)
@@
 		(in_pos_files yes)
 		(dnp no)
-		(property "Reference" "#PWR089"
+		(property "Reference" "#PWR091"
 			(at 176.53 96.52 0)
 			(hide yes)
@@
 			(project "easyfrank"
 				(path "/8c0b3d8b-46d3-4173-ab1e-a61765f77d61/c459dc46-a7cf-48ca-8577-a2dbbf1c0ae2/0dccd710-fd54-4e53-9f08-059759dd7a75"
-					(reference "#PWR089")
+					(reference "#PWR091")
 					(unit 1)
 				)
@@
 		(in_pos_files yes)
 		(dnp no)
-		(property "Reference" "#PWR086"
+		(property "Reference" "#PWR088"
 			(at 157.48 111.76 0)
 			(hide yes)
@@
 			(project "easyfrank"
 				(path "/8c0b3d8b-46d3-4173-ab1e-a61765f77d61/c459dc46-a7cf-48ca-8577-a2dbbf1c0ae2/0dccd710-fd54-4e53-9f08-059759dd7a75"
-					(reference "#PWR086")
+					(reference "#PWR088")
 					(unit 1)
 				)
@@
 		(in_pos_files yes)
 		(dnp no)
-		(property "Reference" "R44"
+		(property "Reference" "R45"
 			(at 173.99 97.79 90)
 			(show_name no)
@@
 			(project "easyfrank"
 				(path "/8c0b3d8b-46d3-4173-ab1e-a61765f77d61/c459dc46-a7cf-48ca-8577-a2dbbf1c0ae2/0dccd710-fd54-4e53-9f08-059759dd7a75"
-					(reference "R44")
+					(reference "R45")
 					(unit 1)
 				)

Commit message: EasyFRANK WIP
Parts:
- added C23: 10u, FRANK:Combined_0805_CR, symbol FRANK:C_Small
- added C24, C25: 100u, FRANK:C_Radial_D6.3mm_P2.50mm, symbol FRANK:C_Polarized_Small
- added R37: 51K, FRANK:Combined_0805_RE, symbol FRANK:R_Small
- added R39, R42: 100R, FRANK:Combined_0805_RE, symbol FRANK:R_Small
- R40: renamed from R45; value 1.5K -> 10K
- renumbered C22 to C21, C23 to C22, R44 to R36, R47 to R38, R46 to R41
Connections:
- net GND: now also R40.1, C23.1, C24.2, C25.2; no longer R38.1, R41.2
- net VBUS: now also R37.1; no longer R40.1
- net at R40.2, U7.7 (IREF): now also C23.2, R37.2
- new net: C24.1, R41.2, R42.2
- new net: C25.1, R38.1, R39.2
- new net +3V3: R39.1, R42.1
Other:
- moved on the sheet: C21, C22, R36, R38, R40, R41, U7
