File: frank_next/frank_next.kicad_pcb (KiCad board)
At the start: 4 copper layers, 174 parts, among them J1 Debug, J10 USB4215-03-A, J11 USB4215-03-A, J12 BAT 3V, J13 PJ-320D, J2 UART, J3 DC3RX19JA2, J4 104031-0811, J5 PJ-320D, J6 Speaker, J7 NES Gamepad 1/2, J8 676430910, J9 676430910, Q1 UMH3N, U1 W25Q128JVPIQ, U10 TPD4S012DRYR, U11 TPD4S012DRYR, U12 TPD4S012DRYR, U13 TPS2116DRL, U14 TS3USB221RSER, U15 AMS1117-3.3, U16 CH334F, U17 CH343P, U18 74HC4052BQ,115, U19 DS3231MZ, U2 ESP-PSRAM64, U20 DS2401P+, U21 CD4069UBM, U3 RP2350B, U4 TLV320DAC3100IRHBR, U5 XC6206P182MR-G, U6 ESP32-D0WD-V3, U7 W25Q32JVSIQ, U9 TPD4S012DRYR, Y1 ASE-12MHz, Y2 40MHz, Y3 12MHz

Commit message: Board Updates
Parts:
- removed R25: 1K, FRANK:R_0603_1608Metric
- removed the R9 at (185.9, 113.6)
- added C75: 100n, FRANK:C_0603_1608Metric, B.Cu at (133.7, 111.5)
- added C76: 100n, FRANK:C_0603_1608Metric, B.Cu at (141.8, 113.5)
- added H1: MountingHole, FRANK:MountingHole_2.5mm_Pad_Via, F.Cu at (131.8, 70.6)
- added H2: MountingHole, FRANK:MountingHole_2.5mm_Pad_Via, F.Cu at (206.8, 70.6)
- added H3: MountingHole, FRANK:MountingHole_2.5mm_Pad_Via, F.Cu at (206.8, 119.0)
- added H4: MountingHole, FRANK:MountingHole_2.5mm_Pad_Via, F.Cu at (131.8, 119.0)
- added LD3: Green, FRANK:LED_0603_1608Metric, F.Cu at (190.5, 119.1)
- added LD4: Orange, FRANK:LED_0603_1608Metric, F.Cu at (153.5, 112.9)
- added R1: 220R, FRANK:R_0603_1608Metric, B.Cu at (149.2, 111.1)
- added R24: 20K, FRANK:R_0603_1608Metric, B.Cu at (141.7, 97.3)
- C16, C20, C21, C22, C23, C24, C25, C26, C27, C28, C29, C30, C31, C32, C33, C34, C35, C36, C37, C38, C39, C40, C41, C42, C43, C44, C46, C48, C49, C50, C51, C53, C54, C55, C56, C57, C58, C59, C60, C62, C63, C64, C65, C67, C70, C71, C72, C73, C74, D1, D2, D3, D4, F1, JP1, JP2, L2, L4, L5, Q1, R10, R11, R12, R13, R15, R21, R26, R28, R29, R30, R38, R39, R40, R41, U10, U11, U12, U14, U15, U19, U20, U21, U5, U9, Y2, Y3: moved to B.Cu
- C68, C69: value 100n -> 12p; moved to B.Cu
- LD1: value WS2812B-2020 -> Blue; footprint FRANK:LED_WS2812B-2020_PLCC4_2.0x2.0mm -> FRANK:LED_0603_1608Metric
- LD2: value Green -> WS2812B-2020; footprint FRANK:LED_0603_1608Metric -> FRANK:LED_WS2812B-2020_PLCC4_2.0x2.0mm
- R14, R37: value 4.7K -> 10K; moved to B.Cu
- R16: value 10K -> 4.7K; moved to B.Cu
- R17: value 499R -> 10K; moved to B.Cu
- R18: value 0R -> 499R; moved to B.Cu
- R19: value 10K -> 0R; moved to B.Cu
- R20: value 330R -> 10K; moved to B.Cu
- R22: value 10K -> 330R; moved to B.Cu
- R23: value 20K -> 10K; moved to B.Cu
- R27: value 5.1K -> 1K; moved to B.Cu
- R31: value 300K -> 5.1K; moved to B.Cu
- R32: value 100K -> 300K; moved to B.Cu
- R33: value 10K -> 100K; moved to B.Cu
- R34: value 1K -> 10K; moved to B.Cu
- R35: value 10K -> 1K; moved to B.Cu
- R36: value 4.7K -> 1K; moved to B.Cu
- moved R4 99.9 mm to (198.9, 98.7)
- moved L1 99.9 mm to (200.6, 96.3)
- moved C12 99.4 mm to (186.4, 89.1)
- moved C18 99.4 mm to (193.8, 90.1)
- moved R2 99.4 mm to (204.8, 81.0)
- moved R6 99.4 mm to (204.4, 83.8)
- moved R7 99.4 mm to (197.8, 91.5)
- moved R8 99.4 mm to (197.8, 93.1)
- moved C1 99.4 mm to (204.4, 87.0)
- moved C10 99.4 mm to (192.0, 88.6)
- moved C11 99.4 mm to (188.0, 88.3)
- moved C13 99.4 mm to (186.5, 93.9)
- moved C14 99.4 mm to (184.0, 96.2)
- moved C15 99.4 mm to (188.2, 93.9)
- moved C17 99.4 mm to (192.0, 93.5)
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- renumbered R1 to R2, R2 to R3, R3 to R4, R4 to R5, R5 to R6, R6 to R7, R7 to R8, R8 to R9
Connections:
- C53 pad 1: Net-(J8-VBUS) -> GND
- C53 pad 2: Net-(C53-Pad2) -> Net-(J8-VBUS)
- C54 pad 1: Net-(J9-VBUS) -> Net-(J8-VBUS)
- C54 pad 2: Net-(C53-Pad2) -> GND
- C63 pad 2: Net-(U16-VDD33_{LDO}) -> /USB/VDD33
- C64 pad 2: Net-(U16-VDD33_{LDO}) -> /USB/VDD33
- C68 pad 1: GND -> /USB/XTAL_N
- C68 pad 2: VBUS -> GND
- C69 pad 1: GND -> /USB/XTAL_P
- C69 pad 2: Net-(U17-V3_{OUT}) -> GND
- C70 pad 2: +3V3 -> VBUS
- C71 pad 2: +3V3 -> Net-(U17-V3_{OUT})
- C72 pad 1: +3V3 -> GND
- C72 pad 2: GND -> +3V3
- C73 pad 1: Net-(C73-Pad1) -> GND
- C73 pad 2: /Tape In/TAPE -> +3V3
- F1 pad 1: Net-(C53-Pad2) -> Net-(J8-VBUS)
- J9 pad 1: Net-(J9-VBUS) -> Net-(J8-VBUS)
- LD1 pad 1: unconnected-(LD1-DOUT-Pad1) -> GND
- LD1 pad 2: GND -> Net-(LD1-A)
- LD2 pad 1: GND -> unconnected-(LD2-DOUT-Pad1)
- LD2 pad 2: Net-(LD2-A) -> GND
- R10 pad 2: /GPIO7/DAT3 -> /GPIO6/DAT2
- R11 pad 2: /GPIO3/CMD -> /GPIO7/DAT3
- R12 pad 2: /GPIO4/DAT0 -> /GPIO3/CMD
- R13 pad 2: /GPIO5/DAT1 -> /GPIO4/DAT0
- R14 pad 1: /GPIO29/SCL -> +3V3
- R14 pad 2: +3V3 -> /GPIO5/DAT1
- R15 pad 1: /GPIO28/SDA -> /GPIO29/SCL
- R16 pad 1: Net-(U4-~{RESET}) -> /GPIO28/SDA
- R17 pad 1: Net-(U6-U0TXD) -> Net-(U4-~{RESET})
- R17 pad 2: /ESP32/U0TXD -> +3V3
- R18 pad 1: Net-(U6-GPIO16) -> Net-(U6-U0TXD)
- R18 pad 2: /ESP32/GPIO16 -> /ESP32/U0TXD
- R19 pad 1: /GPIO38/CHIP_PU -> Net-(U6-GPIO16)
- R19 pad 2: +3V3 -> /ESP32/GPIO16
- R20 pad 1: /ESP Multiplexer/2Z -> /GPIO38/CHIP_PU
- R20 pad 2: /ESP32/U0RXD -> +3V3
- R21 pad 1: /ESP Multiplexer/1Z -> /ESP Multiplexer/2Z
- R21 pad 2: /ESP32/U0TXD -> /ESP32/U0RXD
- R22 pad 1: /GPIO39/GPIO0 -> /ESP Multiplexer/1Z
- R22 pad 2: +3V3 -> /ESP32/U0TXD
- R23 pad 1: /ESP32/CAP2 -> /GPIO39/GPIO0
- R23 pad 2: /ESP32/CAP1 -> +3V3
- R26 pad 1: /GPIO26 -> /GPIO27
- R26 pad 2: /NES Gamepad/G_DATA1 -> /NES Gamepad/G_DATA2
- R27 pad 1: GND -> /GPIO26
- R27 pad 2: Net-(J10-CC1) -> /NES Gamepad/G_DATA1
- R28 pad 2: Net-(J10-CC2) -> Net-(J10-CC1)
- R29 pad 2: Net-(J11-CC1) -> Net-(J10-CC2)
- R30 pad 2: Net-(J11-CC2) -> Net-(J11-CC1)
- R31 pad 1: Net-(U13-PR1) -> GND
- R31 pad 2: /USB/VBUS_IN1 -> Net-(J11-CC2)
- R32 pad 1: GND -> Net-(U13-PR1)
- R32 pad 2: Net-(U13-PR1) -> /USB/VBUS_IN1
- R33 pad 2: /USB/S -> Net-(U13-PR1)
- R34 pad 1: Net-(LD2-A) -> GND
- R34 pad 2: +3V3 -> /USB/S
- R35 pad 1: /GPIO30/S0 -> Net-(LD3-A)
- R35 pad 2: GND -> +3V3
- R36 pad 1: /GPIO29/SCL -> Net-(LD4-A)
- R37 pad 1: /GPIO28/SDA -> /GPIO30/S0
- R37 pad 2: +3V3 -> GND
- R39 pad 2: Net-(C73-Pad1) -> Net-(C75-Pad1)
- R9 pad 1: Net-(LD1-DIN) -> Net-(LD2-DIN)
- U16 pad 1: unconnected-(U16-~{OVCUR}-Pad1) -> /USB/VDD33
- U16 pad 20: Net-(U16-VDD33_{LDO}) -> /USB/VDD33
- U17 pad 10: unconnected-(U17-~{ACT}-Pad10) -> Net-(LD4-K)
Routing:
- net VBUS: track 0.00 -> 220.8 mm, vias 0 -> 16
- net /GPIO0/RXD: track 8.05 -> 98.4 mm
- net /GPIO38/CHIP_PU: track 0.00 -> 89.2 mm, vias 0 -> 7
- net /GPIO39/GPIO0: track 0.00 -> 83.9 mm, vias 0 -> 5
- net /GPIO22/LOAD_IN: track 0.00 -> 81.5 mm, vias 0 -> 5
- net /GPIO1/TXD: track 5.96 -> 87.2 mm
- net /GPIO27: track 0.00 -> 75.0 mm, vias 0 -> 1
- net /READY (GPIO37/GPIO4): track 0.00 -> 67.6 mm, vias 0 -> 4
- net /HS (GPIO36/GPIO2): track 0.00 -> 66.9 mm, vias 0 -> 2
- net /GPIO26: track 0.00 -> 65.4 mm, vias 0 -> 1
- net /GPIO9/BCLK: track 0.00 -> 57.0 mm, vias 0 -> 2
- net /GPIO5/DAT1: track 2.75 -> 59.0 mm, vias 0 -> 1
- net /GPIO10/WCLK: track 0.00 -> 55.6 mm, vias 0 -> 2
- net /GPIO20: track 0.00 -> 54.7 mm
- net /GPIO4/DAT0: track 2.65 -> 56.9 mm, vias 0 -> 1
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- added copper zone on In2.Cu, net +3V3
- added copper zone on B.Cu, net GND
- added copper zone on F.Cu, net GND
- added copper zone on In1.Cu, net GND
Other:
- board outline added: 80.6 x 54 mm
- board text added: "FRANK"
- board text added: "HW ${VERSION} Designed by Mikhail Matveev https://frank.rh1.tech"
- board text added: "NEXT"

Commit message: FRANK Next WIP
Parts:
- removed the LD1 at (149.2, 111.1)
- removed the R1 at (149.2, 111.1)
- added LD2: Blue, FRANK:LED_0603_1608Metric, B.Cu at (149.4, 110.9)
- added R21: 220R, FRANK:R_0603_1608Metric, F.Cu at (149.4, 110.9)
- AE1: value Antenna_Shield -> Antenna
- BT1: value Battery_CR1220 -> CR1220
- C1, C10, C11, C12, C13, C14, C15, C16, C17, C18, C19, C2, C20, C21, C22, C23, C27, C3, C30, C31, C35, C37, C38, C40, C42, C51, C55, C56, C59, C6, C60, C62, C67, C70, C71, C72, C73, C74, C75, C76, C9: value 100n -> 100nF
- C24, C25: value 100u -> 100uF
- C26, C28, C29, C39, C53, C54, C57, C58, C63, C65: value 10u -> 10uF
- C32, C33, C34, C41, C64: value 1u -> 1uF
- C36: value 100p -> 100pF
- C43, C44: value 1n -> 1nF
- C46: value 10n -> 10nF
- C48: value 3.3n -> 3.3nF
- C49, C50, C68, C69: value 12p -> 12pF
- C61, C66: value 22u -> 22uF
- L1: value 3.3u -> 3.3uF
- U18: value 74HC4052BQ,115 -> 74HC4052BQ
- U2: value ESP-PSRAM64 -> ESP-PSRAM64H
- renumbered LD2 to LD1, R2 to R1, R11 to R10, R12 to R11, R13 to R12, R14 to R13, R15 to R14, R16 to R15, R17 to R16, R18 to R17, R19 to R18, R20 to R19, R3 to R2, R21 to R20, R4 to R3, R5 to R4, R6 to R5, R7 to R6, R8 to R7, R9 to R8, R10 to R9
Connections:
- net Net-(J2-Pin_1) renamed /RP2350B/GPIO40/UART_1
- net Net-(J2-Pin_3) renamed /RP2350B/GPIO41/UART_3
Routing:
- net /ESP32/GPIO16: track 3.08 -> 4.09 mm, vias 0 -> 1
- net +3V3: track 69.7 -> 68.9 mm
- net Net-(U4-HPL): track 25.5 -> 26.0 mm
- net Net-(LD2-A): vias 0 -> 1
- net Net-(LD1-A): vias 1 -> 0
Other:
- outline, holes or cut-outs redrawn
- board text added: "AUDIO OUT"
- board text added: "ESP FLSH"
- board text added: "ESP RST"
- board text added: "NES GAMEPAD 1/2"
- board text added: "POWER"
- board text added: "RP BOOT"
- board text added: "RP RST"
- board text added: "SPEAKER"
- board text added: "TAPE IN"
- board text added: "UART"
- board text added: "USB HUB"

Commit message: Board updates
Parts:
- L1: value 3.3uF -> 3.3µH
- L2, L3, L4: footprint FRANK:Inductor_0603_1608Metric_HandSolder -> FRANK:L_0603_1608Metric_HandSolder
- S6: footprint FRANK:SK12D07VG3NS_PWR -> FRANK:Switch_Slide_SK12D07VG3NS_PWR
- U1: footprint FRANK:SON127P600X500X80-9N-D -> FRANK:WSON-8-1EP_6x5mm_P1.27mm_EP3.45x4.35mm
- U19: footprint FRANK:SO-8 -> FRANK:SO-8_3.9x4.9mm_P1.27mm
- U21: footprint FRANK:SOIC127P600X175-14N -> FRANK:SOIC-14_3.9x8.7mm_P1.27mm
- U6: footprint FRANK:QFN35P500X500X90-49N-D -> FRANK:QFN-48-1EP_5x5mm_P0.35mm_EP3.75x3.75mm
- Y1: footprint FRANK:Oscillator_SMD_3225_4Pin -> FRANK:Oscillator_SMD_3225-4Pin_3.2x2.5mm

Commit message: Bugfixes
Parts:
- removed J12: BAT 3V, FRANK:PinHeader_1x02_P2.54mm_Vertical
- LD2: moved to F.Cu
- R21: moved to B.Cu
- moved C53 7.60 mm to (166.5, 70.1)
- moved C54 7.60 mm to (148.3, 70.0)
- moved LD2 0.05 mm to (149.4, 110.9), turned to 0 degrees
- moved R21 0.05 mm to (149.4, 110.9), turned to 180 degrees
- turned U9 to -90 degrees
Connections:
- J4 pad SH: GND -> unconnected-(J4-SHIELD-PadSH)_1
Routing:
- net /USB/DS1+: track 34.6 -> 31.2 mm
- net /USB/DS2+: track 16.3 -> 13.1 mm, vias 0 -> 1
- net /USB/DS1-: track 27.7 -> 30.7 mm
- net Net-(J8-VBUS): track 21.4 -> 23.8 mm
- net Net-(BT1-+): track 18.5 -> 19.6 mm, vias 0 -> 1
- net /USB/DS2-: track 10.5 -> 9.39 mm
- net Net-(U4-HPL): track 26.0 -> 26.9 mm
- net /ESP32/GPIO16: track 4.09 -> 3.44 mm, vias 1 -> 0
- net GND: vias 67 -> 66
Other:
- outline, holes or cut-outs redrawn
- board text added: "ESP32"
- board text added: "RP2350B"
- board text added: "SPK"
- board text removed: "SPEAKER"
