File: frank_next/usb.kicad_sch (KiCad schematic)
At the start: 44 parts, among them J10 USB4215-03-A, J11 USB4215-03-A, J8 676430910, J9 676430910, U10 TPD4S012DRYR, U11 TPD4S012DRYR, U12 TPD4S012DRYR, U13 TPS2116DRL, U14 TS3USB221RSER, U15 AMS1117-3.3, U16 CH334F, U9 TPD4S012DRYR, Y3 12MHz

Commit message: Board updates
Connections:
- net GND: now also C53.2, C54.1
- net at C53.1, J8.1 (VBUS): now also C54.2, F1.1, J9.1 (VBUS)

Commit message: Board Updates
Parts:
- renumbered C54 to C53, C53 to C54, C75 to C68, C76 to C69, LD2 to LD3, R27 to R28, R28 to R29, R29 to R30, R30 to R31, R31 to R32, R32 to R33, R33 to R34, R34 to R35

Commit message: FRANK Next WIP
Parts:
- C53, C54, C57, C58, C63, C65: value 10u -> 10uF
- C55, C56, C59, C60, C62, C67: value 100n -> 100nF
- C61, C66: value 22u -> 22uF
- C64: value 1u -> 1uF
- C68, C69: value 12p -> 12pF
Changed lines of the file:
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@@
 		(rev "${VERSION}")
 		(company "Mikhail Matveev")
-		(comment 1 "https://github.com/rh1tech/frank_next")
+		(comment 1 "https://github.com/rh1tech/frank")
 	)
 	(junction
@@
 			)
 		)
-		(property "Value" "1u"
+		(property "Value" "1uF"
 			(at 220.853 60.579 0)
 			(show_name no)
@@
 			)
 		)
-		(property "Value" "22u"
+		(property "Value" "22uF"
 			(at 244.094 33.274 0)
 			(show_name no)
@@
 			)
 		)
-		(property "Value" "100n"
+		(property "Value" "100nF"
 			(at 136.271 110.617 0)
 			(show_name no)
@@
 			)
 		)
-		(property "Value" "10u"
+		(property "Value" "10uF"
 			(at 43.561 162.433 0)
 			(show_name no)
@@
 			)
 		)
-		(property "Value" "10u"
+		(property "Value" "10uF"
 			(at 146.431 73.533 0)
 			(show_name no)
@@
 			)
 		)
-		(property "Value" "100n"
+		(property "Value" "100nF"
 			(at 136.271 73.533 0)
 			(show_name no)
@@
 			)
 		)
-		(property "Value" "100n"
+		(property "Value" "100nF"
 			(at 220.726 38.1 0)
 			(show_name no)
@@
 			)
 		)
-		(property "Value" "12p"
+		(property "Value" "12pF"
 			(at 253.873 132.969 0)
 			(show_name no)
@@
 			)
 		)
-		(property "Value" "10u"
+		(property "Value" "10uF"
 			(at 146.431 110.617 0)
 			(show_name no)
@@
 			)
 		)
-		(property "Value" "100n"
+		(property "Value" "100nF"
 			(at 249.936 38.1 0)
 			(show_name no)
@@
 			)
 		)
-		(property "Value" "10u"
+		(property "Value" "10uF"
 			(at 237.617 60.579 0)
 			(show_name no)
@@
 			)
 		)
-		(property "Value" "22u"
+		(property "Value" "22uF"
 			(at 211.074 37.592 0)
 			(show_name no)
@@
 			)
 		)
-		(property "Value" "10u"
+		(property "Value" "10uF"
 			(at 42.799 127.127 0)
 			(show_name no)
@@
 			)
 		)
-		(property "Value" "12p"
+		(property "Value" "12pF"
 			(at 254.0254 157.48 0)
 			(show_name no)
@@
 			)
 		)
-		(property "Value" "10u"
+		(property "Value" "10uF"
 			(at 220.853 50.419 0)
 			(show_name no)
@@
 			)
 		)
-		(property "Value" "100n"
+		(property "Value" "100nF"
 			(at 167.64 28.194 90)
 			(show_name no)
@@
 			)
 		)
-		(property "Value" "100n"
+		(property "Value" "100nF"
 			(at 184.023 96.139 0)
 			(show_name no)

Commit message: Board updates
Parts:
- S6: footprint FRANK:SK12D07VG3NS_PWR -> FRANK:Switch_Slide_SK12D07VG3NS_PWR
Changed lines of the file:
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@@
 			)
 		)
-		(property "Footprint" "FRANK:SK12D07VG3NS_PWR"
+		(property "Footprint" "FRANK:Switch_Slide_SK12D07VG3NS_PWR"
 			(at 134.62 -55.55 0)
 			(hide yes)

Commit message: FRANK Next updates
Parts:
- removed C53: 10uF, FRANK:C_0603_1608Metric, symbol FRANK:C
- removed C61, C66: 22uF, FRANK:CP_Tantalum_3528-12, symbol FRANK:C_Polarized_Small
- removed C62, C67: 100nF, FRANK:C_0603_1608Metric, symbol FRANK:C_Small
- removed F1: 1.5A / 6V, FRANK:Fuse_1206_3216Metric, symbol FRANK:Polyfuse
- removed J9: 676430910, FRANK:USB_A_Short, symbol FRANK:USB_A
- removed U10: TPD4S012DRYR, FRANK:TPD4S012DRYR, symbol FRANK:TPD4S012DRYR
- removed U15: AMS1117-3.3, FRANK:SOT-89-3, symbol FRANK:AMS1117-3.3
- added C56: 100n, FRANK:C_0603_1608Metric, symbol FRANK:C
- added C58, C59, C62, C63, C69, C70, C73: 10uF, FRANK:C_0603_1608Metric, symbol FRANK:C
- added C67: 100nF, FRANK:C_0603_1608Metric, symbol FRANK:C
- added C77: 22pF, FRANK:C_0603_1608Metric, symbol FRANK:C
- added J8: 676430910, FRANK:USB_A_Short, symbol FRANK:USB_A
- added L6: 2.2uH, Inductor_SMD:L_Cenker_CKCS3015, symbol FRANK:L
- added R34: 1M, FRANK:R_0603_1608Metric, symbol FRANK:R
- added R35, R36: 100K, FRANK:R_0603_1608Metric, symbol Device:R_Small
- added R38, R42: 100K, FRANK:R_0603_1608Metric, symbol FRANK:R
- added R40: 1K, FRANK:R_0603_1608Metric, symbol FRANK:R
- added R41: 4.7K, FRANK:R_0603_1608Metric, symbol Device:R_Small
- added R43: 22K, FRANK:R_0603_1608Metric, symbol FRANK:R
- added U13, U14: CH217K, Package_TO_SOT_SMD:SOT-23-6, symbol FRANK:CH217K
- added U16: AO3401A, FRANK:SOT-23-3L_AOS, symbol FRANK:AO3401A
- added U18: SY8089AAAC, Package_TO_SOT_SMD:SOT-23-5, symbol FRANK:SY8089AAAC
- added U9: TPD4S012DRYR, FRANK:TPD4S012DRYR, symbol FRANK:TPD4S012DRYR
- C57: renamed from C54; value 10uF -> 100n
- C66: renamed from C59; value 100nF -> 10u
- L5: value 330R -> 330R 2A; footprint FRANK:L_0603_1608Metric -> Inductor_SMD:L_0805_2012Metric
- Y3: footprint FRANK:Crystal_SMD_2520-4Pin_2.5x2.0mm -> FRANK:Crystal_SMD_3225-4Pin_3.2x2.5mm
- renumbered C55 to C60, C56 to C61, C57 to C64, C58 to C65, C60 to C68, C63 to C71, C64 to C72, C65 to C74, C68 to C75, C69 to C76, J8 to J9, R35 to R37, R34 to R39, U9 to U10, U13 to U15, U14 to U17, U16 to U19
Connections:
- net +3V3: now also C73.1, C77.1, L6.1, R42.1
- net DS1+: now also J8.3 (D+), U9.1 (D+); no longer J9.3 (D+), U10.1 (D+)
- net DS1-: now also J8.2 (D-), U9.2 (D-_); no longer J9.2 (D-), U10.2 (D-_)
- net DS2+: now also J9.3 (D+), U10.1 (D+)
- net DS2-: now also J9.2 (D-), U10.2 (D-_)
- net GND: now also S6.2, C56.2, C58.2, C59.2, C62.1, C63.1, C69.2, C70.2, C73.2, J8.4 (GND), J8.5 (Shield), R35.1, R36.1, R41.2, R43.2, U13.2 (GND), U14.2 (GND), U18.2 (GND), U9.4 (GND)
- net VBUS: now also L5.2, C62.2, C63.2, C69.1, C70.1, U13.6 (VIN), U14.6 (VIN), U18.1 (EN), U18.4 (IN); no longer L5.1, U10.6 (VBUS), U11.6 (VBUS), U12.6 (VBUS)
- net VBUS_IN: now also C66.1, C67.2, R38.2, U16.2 (S); no longer S6.2
- net VBUS_IN1: now also U12.6 (VBUS)
- net VBUS_IN2: now also U11.6 (VBUS)
- net VDD33: no longer U19.1 (~{OVCUR})
- net at S6.3: now also R40.2
- net at R32.1, R33.2, U15.4 (PR1): now also R34.1
- net VBUS_P2: now reaches C57.1, J9.1 (VBUS)
- net VBUS_P2: now also U10.6 (VBUS), C59.1, U14.1 (VOUT)
- net ST: now reaches U15.8 (ST)
- net ST: now also R34.2
- net at U19.18 (PSELF): now also R41.1
- net PWREN: now reaches U19.24 (~{PWREN})
- net PWREN: now also U13.4 (EN#), U14.4 (EN#)
- new net: R36.2, U14.5 (ISET)
- new net: C67.1, R38.1, R40.1, U16.1 (G)
- new net: L6.2, U18.3 (LX)
- new net: C77.2, R42.2, R43.1, U18.5 (FB)
- new net: R35.2, U13.5 (ISET)
- new net: L5.1, U16.3 (D)
- new net OVCUR: U13.3 (FLAG#), U14.3 (FLAG#), U19.1 (~{OVCUR})
- new net VBUS_P1: C56.1, C58.1, J8.1 (VBUS), U13.1 (VOUT), U9.6 (VBUS)
- now unconnected: S6.1
- no-connect marks 22 -> 19
Other:
- moved on the sheet: C57, C60, C61, C64, C65, C66, C68, C71, C72, C74, C75, C76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

Commit message: FRANK Next WIP
Parts:
- L6: footprint Inductor_SMD:L_Cenker_CKCS3015 -> FRANK:L_Cenker_CKCS3015
- U18: footprint Package_TO_SOT_SMD:SOT-23-5 -> FRANK:SOT-23-5
Changed lines of the file:
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@@
 			)
 		)
-		(property "Footprint" "Inductor_SMD:L_Cenker_CKCS3015"
+		(property "Footprint" "FRANK:L_Cenker_CKCS3015"
 			(at 232.41 22.86 0)
 			(hide yes)
@@
 			)
 		)
-		(property "Footprint" "Package_TO_SOT_SMD:SOT-23-5"
+		(property "Footprint" "FRANK:SOT-23-5"
 			(at 209.55 25.4 0)
 			(hide yes)

Commit message: FRANK Next 1.01 WIP
Parts:
- L5: footprint Inductor_SMD:L_0805_2012Metric -> FRANK:L_0805_2012Metric
- R35, R36, R41: symbol Device:R_Small -> FRANK:R_Small
- U13, U14: footprint Package_TO_SOT_SMD:SOT-23-6 -> FRANK:SOT-23-6
Changed lines of the file:
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@@
 			)
 		)
-		(property "Footprint" "Package_TO_SOT_SMD:SOT-23-6"
+		(property "Footprint" "FRANK:SOT-23-6"
 			(at 93.98 177.8 0)
 			(hide yes)
@@
 	(symbol
 		(lib_name "R_Small_4")
-		(lib_id "Device:R_Small")
+		(lib_id "FRANK:R_Small")
 		(at 121.92 172.72 270)
 		(mirror x)
@@
 	)
 	(symbol
-		(lib_id "Device:R_Small")
+		(lib_id "FRANK:R_Small")
 		(at 214.63 118.11 0)
 		(unit 1)
@@
 	(symbol
 		(lib_name "R_Small_1")
-		(lib_id "Device:R_Small")
+		(lib_id "FRANK:R_Small")
 		(at 121.92 156.21 270)
 		(mirror x)
@@
 			)
 		)
-		(property "Footprint" "Inductor_SMD:L_0805_2012Metric"
+		(property "Footprint" "FRANK:L_0805_2012Metric"
 			(at 147.32 46.482 90)
 			(hide yes)
@@
 			)
 		)
-		(property "Footprint" "Package_TO_SOT_SMD:SOT-23-6"
+		(property "Footprint" "FRANK:SOT-23-6"
 			(at 93.98 161.29 0)
 			(hide yes)

Commit message: FRANK Next WIP
Parts:
- added C85: 10uF, FRANK:C_0603_1608Metric, symbol FRANK:C
- C58, C59: value 10uF -> 100uF; footprint FRANK:C_0603_1608Metric -> FRANK:C_1206_3216Metric
- U13, U14: footprint FRANK:SOT-23-6 -> Package_TO_SOT_SMD:SOT-23-6
Connections:
- net +3V3: now also C85.1
- net GND: now also C85.2
Other:
- moved on the sheet: C73
Changed lines of the file:
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@@
 	)
 	(junction
-		(at 242.57 22.86)
-		(diameter 0)
-		(color 0 0 0 0)
-	)
-	(junction
 		(at 220.98 63.5)
 		(diameter 0)
@@
 	)
 	(junction
+		(at 243.84 22.86)
+		(diameter 0)
+		(color 0 0 0 0)
+	)
+	(junction
 		(at 63.5 35.56)
 		(diameter 0)
@@
 	)
 	(junction
+		(at 238.76 22.86)
+		(diameter 0)
+		(color 0 0 0 0)
+	)
+	(junction
 		(at 105.41 100.33)
 		(diameter 0)
@@
 	(wire
 		(pts
+			(xy 238.76 22.86) (xy 243.84 22.86)
+		)
+		(stroke
+			(width 0)
+			(type default)
+		)
+	)
+	(wire
+		(pts
 			(xy 67.31 82.55) (xy 77.47 82.55)
 		)
@@
 	(wire
 		(pts
-			(xy 236.22 22.86) (xy 242.57 22.86)
+			(xy 236.22 22.86) (xy 238.76 22.86)
 		)
 		(stroke
@@
 	(wire
 		(pts
+			(xy 243.84 22.86) (xy 264.16 22.86)
+		)
+		(stroke
+			(width 0)
+			(type default)
+		)
+	)
+	(wire
+		(pts
 			(xy 148.59 153.67) (xy 160.02 153.67)
 		)
@@
 	(wire
 		(pts
-			(xy 242.57 22.86) (xy 264.16 22.86)
-		)
-		(stroke
-			(width 0)
-			(type default)
-		)
-	)
-	(wire
-		(pts
 			(xy 194.31 27.94) (xy 194.31 22.86)
 		)
@@
 			)
 		)
-		(property "Footprint" "FRANK:SOT-23-6"
+		(property "Footprint" "Package_TO_SOT_SMD:SOT-23-6"
 			(at 93.98 177.8 0)
 			(hide yes)
@@
 	)
 	(symbol
-		(lib_name "R_Small_4")
 		(lib_id "FRANK:R_Small")
 		(at 121.92 172.72 270)
@@
 	(symbol
 		(lib_id "FRANK:C")
-		(at 242.57 26.67 0)
+		(at 238.76 26.67 0)
 		(unit 1)
 		(body_style 1)
@@
 		(dnp no)
 		(property "Reference" "C73"
-			(at 245.11 25.4 0)
+			(at 232.41 25.4 0)
 			(show_name no)
 			(do_not_autoplace no)
@@
 		)
 		(property "Value" "10uF"
-			(at 245.11 27.94 0)
+			(at 231.14 27.94 0)
 			(show_name no)
 			(do_not_autoplace no)
@@
 		)
 		(property "Footprint" "FRANK:C_0603_1608Metric"
-			(at 242.57 26.67 0)
+			(at 238.76 26.67 0)
 			(hide yes)
 			(show_name no)
@@
 		)
 		(property "Datasheet" ""
-			(at 242.57 26.67 0)
+			(at 238.76 26.67 0)
 			(show_name no)
 			(do_not_autoplace no)
@@
 		)
 		(property "Description" ""
-			(at 242.57 26.67 0)
+			(at 238.76 26.67 0)
 			(show_name no)
 			(do_not_autoplace no)
@@
 		)
 		(property "LCSC" "C96446"
-			(at 242.57 26.67 0)
+			(at 238.76 26.67 0)
 			(hide yes)
 			(show_name no)
@@
 	)
 	(symbol
-		(lib_name "R_Small_1")
 		(lib_id "FRANK:R_Small")
 		(at 121.92 156.21 270)
@@
 	)
 	(symbol
-		(lib_name "R_Small_3")
 		(lib_id "FRANK:R_Small")
 		(at 55.88 26.67 270)
@@
 	)
 	(symbol
+		(lib_id "FRANK:C")
+		(at 243.84 26.67 0)
+		(unit 1)
+		(body_style 1)
+		(exclude_from_sim no)
+		(in_bom yes)
+		(on_board yes)
+		(in_pos_files yes)
+		(dnp no)
+		(property "Reference" "C85"
+			(at 246.38 25.4 0)
+			(show_name no)
+			(do_not_autoplace no)
+			(effects
+				(font
+					(size 1.27 1.27)
+				)
+				(justify left)
+			)
+		)
+		(property "Value" "10uF"
+			(at 246.38 27.94 0)
+			(show_name no)
+			(do_not_autoplace no)
+			(effects
+				(font
+					(size 1.27 1.27)
+				)
+				(justify left)
+			)
+		)
+		(property "Footprint" "FRANK:C_0603_1608Metric"
+			(at 243.84 26.67 0)
+			(hide yes)
+			(show_name no)
+			(do_not_autoplace no)
+			(effects
+				(font
+					(size 1.27 1.27)
+				)
+			)
+		)
+		(property "Datasheet" ""
+			(at 243.84 26.67 0)
+			(show_name no)
+			(do_not_autoplace no)
+			(effects
+				(font
+					(size 1.27 1.27)
+				)
+			)
+		)
+		(property "Description" ""
+			(at 243.84 26.67 0)
+			(show_name no)
+			(do_not_autoplace no)
+			(effects
+				(font
+					(size 1.27 1.27)
+				)
+			)
+		)
+		(property "LCSC" "C96446"
+			(at 243.84 26.67 0)
+			(hide yes)
+			(show_name no)
+			(do_not_autoplace no)
+			(effects
+				(font
+					(size 1.27 1.27)
+				)
+			)
+		)
+		(pin "1"
+		)
+		(pin "2"
+		)
+		(instances
+			(project "frank_next"
+				(path "/8c0b3d8b-46d3-4173-ab1e-a61765f77d61/8add5a37-def3-463f-a5fe-02872c49aeb0"
+					(reference "C85")
+					(unit 1)
+				)
+			)
+		)
+	)
+	(symbol
+		(lib_id "FRANK:GND")
+		(at 243.84 30.48 0)
+		(unit 1)
+		(body_style 1)
+		(exclude_from_sim no)
+		(in_bom yes)
+		(on_board yes)
+		(in_pos_files yes)
+		(dnp no)
+		(property "Reference" "#PWR0200"
+			(at 243.84 36.83 0)
+			(hide yes)
+			(show_name no)
+			(do_not_autoplace no)
+			(effects
+				(font
+					(size 1.27 1.27)
+				)
+			)
+		)
+		(property "Value" "GND"
+			(at 243.84 34.29 0)
+			(show_name no)
+			(do_not_autoplace no)
+			(effects
+				(font
+					(size 1.27 1.27)
+				)
+			)
+		)
+		(property "Footprint" ""
+			(at 243.84 30.48 0)
+			(hide yes)
+			(show_name no)
+			(do_not_autoplace no)
+			(effects
+				(font
+					(size 1.27 1.27)
+				)
+			)
+		)
+		(property "Datasheet" ""
+			(at 243.84 30.48 0)
+			(hide yes)
+			(show_name no)
+			(do_not_autoplace no)
+			(effects
+				(font
+					(size 1.27 1.27)
+				)
+			)
+		)
+		(property "Description" "Power symbol creates a global label with name \"GND\" , ground"
+			(at 243.84 30.48 0)
+			(hide yes)
+			(show_name no)
+			(do_not_autoplace no)
+			(effects
+				(font
+					(size 1.27 1.27)
+				)
+			)
+		)
+		(pin "1"
+		)
+		(instances
+			(project "frank_next"
+				(path "/8c0b3d8b-46d3-4173-ab1e-a61765f77d61/8add5a37-def3-463f-a5fe-02872c49aeb0"
+					(reference "#PWR0200")
+					(unit 1)
+				)
+			)
+		)
+	)
+	(symbol
 		(lib_id "FRANK:GND")
 		(at 175.26 30.48 0)
@@
 			)
 		)
-		(property "Value" "10uF"
+		(property "Value" "100uF"
 			(at 49.149 163.957 0)
 			(show_name no)
@@
 			)
 		)
-		(property "Footprint" "FRANK:C_0603_1608Metric"
+		(property "Footprint" "FRANK:C_1206_3216Metric"
 			(at 51.1048 161.29 0)
 			(hide yes)
@@
 	)
 	(symbol
+		(lib_name "CH217K_1")
 		(lib_id "FRANK:CH217K")
 		(at 100.33 156.21 0)
@@
 			)
 		)
-		(property "Footprint" "FRANK:SOT-23-6"
+		(property "Footprint" "Package_TO_SOT_SMD:SOT-23-6"
 			(at 93.98 161.29 0)
 			(hide yes)
@@
 	)
 	(symbol
-		(lib_name "R_Small_2")
 		(lib_id "FRANK:R_Small")
 		(at 36.83 88.9 270)
@@
 			)
 		)
-		(property "Value" "10uF"
+		(property "Value" "100uF"
 			(at 49.149 122.047 0)
 			(show_name no)
@@
 			)
 		)
-		(property "Footprint" "FRANK:C_0603_1608Metric"
+		(property "Footprint" "FRANK:C_1206_3216Metric"
 			(at 51.1048 119.38 0)
 			(hide yes)
@@
 	(symbol
 		(lib_id "FRANK:GND")
-		(at 242.57 30.48 0)
+		(at 238.76 30.48 0)
 		(unit 1)
 		(body_style 1)
@@
 		(dnp no)
 		(property "Reference" "#PWR0159"
-			(at 242.57 30.48 0)
+			(at 238.76 30.48 0)
 			(hide yes)
 			(show_name no)
@@
 		)
 		(property "Value" "GND"
-			(at 242.57 34.29 0)
+			(at 238.76 34.29 0)
 			(show_name no)
 			(do_not_autoplace no)
@@
 		)
 		(property "Footprint" ""
-			(at 242.57 30.48 0)
+			(at 238.76 30.48 0)
 			(show_name no)
 			(do_not_autoplace no)
@@
 		)
 		(property "Datasheet" ""
-			(at 242.57 30.48 0)
+			(at 238.76 30.48 0)
 			(show_name no)
 			(do_not_autoplace no)
@@
 		)
 		(property "Description" ""
-			(at 242.57 30.48 0)
+			(at 238.76 30.48 0)
 			(show_name no)
 			(do_not_autoplace no)
@@
 	)
 	(symbol
-		(lib_name "R_Small_2")
 		(lib_id "FRANK:R_Small")
 		(at 55.88 41.91 270)
@@
 	)
 	(symbol
-		(lib_name "R_Small_3")
 		(lib_id "FRANK:R_Small")
 		(at 36.83 73.66 270)
