File: frank_next/ds2401.kicad_sch (KiCad schematic)
At the start: 2 parts, among them U20 DS2401P+

Commit message: FRANK Next updates
Parts:
- renumbered R38 to R46, U20 to U23
Changed lines of the file:
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@@
 		(in_pos_files yes)
 		(dnp no)
-		(property "Reference" "R38"
+		(property "Reference" "R46"
 			(at 141.986 104.14 90)
 			(show_name no)
@@
 			(project "frank_next"
 				(path "/8c0b3d8b-46d3-4173-ab1e-a61765f77d61/dc291665-7d36-4b6a-bffa-6099b8b37444"
-					(reference "R38")
+					(reference "R46")
 					(unit 1)
 				)
@@
 		(in_pos_files yes)
 		(dnp no)
-		(property "Reference" "#PWR0181"
+		(property "Reference" "#PWR0190"
 			(at 130.81 96.52 0)
 			(hide yes)
@@
 			(project "frank_next"
 				(path "/8c0b3d8b-46d3-4173-ab1e-a61765f77d61/dc291665-7d36-4b6a-bffa-6099b8b37444"
-					(reference "#PWR0181")
+					(reference "#PWR0190")
 					(unit 1)
 				)
@@
 		(dnp no)
 		(fields_autoplaced yes)
-		(property "Reference" "#PWR0182"
+		(property "Reference" "#PWR0191"
 			(at 139.7 104.14 0)
 			(hide yes)
@@
 			(project "frank_next"
 				(path "/8c0b3d8b-46d3-4173-ab1e-a61765f77d61/dc291665-7d36-4b6a-bffa-6099b8b37444"
-					(reference "#PWR0182")
+					(reference "#PWR0191")
 					(unit 1)
 				)
@@
 		(dnp no)
 		(fields_autoplaced yes)
-		(property "Reference" "U20"
+		(property "Reference" "U23"
 			(at 160.02 88.9 0)
 			(show_name no)
@@
 			(project "frank_next"
 				(path "/8c0b3d8b-46d3-4173-ab1e-a61765f77d61/dc291665-7d36-4b6a-bffa-6099b8b37444"
-					(reference "U20")
+					(reference "U23")
 					(unit 1)
 				)

Commit message: Boards WIP
Parts:
- R46: LCSC (none) -> C23162
- U23: LCSC (none) -> C518978
Changed lines of the file:
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@@
 			)
 		)
-		(property "Datasheet" "https://www.vishay.com/docs/28952/mcs0402at-mct0603at-mcu0805at-mca1206at.pdf"
+		(property "Datasheet" "https://jlcpcb.com/api/file/downloadByFileSystemAccessId/8579706251506339840"
 			(at 139.7 104.14 0)
 			(hide yes)
@@
 		(property "Description" "Resistor, small symbol"
 			(at 139.7 104.14 0)
+			(hide yes)
+			(show_name no)
+			(do_not_autoplace no)
+			(effects
+				(font
+					(size 1.27 1.27)
+				)
+			)
+		)
+		(property "LCSC" "C23162"
+			(at 0 0 0)
 			(hide yes)
 			(show_name no)
@@
 			)
 		)
-		(property "Datasheet" "http://pdfserv.maximintegrated.com/en/ds/DS2401.pdf"
+		(property "Datasheet" "https://jlcpcb.com/api/file/downloadByFileSystemAccessId/8588913591751335936"
 			(at 170.18 291.44 0)
 			(hide yes)
@@
 			(hide yes)
 			(show_name no)
+			(do_not_autoplace no)
+			(effects
+				(font
+					(size 1.27 1.27)
+				)
+			)
+		)
+		(property "LCSC" "C518978"
+			(at 0 0 0)
+			(hide yes)
+			(show_name no)
