File: frank_next/ch343p.kicad_sch (KiCad schematic)
At the start: 4 parts, among them U17 CH343P

Commit message: Board Updates
Parts:
- added LD4: Orange, FRANK:LED_0603_1608Metric, symbol FRANK:LED
- added R36: 1K, FRANK:R_0603_1608Metric, symbol FRANK:R
- renumbered C68 to C70, C69 to C71, C70 to C72
Connections:
- net +3V3: now also R36.2
- net at U17.10 (~{ACT}): now also LD4.1 (K)
- new net: LD4.2 (A), R36.1
- no-connect marks 5 -> 4

Commit message: FRANK Next WIP
Parts:
- C70, C71, C72: value 100n -> 100nF
Changed lines of the file:
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@@
 		(rev "${VERSION}")
 		(company "Mikhail Matveev")
-		(comment 1 "https://github.com/rh1tech/frank_next")
+		(comment 1 "https://github.com/rh1tech/frank")
 	)
 	(junction
@@
 			)
 		)
-		(property "Value" "100n"
+		(property "Value" "100nF"
 			(at 96.393 84.709 0)
 			(show_name no)
@@
 			)
 		)
-		(property "Value" "100n"
+		(property "Value" "100nF"
 			(at 99.06 77.2414 0)
 			(show_name no)
@@
 			)
 		)
-		(property "Value" "100n"
+		(property "Value" "100nF"
 			(at 114.681 84.963 0)
 			(show_name no)

Commit message: FRANK Next updates
Parts:
- renumbered C70 to C78, C71 to C79, C72 to C80, R36 to R44, U17 to U20
Other:
- moved on the sheet: C78, C79, C80, LD4, R44, U20

Commit message: Boards WIP
Parts:
- C78, C79, C80: LCSC (none) -> C14663
- LD4: LCSC (none) -> C965800
- R44: LCSC (none) -> C21190
- U20: LCSC (none) -> C2846043
Changed lines of the file:
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@@
 			)
 		)
-		(property "Datasheet" ""
+		(property "Datasheet" "https://jlcpcb.com/api/file/downloadByFileSystemAccessId/8757826625847070720"
 			(at 180.34 102.87 0)
 			(hide yes)
@@
 		(property "Description" "Light emitting diode"
 			(at 180.34 102.87 0)
+			(hide yes)
+			(show_name no)
+			(do_not_autoplace no)
+			(effects
+				(font
+					(size 1.27 1.27)
+				)
+			)
+		)
+		(property "LCSC" "C965800"
+			(at 0 0 0)
 			(hide yes)
 			(show_name no)
@@
 			)
 		)
-		(property "Datasheet" ""
+		(property "Datasheet" "https://jlcpcb.com/api/file/downloadByFileSystemAccessId/8579706098733010944"
 			(at 187.96 102.87 0)
 			(hide yes)
@@
 			)
 		)
-		(property "LCSC" ""
+		(property "LCSC" "C21190"
 			(at 187.96 102.87 0)
 			(show_name no)
@@
 			)
 		)
+		(property "LCSC" "C2846043"
+			(at 0 0 0)
+			(hide yes)
+			(show_name no)
+			(do_not_autoplace no)
+			(effects
+				(font
+					(size 1.27 1.27)
+				)
+			)
+		)
 		(pin "3"
 		)
@@
 			)
 		)
-		(property "LCSC" ""
+		(property "LCSC" "C14663"
 			(at 146.05 91.44 0)
 			(show_name no)
@@
 			)
 		)
-		(property "LCSC" ""
+		(property "LCSC" "C14663"
 			(at 157.48 80.01 0)
 			(show_name no)
@@
 			)
 		)
-		(property "LCSC" ""
+		(property "LCSC" "C14663"
 			(at 162.56 87.63 0)
 			(show_name no)

Commit message: Board updates
Parts:
- removed C78, C79, C80: 100nF, FRANK:C_0603_1608Metric, symbol FRANK:C
- removed R44: 1K, FRANK:R_0603_1608Metric, symbol FRANK:R
- added C92, C93, C94: 100nF, FRANK:C_0603_1608Metric, symbol FRANK:C
- added R64: 1K, FRANK:R_0603_1608Metric, symbol FRANK:R
Connections:
- net +3V3: now also C94.2, R64.2
- net GND: now also C92.1, C93.1, C94.1
- net VBUS: now also C92.2
- net at LD4.2 (A): now also R64.1
- net at U20.6 (V3_{OUT}): now also C93.2
