File: frank_next/rp2350b.kicad_sch (KiCad schematic)
At the start: 38 parts, among them J1 Debug, J2 UART, U1 W25Q128JVPIQ, U2 ESP-PSRAM64, U3 RP2350B, Y1 ASE-12MHz

Commit message: Board Updates
Parts:
- renumbered LD1 to LD2, R1 to R2, R2 to R3, R3 to R4, R4 to R5, R5 to R6, R6 to R7, R7 to R8, R8 to R9

Commit message: FRANK Next WIP
Parts:
- C1, C10, C11, C12, C13, C14, C15, C16, C17, C18, C19, C2, C3, C6, C9: value 100n -> 100nF
- L1: value 3.3u -> 3.3uF
- U2: value ESP-PSRAM64 -> ESP-PSRAM64H
- renumbered LD2 to LD1, R2 to R1, R3 to R2, R4 to R3, R5 to R4, R6 to R5, R7 to R6, R8 to R7, R9 to R8
Connections:
- net GPIO40/UART_1: now reaches J2.1 (Pin_1), U3.49 (GPIO40_ADC0)
- net GPIO41/UART_3: now reaches J2.3 (Pin_3), U3.52 (GPIO41_ADC1)
Other:
- moved on the sheet: J2

Commit message: Board updates
Parts:
- L1: value 3.3uF -> 3.3µH
- U1: footprint FRANK:SON127P600X500X80-9N-D -> FRANK:WSON-8-1EP_6x5mm_P1.27mm_EP3.45x4.35mm
- Y1: footprint FRANK:Oscillator_SMD_3225_4Pin -> FRANK:Oscillator_SMD_3225-4Pin_3.2x2.5mm
Changed lines of the file:
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@@
 		(fields_autoplaced yes)
 		(property "Reference" "L1"
-			(at 147.32 96.52 0)
+			(at 147.32 96.5199 0)
 			(show_name no)
 			(do_not_autoplace no)
@@
 			)
 		)
-		(property "Value" "3.3uF"
-			(at 147.32 99.06 0)
+		(property "Value" "3.3µH"
+			(at 147.32 99.0599 0)
 			(show_name no)
 			(do_not_autoplace no)
@@
 			)
 		)
-		(property "Footprint" "FRANK:SON127P600X500X80-9N-D"
+		(property "Footprint" "FRANK:WSON-8-1EP_6x5mm_P1.27mm_EP3.45x4.35mm"
 			(at 147.32 277.8 0)
 			(hide yes)
@@
 			)
 		)
-		(property "Footprint" "FRANK:Oscillator_SMD_3225_4Pin"
+		(property "Footprint" "FRANK:Oscillator_SMD_3225-4Pin_3.2x2.5mm"
 			(at 143.51 146.05 0)
 			(hide yes)

Commit message: FRANK Next updates
Parts:
- removed C3: 100nF, FRANK:C_0603_1608Metric, symbol FRANK:C
- removed R2: 10K, FRANK:R_0603_1608Metric, symbol FRANK:R_Small
- removed U2: ESP-PSRAM64H, FRANK:SO-8_3.9x4.9mm_P1.27mm, symbol FRANK:ESP-PSRAM64H
- removed Y1: ASE-12MHz, FRANK:Oscillator_SMD_3225-4Pin_3.2x2.5mm, symbol FRANK:ASE-xxxMHz
- added C5, C6: 15pF, FRANK:C_0603_1608Metric, symbol FRANK:C
- added R1: 10K, FRANK:R_0603_1608Metric, symbol FRANK:R_Small
- added R6: 1K, FRANK:R_0603_1608Metric, symbol FRANK:R
- added U1: APS6404L-3SQR-ZR, FRANK:PSON50P200X300X50-9N, symbol FRANK:APS6404L-3SQR-ZR
- added Y1: 12MHz, FRANK:Crystal_SMD_3225-4Pin_3.2x2.5mm, symbol FRANK:Crystal_GND24
- renumbered C9 to C10, C10 to C11, C11 to C12, C12 to C13, C13 to C14, C14 to C15, C15 to C16, C16 to C17, C17 to C18, C18 to C19, C19 to C20, C4 to C3, C5 to C4, C6 to C7, C7 to C8, C8 to C9, R1 to R2, R6 to R7, R7 to R8, R8 to R9, U1 to U2
Connections:
- net +3V3: now also C2.2, R1.2, U1.8 (VDD); no longer C2.1
- net GND: now also C2.1, C5.2, C6.2, U1.4 (VSS), U1.9 (EXP), Y1.2, Y1.4; no longer C2.2
- net GPIO47: now also R1.1, U1.1 (~{CE})
- net QSPI_SCLK: now also U1.6 (SCLK)
- net QSPI_SD0: now also U1.5 (SI/SIO(0))
- net QSPI_SD1: now also U1.2 (SO/SIO(1))
- net QSPI_SD2: now also U1.3 (SIO(2))
- net QSPI_SD3: now also U1.7 (SIO(3))
- net XIN: now also C5.1, Y1.3
- net XOUT: now reaches U3.31 (XOUT)
- net XOUT: now also R6.2
- new net: C6.1, R6.1, Y1.1
- no-connect marks 2 -> 1

Commit message: FRANK Next WIP
Parts:
- added R52, R53: 1K, FRANK:R_0603_1608Metric, symbol FRANK:R
Connections:
- net GPIO38: now also R52.2; no longer U3.47 (GPIO38)
- net GPIO39: now also R53.2; no longer U3.48 (GPIO39)
- new net: R52.1, U3.47 (GPIO38)
- new net: R53.1, U3.48 (GPIO39)
Changed lines of the file:
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@@
 	(wire
 		(pts
+			(xy 246.38 198.12) (xy 247.65 198.12)
+		)
+		(stroke
+			(width 0)
+			(type default)
+		)
+	)
+	(wire
+		(pts
+			(xy 255.27 198.12) (xy 259.08 198.12)
+		)
+		(stroke
+			(width 0)
+			(type default)
+		)
+	)
+	(wire
+		(pts
+			(xy 246.38 200.66) (xy 247.65 200.66)
+		)
+		(stroke
+			(width 0)
+			(type default)
+		)
+	)
+	(wire
+		(pts
+			(xy 255.27 200.66) (xy 259.08 200.66)
+		)
+		(stroke
+			(width 0)
+			(type default)
+		)
+	)
+	(wire
+		(pts
 			(xy 308.61 128.27) (xy 303.53 128.27)
 		)
@@
 	(hierarchical_label "GPIO38"
 		(shape input)
-		(at 246.38 198.12 0)
+		(at 259.08 198.12 0)
 		(effects
 			(font
@@
 	(hierarchical_label "GPIO39"
 		(shape input)
-		(at 246.38 200.66 0)
+		(at 259.08 200.66 0)
 		(effects
 			(font
@@
 					(unit 1)
 				)
+			)
+		)
+	)
+	(symbol
+		(lib_id "FRANK:R")
+		(at 251.46 198.12 90)
+		(unit 1)
+		(body_style 1)
+		(exclude_from_sim no)
+		(in_bom yes)
+		(on_board yes)
+		(in_pos_files yes)
+		(dnp no)
+		(property "Reference" "R52"
+			(at 251.46 203.3778 90)
+			(show_name no)
+			(do_not_autoplace no)
+			(effects
+				(font
+					(size 1.27 1.27)
+				)
+			)
+		)
+		(property "Value" "1K"
+			(at 251.46 201.0664 90)
+			(show_name no)
+			(do_not_autoplace no)
+			(effects
+				(font
+					(size 1.27 1.27)
+				)
+			)
+		)
+		(property "Footprint" "FRANK:R_0603_1608Metric"
+			(at 251.46 199.898 90)
+			(hide yes)
+			(show_name no)
+			(do_not_autoplace no)
+			(effects
+				(font
+					(size 1.27 1.27)
+				)
+			)
+		)
+		(property "Datasheet" ""
+			(at 251.46 198.12 0)
+			(hide yes)
+			(show_name no)
+			(do_not_autoplace no)
+			(effects
+				(font
+					(size 1.27 1.27)
+				)
+			)
+		)
+		(property "Description" "Resistor"
+			(at 251.46 198.12 0)
+			(hide yes)
+			(show_name no)
+			(do_not_autoplace no)
+			(effects
+				(font
+					(size 1.27 1.27)
+				)
+			)
+		)
+		(pin "1"
+		)
+		(pin "2"
+		)
+		(instances
+			(project "frank_next"
+				(path "/8c0b3d8b-46d3-4173-ab1e-a61765f77d61/234038a0-7aa6-4796-a12c-a2cfd2cf99bc"
+					(reference "R52")
+					(unit 1)
+				)
+			)
+		)
+	)
+	(symbol
+		(lib_id "FRANK:R")
+		(at 251.46 200.66 90)
+		(unit 1)
+		(body_style 1)
+		(exclude_from_sim no)
+		(in_bom yes)
+		(on_board yes)
+		(in_pos_files yes)
+		(dnp no)
+		(property "Reference" "R53"
+			(at 251.46 205.9178 90)
+			(show_name no)
+			(do_not_autoplace no)
+			(effects
+				(font
+					(size 1.27 1.27)
+				)
+			)
+		)
+		(property "Value" "1K"
+			(at 251.46 203.6064 90)
+			(show_name no)
+			(do_not_autoplace no)
+			(effects
+				(font
+					(size 1.27 1.27)
+				)
+			)
+		)
+		(property "Footprint" "FRANK:R_0603_1608Metric"
+			(at 251.46 202.438 90)
+			(hide yes)
+			(show_name no)
+			(do_not_autoplace no)
+			(effects
+				(font
+					(size 1.27 1.27)
+				)
+			)
+		)
+		(property "Datasheet" ""
+			(at 251.46 200.66 0)
+			(hide yes)
+			(show_name no)
+			(do_not_autoplace no)
+			(effects
+				(font
+					(size 1.27 1.27)
+				)
+			)
+		)
+		(property "Description" "Resistor"
+			(at 251.46 200.66 0)
+			(hide yes)
+			(show_name no)
+			(do_not_autoplace no)
+			(effects
+				(font
+					(size 1.27 1.27)
+				)
+			)
+		)
+		(pin "1"
+		)
+		(pin "2"
+		)
+		(instances
+			(project "frank_next"
+				(path "/8c0b3d8b-46d3-4173-ab1e-a61765f77d61/234038a0-7aa6-4796-a12c-a2cfd2cf99bc"
+					(reference "R53")
+					(unit 1)
+				)

Commit message: Board updated
Parts:
- C3, C4, C8, C9: value 4.7u -> 4.7uF
- Y1: value 12MHz -> 12 MHz
Changed lines of the file:
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@@
 			)
 		)
-		(property "Value" "4.7u"
+		(property "Value" "4.7uF"
 			(at 134.62 99.06 0)
 			(show_name no)
@@
 			)
 		)
-		(property "Value" "12MHz"
+		(property "Value" "12 MHz"
 			(at 153.67 154.686 90)
 			(show_name no)
@@
 			)
 		)
-		(property "Value" "4.7u"
+		(property "Value" "4.7uF"
 			(at 123.19 99.06 0)
 			(show_name no)
@@
 			)
 		)
-		(property "Value" "4.7u"
+		(property "Value" "4.7uF"
 			(at 168.91 86.36 0)
 			(show_name no)
@@
 			)
 		)
-		(property "Value" "4.7u"
+		(property "Value" "4.7uF"
 			(at 169.291 57.023 0)
 			(show_name no)

Commit message: Boards WIP
Parts:
- C1, C10, C11, C12, C13, C14, C15, C16, C17, C18, C19, C2, C20, C7: LCSC (none) -> C14663
- C3, C4, C8, C9: LCSC (none) -> C5360844
- C5, C6: LCSC C63339 -> C1644
- D1: LCSC (none) -> C191023
- J1, J2: LCSC (none) -> C160389
- L1: LCSC (none) -> C98035
- LD1: LCSC (none) -> C965555
- R1, R2: LCSC (none) -> C2906982
- R3: LCSC (none) -> C23140
- R4, R52, R53, R6: LCSC (none) -> C21190
- R5: LCSC (none) -> C21189
- R7, R8: LCSC (none) -> C25190
- R9: LCSC (none) -> C23138
- S1, S2: LCSC (none) -> C36498961
- U1: LCSC (none) -> C3040877
- U2: LCSC (none) -> C190862
- U3: LCSC (none) -> C42415655
- Y1: LCSC C9900023240 -> C9002

Commit message: Board updates
Parts:
- removed C17: 100nF, FRANK:C_0603_1608Metric, symbol FRANK:C
- removed D1: 1N5819WS, FRANK:D_SOD-323, symbol FRANK:D_Schottky
- removed LD1: WS2812B-2020, FRANK:LED_WS2812B-2020_PLCC4_2.0x2.0mm, symbol FRANK:WS2812B-2020
- removed R52: 1K, FRANK:R_0603_1608Metric, symbol FRANK:R
- removed R9: 330R, FRANK:R_0603_1608Metric, symbol FRANK:R
- added R10, R11, R12: 100R, FRANK:R_0603_1608Metric, symbol FRANK:R
- added R16, R17: 330R, FRANK:R_0603_1608Metric, symbol FRANK:R
- L1: footprint FRANK:L_Murata_LQH2MCN_2.0x1.6mm -> FRANK:L_AOTA-B201610_2.0x1.6mm
- R13: renamed from R53; value 1K -> 100R
- renumbered C18 to C17, C19 to C18, C20 to C19, R7 to R14, R8 to R15, R1 to R4, R2 to R5, R3 to R6, R4 to R7, R5 to R8, R6 to R9
Connections:
- net GPIO28: now also R10.2; no longer U3.36 (GPIO28)
- net GPIO29: now also R11.2; no longer U3.37 (GPIO29)
- net GPIO38: now also R12.2
- net GPIO45: now also R17.2
- net GPIO46: now also R16.2
- net GPIO25: now reaches U3.26 (GPIO25)
- net at U3.47 (GPIO38): now also R12.1
- net GPIO40/UART_1: no longer names the net of J2.1 (Pin_1)
- net GPIO40/UART_1: now also R16.1; no longer U3.49 (GPIO40_ADC0)
- net GPIO41/UART_3: no longer names the net of J2.3 (Pin_3)
- net GPIO41/UART_3: now also R17.1; no longer U3.52 (GPIO41_ADC1)
- new net: R10.1, U3.36 (GPIO28)
- new net: R11.1, U3.37 (GPIO29)
- new net GPIO40: U3.49 (GPIO40_ADC0)
- new net GPIO41: U3.52 (GPIO41_ADC1)
- no-connect marks 1 -> 0
Other:
- moved on the sheet: S1, S2
