File: frank_core2/rp2350b.kicad_sch (KiCad schematic)
At the start: 42 parts, among them J1 Debug, J2 UART, U1 APS6404L-3SQR-ZR, U2 W25Q128JVPIQ, U3 RP2350B, Y1 12 MHz

Commit message: FRANK Core 2 WIP
Parts:
- renumbered S1 to S2, S2 to S3
Connections:
- net GPIO0/UART_1 renamed GPIO0
- net GPIO1/UART_3 renamed GPIO1
