File: frank_core2/frank_core2.kicad_sch (KiCad schematic)
At the start: 7 parts

Commit message: Boards WIP
Parts:
- R2: value 33R -> 10K; AliExpress https://www.aliexpress.com/item/1005005945735199.html -> https://www.vishay.com/docs/28952/mcs0402at-mct0603at-mcu08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
- R3: value 10K -> 33R; AliExpress https://www.vishay.com/docs/28952/mcs0402at-mct0603at-mcu08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 -> https://www.aliexpress.com/item/1005005945735199.html
Connections:
- net RP2350A/GPIO19 is gone; now on net RP2350/43B/RUNA/SR: R2.1
- net +3V3: now also R2.2; no longer R3.2
- net RP2350/38B/19A/CLK: now also R3.2; no longer R2.2
- net RP2350/43B/RUNA/SR: no longer R3.1
- net RP2350B/GPIO28 renamed RP2350A/GPIO9
- new net RP2350B/GPIO38: R3.1
- no-connect marks 8 -> 6
Other:
- removed sheet Power
- removed sheet SD
- removed sheet TDA Audio
- removed sheet USB Master
- removed sheet USB Slave
- added sheet Audio (audio.kicad_sch)
- added sheet MicroSD (sd.kicad_sch)
- added sheet RTC (rtc.kicad_sch)
- added sheet Tape (tape.kicad_sch)
- added sheet USB (usb.kicad_sch)
- sheet RP2350B: file rp2350b_master.kicad_sch -> rp2350b.kicad_sch
- moved on the sheet: H1, H2, H3, H4

Commit message: FRANK Core2 WIP
Changed lines of the file:
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@@
-	(wire
-		(pts
-			(xy 43.18 171.45) (xy 41.91 171.45)
-		)
-		(stroke
-			(width 0)
-			(type default)
-		)
-	)
 	(wire
 		(pts
@@
 	(wire
 		(pts
-			(xy 43.18 168.91) (xy 41.91 168.91)
-		)
-		(stroke
-			(width 0)
-			(type default)
-		)
-	)
-	(wire
-		(pts
 			(xy 81.28 147.32) (xy 110.49 147.32)
 		)
@@
 	(wire
 		(pts
-			(xy 43.18 168.91) (xy 81.28 168.91)
+			(xy 54.61 168.91) (xy 81.28 168.91)
 		)
 		(stroke
@@
 	(wire
 		(pts
-			(xy 43.18 171.45) (xy 81.28 171.45)
+			(xy 54.61 171.45) (xy 81.28 171.45)
 		)
 		(stroke
@@
 		)
 	)
-	(label "GPIO28{slash}SDA"
-		(at 43.18 171.45 0)
-		(effects
-			(font
-				(size 1.27 1.27)
-			)
-			(justify left bottom)
-		)
-	)
 	(label "GPIO14{slash}D0N"
 		(at 97.79 54.61 180)
@@
 	(label "SD{slash}CMD{slash}GPIO7"
 		(at 82.55 147.32 0)
-		(effects
-			(font
-				(size 1.27 1.27)
-			)
-			(justify left bottom)
-		)
-	)
-	(label "GPIO29{slash}SCL"
-		(at 43.18 168.91 0)
 		(effects
 			(font
@@
 	)
 	(sheet
-		(at 29.21 166.37)
+		(at 41.91 166.37)
 		(size 12.7 7.62)
 		(exclude_from_sim no)
@@
 		)
 		(property "Sheetname" "RTC"
-			(at 29.21 165.6584 0)
+			(at 41.91 165.6584 0)
 			(show_name no)
 			(do_not_autoplace no)
@@
 		)
 		(property "Sheetfile" "rtc.kicad_sch"
-			(at 29.21 174.5746 0)
+			(at 41.91 174.5746 0)
 			(hide yes)
 			(show_name no)
@@
 		)
 		(pin "SCL" input
-			(at 41.91 168.91 0)
+			(at 54.61 168.91 0)
 			(effects
 				(font
@@
 		)
 		(pin "SDA" input
-			(at 41.91 171.45 0)
-			(effects
-				(font
+			(at 54.61 171.45 0)
+			(effects
+				(font

Commit message: FRANK Core 2 WIP
Parts:
- added S1: ESP Reset, FRANK:Button_SMD_3x4x2mm, symbol FRANK:KMR221G_LFS
- R1, R3: LCSC (none) -> C23140
- R2: LCSC (none) -> C2906982
Connections:
- net GND: now also S1.2, S1.4
- new net ERST: S1.1, S1.3
Other:
- added sheet ESP01 (esp01s.kicad_sch)
- sheet RP2350B ports: added GPIO0, GPIO1; removed none

Commit message: Board updates
Parts:
- removed S1: ESP Reset, FRANK:Button_SMD_3x4x2mm, symbol FRANK:KMR221G_LFS
Other:
- sheet ESP01 ports: added none; removed RST
