File: dino/power.kicad_sch (KiCad schematic)
At the start: 30 parts, among them J8 DC-005-5A-2.0, Q2 AO3401A, Q3 AO3401A, U11 MP1584EN-LF-Z

Commit message: Dino HW 1.00
Parts:
- renumbered C40 to C41, C41 to C42, C42 to C43, C43 to C44, C44 to C45, C45 to C46, C46 to C47, C47 to C48, C48 to C49, R31 to R33, R32 to R34, R33 to R35, R34 to R36, R35 to R37, R36 to R38, R37 to R39, R38 to R40, R39 to R41, R40 to R42, U11 to U12
