File: dino/sd.kicad_sch (KiCad schematic)
At the start: 2 parts, among them J3 104031-0811

Commit message: Dino HW 1.00
Parts:
- renumbered C8 to C9
Changed lines of the file:
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@@
 		(in_pos_files yes)
 		(dnp no)
-		(property "Reference" "C8"
+		(property "Reference" "C9"
 			(at 120.7516 94.869 0)
 			(show_name no)
@@
 			(project "dino"
 				(path "/8c0b3d8b-46d3-4173-ab1e-a61765f77d61/2e81912e-397c-4129-8da5-abf37a4f2667"
-					(reference "C8")
+					(reference "C9")
 					(unit 1)
 				)
@@
 		(dnp no)
 		(fields_autoplaced yes)
-		(property "Reference" "#PWR037"
+		(property "Reference" "#PWR044"
 			(at 132.08 99.06 0)
 			(hide yes)
@@
 			(project "dino"
 				(path "/8c0b3d8b-46d3-4173-ab1e-a61765f77d61/2e81912e-397c-4129-8da5-abf37a4f2667"
-					(reference "#PWR037")
+					(reference "#PWR044")
 					(unit 1)
 				)
@@
 		(dnp no)
 		(fields_autoplaced yes)
-		(property "Reference" "#PWR033"
+		(property "Reference" "#PWR040"
 			(at 111.76 97.79 0)
 			(hide yes)
@@
 			(project "dino"
 				(path "/8c0b3d8b-46d3-4173-ab1e-a61765f77d61/2e81912e-397c-4129-8da5-abf37a4f2667"
-					(reference "#PWR033")
+					(reference "#PWR040")
 					(unit 1)
 				)
@@
 		(dnp no)
 		(fields_autoplaced yes)
-		(property "Reference" "#PWR040"
+		(property "Reference" "#PWR047"
 			(at 194.31 113.03 0)
 			(hide yes)
@@
 			(project "dino"
 				(path "/8c0b3d8b-46d3-4173-ab1e-a61765f77d61/2e81912e-397c-4129-8da5-abf37a4f2667"
-					(reference "#PWR040")
+					(reference "#PWR047")
 					(unit 1)
 				)
@@
 		(dnp no)
 		(fields_autoplaced yes)
-		(property "Reference" "#PWR038"
+		(property "Reference" "#PWR045"
 			(at 138.43 102.87 0)
 			(hide yes)
@@
 			(project "dino"
 				(path "/8c0b3d8b-46d3-4173-ab1e-a61765f77d61/2e81912e-397c-4129-8da5-abf37a4f2667"
-					(reference "#PWR038")
-					(unit 1)
-				)
+					(reference "#PWR045")
+					(unit 1)
+				)
