File: dino/usb.kicad_sch (KiCad schematic)
At the start: 24 parts, among them J6 USB4215-03-A, J7 SS-52100-004, U10 USBLC6-2SC6, U7 USBLC6-2SC6, U8 TPS2116DRL, U9 USBLC6-2SC6

Commit message: Dino HW 1.00
Parts:
- renumbered C27 to C28, C28 to C29, C29 to C30, C30 to C31, C31 to C32, C32 to C33, C33 to C34, C34 to C35, C35 to C36, C36 to C37, C37 to C38, C38 to C39, R26 to R28, R27 to R29, R28 to R30, R29 to R31, R30 to R32, U9 to U10, U10 to U11, U7 to U8, U8 to U9
