File: xt8086_beta/xt8086_beta.kicad_sch (KiCad schematic)
At the start: 18 parts, among them J1 UART, J2 PWR, U1 SN74LS04, U2 SN74LS74

Commit message: Board updates
Parts:
- removed S2: DS01-254-S-06BE, xt8086:DS01-254-S-06BE, symbol xt8086:DS01-254-S-06BE
- added JP1: HDMI Audio, xt8086:SolderJumper-2_P1.3mm_Open_Pad1.0x1.5mm, symbol xt8086:Conn_01x02_Pin
- added JP2: Jack In, xt8086:SolderJumper-2_P1.3mm_Open_Pad1.0x1.5mm, symbol xt8086:Conn_01x02_Pin
- added JP3: Speaker In, xt8086:SolderJumper-2_P1.3mm_Open_Pad1.0x1.5mm, symbol xt8086:Conn_01x02_Pin
- added LD1: Red, xt8086:LED_0805_2012Metric_Pad1.15x1.40mm_HandSolder, symbol xt8086:LED
- added R3: 1K, xt8086:R_0603_1608Metric, symbol xt8086:R
- added S2: SS12D00, xt8086:Switch_Slide_SS12D00, symbol xt8086:SS12D00
- renumbered LD1 to LD3, R3 to R5
Connections:
- net Audio/JACK_IN: now also JP2.1 (Pin_1)
- net Audio/SPK_IN: now also JP3.2 (Pin_2)
- net BHE/GP25: now also R3.2
- net GND: now also S1.2, LD1.1 (K), S2.2
- net HDMI_AUDIO: now also JP1.1 (Pin_1)
- net SPEAKER: now also JP1.2 (Pin_2), JP2.2 (Pin_2), JP3.1 (Pin_1)
- net VBUS: no longer S1.2
- new net: LD1.2 (A), R3.1
- new net Video/VGA_GND: S2.1
- no-connect marks 24 -> 23
Other:
- sheet USB renamed USB, Power
- removed sheet Power
- added sheet RTC (rtc.kicad_sch)
- sheet Video ports: added VGA_GND; removed B, B_IN, G, G_IN, R, R_IN
- moved on the sheet: J1, J2, LD3, R5

Commit message: Board updates
Parts:
- renumbered LD3 to LD2, R5 to R4
Changed lines of the file:
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@@
 		(in_pos_files yes)
 		(dnp no)
-		(property "Reference" "#PWR019"
+		(property "Reference" "#PWR018"
 			(at 251.46 99.06 0)
 			(hide yes)
@@
 			(project "xt8086_beta"
 				(path "/8c0b3d8b-46d3-4173-ab1e-a61765f77d61"
-					(reference "#PWR019")
+					(reference "#PWR018")
 					(unit 1)
 				)
@@
 		(in_pos_files yes)
 		(dnp no)
-		(property "Reference" "#PWR021"
+		(property "Reference" "#PWR020"
 			(at 265.43 41.91 0)
 			(hide yes)
@@
 			(project "xt8086_beta"
 				(path "/8c0b3d8b-46d3-4173-ab1e-a61765f77d61"
-					(reference "#PWR021")
+					(reference "#PWR020")
 					(unit 1)
 				)
@@
 		(in_pos_files yes)
 		(dnp no)
-		(property "Reference" "#PWR012"
+		(property "Reference" "#PWR011"
 			(at 171.45 44.45 0)
 			(hide yes)
@@
 			(project "xt8086_beta"
 				(path "/8c0b3d8b-46d3-4173-ab1e-a61765f77d61"
-					(reference "#PWR012")
+					(reference "#PWR011")
 					(unit 1)
 				)
@@
 		(in_pos_files yes)
 		(dnp no)
-		(property "Reference" "#PWR015"
+		(property "Reference" "#PWR014"
 			(at 217.17 80.01 0)
 			(hide yes)
@@
 			(project "xt8086_beta"
 				(path "/8c0b3d8b-46d3-4173-ab1e-a61765f77d61"
-					(reference "#PWR015")
+					(reference "#PWR014")
 					(unit 1)
 				)
@@
 		(in_pos_files yes)
 		(dnp no)
-		(property "Reference" "#PWR010"
+		(property "Reference" "#PWR09"
 			(at 130.81 137.16 0)
 			(hide yes)
@@
 			(project "xt8086_beta"
 				(path "/8c0b3d8b-46d3-4173-ab1e-a61765f77d61"
-					(reference "#PWR010")
+					(reference "#PWR09")
 					(unit 1)
 				)
@@
 		(dnp no)
 		(fields_autoplaced yes)
-		(property "Reference" "#PWR08"
+		(property "Reference" "#PWR07"
 			(at 60.96 160.02 0)
 			(hide yes)
@@
 			(project "xt8086_beta"
 				(path "/8c0b3d8b-46d3-4173-ab1e-a61765f77d61"
-					(reference "#PWR08")
+					(reference "#PWR07")
 					(unit 1)
 				)
@@
 		(in_pos_files yes)
 		(dnp no)
-		(property "Reference" "#PWR013"
+		(property "Reference" "#PWR012"
 			(at 171.45 63.5 0)
 			(hide yes)
@@
 			(project "xt8086_beta"
 				(path "/8c0b3d8b-46d3-4173-ab1e-a61765f77d61"
-					(reference "#PWR013")
+					(reference "#PWR012")
 					(unit 1)
 				)
@@
 		(dnp no)
 		(fields_autoplaced yes)
-		(property "Reference" "R5"
+		(property "Reference" "R4"
 			(at 58.42 153.67 90)
 			(show_name no)
@@
 			(project "xt8086_beta"
 				(path "/8c0b3d8b-46d3-4173-ab1e-a61765f77d61"
-					(reference "R5")
+					(reference "R4")
 					(unit 1)
 				)
@@
 		(in_pos_files yes)
 		(dnp no)
-		(property "Reference" "#PWR017"
+		(property "Reference" "#PWR016"
 			(at 222.25 77.47 0)
 			(hide yes)
@@
 			(project "xt8086_beta"
 				(path "/8c0b3d8b-46d3-4173-ab1e-a61765f77d61"
-					(reference "#PWR017")
+					(reference "#PWR016")
 					(unit 1)
 				)
@@
 		(in_pos_files yes)
 		(dnp no)
-		(property "Reference" "#PWR018"
+		(property "Reference" "#PWR017"
 			(at 241.3 96.52 0)
 			(hide yes)
@@
 			(project "xt8086_beta"
 				(path "/8c0b3d8b-46d3-4173-ab1e-a61765f77d61"
-					(reference "#PWR018")
+					(reference "#PWR017")
 					(unit 1)
 				)
@@
 		(in_pos_files yes)
 		(dnp no)
-		(property "Reference" "#PWR022"
+		(property "Reference" "#PWR021"
 			(at 270.51 41.91 0)
 			(hide yes)
@@
 			(project "xt8086_beta"
 				(path "/8c0b3d8b-46d3-4173-ab1e-a61765f77d61"
-					(reference "#PWR022")
+					(reference "#PWR021")
 					(unit 1)
 				)
@@
 		(dnp no)
 		(fields_autoplaced yes)
-		(property "Reference" "#PWR016"
+		(property "Reference" "#PWR015"
 			(at 218.44 55.88 0)
 			(hide yes)
@@
 			(project "xt8086_beta"
 				(path "/8c0b3d8b-46d3-4173-ab1e-a61765f77d61"
-					(reference "#PWR016")
+					(reference "#PWR015")
 					(unit 1)
 				)
@@
 		(dnp no)
 		(fields_autoplaced yes)
-		(property "Reference" "#PWR023"
+		(property "Reference" "#PWR022"
 			(at 270.51 62.23 0)
 			(hide yes)
@@
 			(project "xt8086_beta"
 				(path "/8c0b3d8b-46d3-4173-ab1e-a61765f77d61"
-					(reference "#PWR023")
+					(reference "#PWR022")
 					(unit 1)
 				)
@@
 		(in_pos_files yes)
 		(dnp no)
-		(property "Reference" "#PWR09"
+		(property "Reference" "#PWR08"
 			(at 123.19 49.53 0)
 			(hide yes)
@@
 			(project "xt8086_beta"
 				(path "/8c0b3d8b-46d3-4173-ab1e-a61765f77d61"
-					(reference "#PWR09")
+					(reference "#PWR08")
 					(unit 1)
 				)
@@
 		(dnp no)
 		(fields_autoplaced yes)
-		(property "Reference" "LD3"
+		(property "Reference" "LD2"
 			(at 49.2125 153.67 0)
 			(show_name no)
@@
 			(project "xt8086_beta"
 				(path "/8c0b3d8b-46d3-4173-ab1e-a61765f77d61"
-					(reference "LD3")
+					(reference "LD2")
 					(unit 1)
 				)
@@
 		(in_pos_files yes)
 		(dnp no)
-		(property "Reference" "#PWR014"
+		(property "Reference" "#PWR013"
 			(at 176.53 44.45 0)
 			(hide yes)
@@
 			(project "xt8086_beta"
 				(path "/8c0b3d8b-46d3-4173-ab1e-a61765f77d61"
-					(reference "#PWR014")
+					(reference "#PWR013")
 					(unit 1)
 				)
@@
 		(dnp no)
 		(fields_autoplaced yes)
-		(property "Reference" "#PWR020"
+		(property "Reference" "#PWR019"
 			(at 241.3 101.6 0)
 			(hide yes)
@@
 			(project "xt8086_beta"
 				(path "/8c0b3d8b-46d3-4173-ab1e-a61765f77d61"
-					(reference "#PWR020")
+					(reference "#PWR019")
 					(unit 1)
 				)
@@
 		(in_pos_files yes)
 		(dnp no)
-		(property "Reference" "#PWR011"
+		(property "Reference" "#PWR010"
 			(at 133.35 83.82 0)
 			(hide yes)
@@
 			(project "xt8086_beta"
 				(path "/8c0b3d8b-46d3-4173-ab1e-a61765f77d61"
-					(reference "#PWR011")
+					(reference "#PWR010")
 					(unit 1)
 				)
@@
 		(dnp no)
 		(fields_autoplaced yes)
-		(property "Reference" "#PWR07"
+		(property "Reference" "#PWR06"
 			(at 40.64 160.02 0)
 			(hide yes)
@@
 			(project "xt8086_beta"
 				(path "/8c0b3d8b-46d3-4173-ab1e-a61765f77d61"
-					(reference "#PWR07")
+					(reference "#PWR06")
 					(unit 1)
 				)

Commit message: Board updates
Other:
- moved on the sheet: J2, JP1, JP2, JP3, LD2, R4

Commit message: Board updates
Parts:
- removed JP1: HDMI Audio, xt8086:SolderJumper-2_P1.3mm_Open_Pad1.0x1.5mm, symbol xt8086:Conn_01x02_Pin
- removed JP2: Jack In, xt8086:SolderJumper-2_P1.3mm_Open_Pad1.0x1.5mm, symbol xt8086:Conn_01x02_Pin
- removed JP3: Speaker In, xt8086:SolderJumper-2_P1.3mm_Open_Pad1.0x1.5mm, symbol xt8086:Conn_01x02_Pin
- removed S2: SS12D00, xt8086:Switch_Slide_SS12D00, symbol xt8086:SS12D00
- added S2: DS05-127-2-03BK-SMT-TR, xt8086:SW_DIP_DS05-127-2-03BK-SMT, symbol xt8086:DS05-127-2-03BK-SMT-TR
Connections:
- net GND: now also U1.11 (5A), U1.13 (6A), U1.3 (2A), U1.5 (3A), U1.9 (4A), U2.11 (CLK2), U2.12 (D2)
- net HDMI_AUDIO: now also S2.2 (NO_1)
- net SPEAKER: now also S2.1 (COM_1), S2.3 (COM_2), S2.5 (COM_3)
- net VBUS: now also U2.10 (PR2), U2.13 (CLR2)
- new net JACK_IN: S2.4 (NO_2)
- new net SPK_IN: S2.6 (NO_3)
- no-connect marks 23 -> 13
Other:
- sheet Video ports: added none; removed VGA_GND
- moved on the sheet: C4, J2

Commit message: Board updates
Parts:
- renumbered LD1 to D1, LD2 to D2
Other:
- moved on the sheet: C1, C2, C3, C4, D1, D2, J1, J2, R1, R2, R3, R4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

Commit message: feat: xt8086_beta gets Dino's sound and schematic changes
xt8086_beta and dino_z80 share their platform, so everything done to the
Dino schematic is carried over:

- Buzzer sheet replaced by Dino's Sound + Speaker sheets: LM358 line out,
  PAM8403 driving a CVS-2308 speaker, S2 as HDMI L/R + speaker enable,
  stereo HDMI audio (AUDIO_IN_L/R no longer tied together).
- GP46 is PWM_L, GP44 is PWM_R, exactly as on Dino; J1 (UART) is gone
  and GP45 is left unconnected.
- USB defaults to the RP2350: R3 pulls SW low, S1's common goes to +3V3,
  JP3 (USB Test) straps SW high.
- H1-H4 become 2.5 mm pad-and-via holes tied to GND.
- MS9288A footprint renamed QFN-48_6x6mm.
- Shared sheets take Dino's current versions with xt8086_beta's own
  references; SI values, X1 renamed Y2, datasheet links fixed, plus TI
  SN74LS74A and Analog Devices DS3231M links for xt-only parts.
- Libraries: PAM8403D, LM358, CVS-2308, MountingHole_Pad symbols and
  their footprints/3D models; SOT-23 pad mirror fix and SOIC-8 from Dino.

dino.kicad_sym also gains CVS-2308 and MountingHole_Pad, which Dino's
schematic had only in its symbol cache.

ERC: 0. The board is not updated yet.
Parts:
- removed J1: UART, xt8086:JST_SH_1x03_P1.00mm_Vertical, symbol xt8086:Conn_01x03_Pin
- removed S2: DS05-127-2-03BK-SMT-TR, xt8086:SW_DIP_DS05-127-2-03BK-SMT, symbol xt8086:DS05-127-2-03BK-SMT-TR
- added JP3: USB Test, xt8086:SolderJumper-2_P1.3mm_Open_Pad1.0x1.5mm, symbol xt8086:SolderJumper_2_Open
- C1, C4: value 100u -> 100µF
- C2, C3: value 100n -> 100nF
- H1, H2, H3, H4: value Hole 2.7mm -> Hole 2.5mm; footprint xt8086:MountingHole_2.7mm -> xt8086:MountingHole_2.5mm_Pad_Via; symbol xt8086:MountingHole -> xt8086:MountingHole_Pad
- R1, R2: value 1K -> 1kΩ
- R3, R4: value 1K -> 1kΩ; AliExpress https://www.vishay.com/docs/28952/mcs0402at-mct0603at-mcu08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 -> (none)
Connections:
- net +3V3: now also S1.2, JP3.1 (A)
- net GND: now also H1.1, H2.1, H3.1, H4.1; no longer S1.2
- net USB, Power/SW: now also JP3.2 (B)
- no-connect marks 13 -> 14
Other:
- removed sheet Audio
- added sheet Sound (sound.kicad_sch)

Commit message: feat: xt8086_beta board takes Dino's layout; courtyards on every footprint
xt8086_beta board:
- Synced to the new schematic: buzzer, UART J1 and the old S2 are gone;
  the Sound/Speaker parts, JP3 and the pad-and-via holes are placed as
  on Dino, and Dino's decoupling moves, label positions and board texts
  are carried over.
- Speaker 1.8 mm lower than on Dino to clear the lower 8086 socket; the
  PWM filter column, C104, D1, C106 and JP3 moved to make room.
- Sound nets, SD lines near the socket, VSIN, the LED line and a few GND
  ties rerouted around the 8086 bus. J5 (SWD) placed by hand.
- Overlapping VBUS zones on In2 given distinct priorities.
- JP3 moved off S1's through-hole pins.

Both boards:
- Battery_CR1220 (xt), Button_SMD_3x4x2mm, HDMI_Female and
  USB_C_Receptacle had no courtyard, so nothing was checked against them.
  They get one: the battery follows the holder's contour, buttons +0.25 mm,
  connectors +0.5 mm.

DRC (all severities): no errors, 0 unconnected, 0 schematic parity on
both boards; no through-hole pin under an opposite-side part.
Other:
- moved on the sheet: H1, H2, H3, H4

Commit message: feat: compact rounded solder jumpers and debug jumpers across S2
- all solder jumpers use a compact rounded footprint
  (SolderJumper-2_P1.0mm_Open_RoundedPad0.7x1.0mm: 0.7x1.0 mm pads,
  0.3 mm gap), scaled from KiCad's stock RoundedPad jumper
- JP4/JP5/JP6 (Audio L, Audio R, Speaker) bridge each S2 position, on
  the back under S2, so the DIP switch can be left unfitted
- JP3 on Dino gets short tracks to its vias, which the smaller pads no
  longer cover
Parts:
- JP3: footprint xt8086:SolderJumper-2_P1.3mm_Open_Pad1.0x1.5mm -> xt8086:SolderJumper-2_P1.0mm_Open_RoundedPad0.7x1.0mm
Changed lines of the file:
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@@
 			)
 		)
-		(property "Footprint" "xt8086:SolderJumper-2_P1.3mm_Open_Pad1.0x1.5mm"
+		(property "Footprint" "xt8086:SolderJumper-2_P1.0mm_Open_RoundedPad0.7x1.0mm"
 			(at 124.46 41.91 0)
 			(hide yes)
