File: xt8086_beta/rp2350b.kicad_sch (KiCad schematic)
At the start: 31 parts, among them J6 Debug, U10 ESP-PSRAM64, U6 RP2350B, U8 W25Q128JVPIQ, Y1 ASE-12MHz

Commit message: Board updates
Parts:
- U8: renamed from U10; value ESP-PSRAM64 -> ESP-PSRAM64H
- renumbered C15 to C14, C19 to C15, C21 to C16, C24 to C17, C25 to C18, C26 to C19, C27 to C20, C30 to C21, C34 to C22, C35 to C23, C36 to C24, C37 to C25, R8 to R10, R14 to R11, R15 to R12, R17 to R13, R18 to R14, R19 to R15, R7 to R9, U8 to U7

Commit message: Board updates
Parts:
- renumbered R11 to R10, R12 to R11, R13 to R12, R14 to R13, R15 to R14, R9 to R8, R10 to R9
Changed lines of the file:
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@@
 		(in_pos_files yes)
 		(dnp no)
-		(property "Reference" "#PWR059"
+		(property "Reference" "#PWR058"
 			(at 222.25 115.57 0)
 			(hide yes)
@@
 			(project "xt8086_beta"
 				(path "/8c0b3d8b-46d3-4173-ab1e-a61765f77d61/69d580d4-830a-4ad1-89c3-268c1b1da372"
-					(reference "#PWR059")
+					(reference "#PWR058")
 					(unit 1)
 				)
@@
 		(dnp no)
 		(fields_autoplaced yes)
-		(property "Reference" "#PWR050"
+		(property "Reference" "#PWR049"
 			(at 71.12 128.27 0)
 			(hide yes)
@@
 			(project "xt8086_beta"
 				(path "/8c0b3d8b-46d3-4173-ab1e-a61765f77d61/69d580d4-830a-4ad1-89c3-268c1b1da372"
-					(reference "#PWR050")
+					(reference "#PWR049")
 					(unit 1)
 				)
@@
 		(in_pos_files yes)
 		(dnp no)
-		(property "Reference" "#PWR052"
+		(property "Reference" "#PWR051"
 			(at 104.14 20.32 0)
 			(hide yes)
@@
 			(project "xt8086_beta"
 				(path "/8c0b3d8b-46d3-4173-ab1e-a61765f77d61/69d580d4-830a-4ad1-89c3-268c1b1da372"
-					(reference "#PWR052")
+					(reference "#PWR051")
 					(unit 1)
 				)
@@
 		(in_pos_files yes)
 		(dnp no)
-		(property "Reference" "#PWR044"
+		(property "Reference" "#PWR043"
 			(at 36.83 39.37 0)
 			(hide yes)
@@
 			(project "xt8086_beta"
 				(path "/8c0b3d8b-46d3-4173-ab1e-a61765f77d61/69d580d4-830a-4ad1-89c3-268c1b1da372"
-					(reference "#PWR044")
+					(reference "#PWR043")
 					(unit 1)
 				)
@@
 		(in_pos_files yes)
 		(dnp no)
-		(property "Reference" "#PWR061"
+		(property "Reference" "#PWR060"
 			(at 261.62 50.8 0)
 			(hide yes)
@@
 			(project "xt8086_beta"
 				(path "/8c0b3d8b-46d3-4173-ab1e-a61765f77d61/69d580d4-830a-4ad1-89c3-268c1b1da372"
-					(reference "#PWR061")
+					(reference "#PWR060")
 					(unit 1)
 				)
@@
 		(in_pos_files yes)
 		(dnp no)
-		(property "Reference" "R11"
+		(property "Reference" "R10"
 			(at 182.88 49.53 90)
 			(show_name no)
@@
 			(project "xt8086_beta"
 				(path "/8c0b3d8b-46d3-4173-ab1e-a61765f77d61/69d580d4-830a-4ad1-89c3-268c1b1da372"
-					(reference "R11")
+					(reference "R10")
 					(unit 1)
 				)
@@
 		(in_pos_files yes)
 		(dnp no)
-		(property "Reference" "R10"
+		(property "Reference" "R9"
 			(at 73.66 67.1322 90)
 			(show_name no)
@@
 			(project "xt8086_beta"
 				(path "/8c0b3d8b-46d3-4173-ab1e-a61765f77d61/69d580d4-830a-4ad1-89c3-268c1b1da372"
-					(reference "R10")
+					(reference "R9")
 					(unit 1)
 				)
@@
 		(in_pos_files yes)
 		(dnp no)
-		(property "Reference" "R15"
+		(property "Reference" "R14"
 			(at 264.0584 151.638 0)
 			(hide yes)
@@
 			(project "xt8086_beta"
 				(path "/8c0b3d8b-46d3-4173-ab1e-a61765f77d61/69d580d4-830a-4ad1-89c3-268c1b1da372"
-					(reference "R15")
+					(reference "R14")
 					(unit 1)
 				)
@@
 		(in_pos_files yes)
 		(dnp no)
-		(property "Reference" "#PWR048"
+		(property "Reference" "#PWR047"
 			(at 46.99 54.61 0)
 			(hide yes)
@@
 			(project "xt8086_beta"
 				(path "/8c0b3d8b-46d3-4173-ab1e-a61765f77d61/69d580d4-830a-4ad1-89c3-268c1b1da372"
-					(reference "#PWR048")
+					(reference "#PWR047")
 					(unit 1)
 				)
@@
 		(in_pos_files yes)
 		(dnp no)
-		(property "Reference" "#PWR057"
+		(property "Reference" "#PWR056"
 			(at 200.66 139.7 0)
 			(hide yes)
@@
 			(project "xt8086_beta"
 				(path "/8c0b3d8b-46d3-4173-ab1e-a61765f77d61/69d580d4-830a-4ad1-89c3-268c1b1da372"
-					(reference "#PWR057")
+					(reference "#PWR056")
 					(unit 1)
 				)
@@
 		(in_pos_files yes)
 		(dnp no)
-		(property "Reference" "#PWR055"
+		(property "Reference" "#PWR054"
 			(at 189.23 137.16 0)
 			(hide yes)
@@
 			(project "xt8086_beta"
 				(path "/8c0b3d8b-46d3-4173-ab1e-a61765f77d61/69d580d4-830a-4ad1-89c3-268c1b1da372"
-					(reference "#PWR055")
+					(reference "#PWR054")
 					(unit 1)
 				)
@@
 		(dnp no)
 		(fields_autoplaced yes)
-		(property "Reference" "#PWR047"
+		(property "Reference" "#PWR046"
 			(at 38.1 114.3 0)
 			(hide yes)
@@
 			(project "xt8086_beta"
 				(path "/8c0b3d8b-46d3-4173-ab1e-a61765f77d61/69d580d4-830a-4ad1-89c3-268c1b1da372"
-					(reference "#PWR047")
+					(reference "#PWR046")
 					(unit 1)
 				)
@@
 		(in_pos_files yes)
 		(dnp no)
-		(property "Reference" "#PWR054"
+		(property "Reference" "#PWR053"
 			(at 147.32 31.75 0)
 			(hide yes)
@@
 			(project "xt8086_beta"
 				(path "/8c0b3d8b-46d3-4173-ab1e-a61765f77d61/69d580d4-830a-4ad1-89c3-268c1b1da372"
-					(reference "#PWR054")
+					(reference "#PWR053")
 					(unit 1)
 				)
@@
 		(in_pos_files yes)
 		(dnp no)
-		(property "Reference" "R12"
+		(property "Reference" "R11"
 			(at 182.88 54.864 90)
 			(show_name no)
@@
 			(project "xt8086_beta"
 				(path "/8c0b3d8b-46d3-4173-ab1e-a61765f77d61/69d580d4-830a-4ad1-89c3-268c1b1da372"
-					(reference "R12")
+					(reference "R11")
 					(unit 1)
 				)
@@
 		(dnp no)
 		(fields_autoplaced yes)
-		(property "Reference" "#PWR060"
+		(property "Reference" "#PWR059"
 			(at 233.68 74.93 0)
 			(hide yes)
@@
 			(project "xt8086_beta"
 				(path "/8c0b3d8b-46d3-4173-ab1e-a61765f77d61/69d580d4-830a-4ad1-89c3-268c1b1da372"
-					(reference "#PWR060")
+					(reference "#PWR059")
 					(unit 1)
 				)
@@
 		(in_pos_files yes)
 		(dnp no)
-		(property "Reference" "#PWR058"
+		(property "Reference" "#PWR057"
 			(at 201.93 105.41 0)
 			(hide yes)
@@
 			(project "xt8086_beta"
 				(path "/8c0b3d8b-46d3-4173-ab1e-a61765f77d61/69d580d4-830a-4ad1-89c3-268c1b1da372"
-					(reference "#PWR058")
+					(reference "#PWR057")
 					(unit 1)
 				)
@@
 		(in_pos_files yes)
 		(dnp no)
-		(property "Reference" "#PWR046"
+		(property "Reference" "#PWR045"
 			(at 38.1 83.82 0)
 			(hide yes)
@@
 			(project "xt8086_beta"
 				(path "/8c0b3d8b-46d3-4173-ab1e-a61765f77d61/69d580d4-830a-4ad1-89c3-268c1b1da372"
-					(reference "#PWR046")
+					(reference "#PWR045")
 					(unit 1)
 				)
@@
 		(in_pos_files yes)
 		(dnp no)
-		(property "Reference" "#PWR045"
+		(property "Reference" "#PWR044"
 			(at 35.56 73.66 0)
 			(hide yes)
@@
 			(project "xt8086_beta"
 				(path "/8c0b3d8b-46d3-4173-ab1e-a61765f77d61/69d580d4-830a-4ad1-89c3-268c1b1da372"
-					(reference "#PWR045")
+					(reference "#PWR044")
 					(unit 1)
 				)
@@
 		(in_pos_files yes)
 		(dnp no)
-		(property "Reference" "#PWR049"
+		(property "Reference" "#PWR048"
 			(at 62.23 30.48 0)
 			(hide yes)
@@
 			(project "xt8086_beta"
 				(path "/8c0b3d8b-46d3-4173-ab1e-a61765f77d61/69d580d4-830a-4ad1-89c3-268c1b1da372"
-					(reference "#PWR049")
+					(reference "#PWR048")
 					(unit 1)
 				)
@@
 		(in_pos_files yes)
 		(dnp no)
-		(property "Reference" "R13"
+		(property "Reference" "R12"
 			(at 191.9478 147.32 90)
 			(show_name no)
@@
 			(project "xt8086_beta"
 				(path "/8c0b3d8b-46d3-4173-ab1e-a61765f77d61/69d580d4-830a-4ad1-89c3-268c1b1da372"
-					(reference "R13")
+					(reference "R12")
 					(unit 1)
 				)
@@
 		(in_pos_files yes)
 		(dnp no)
-		(property "Reference" "R9"
+		(property "Reference" "R8"
 			(at 68.6816 37.592 0)
 			(show_name no)
@@
 			(project "xt8086_beta"
 				(path "/8c0b3d8b-46d3-4173-ab1e-a61765f77d61/69d580d4-830a-4ad1-89c3-268c1b1da372"
-					(reference "R9")
+					(reference "R8")
 					(unit 1)
 				)
@@
 		(in_pos_files yes)
 		(dnp no)
-		(property "Reference" "#PWR053"
+		(property "Reference" "#PWR052"
 			(at 125.73 196.85 0)
 			(hide yes)
@@
 			(project "xt8086_beta"
 				(path "/8c0b3d8b-46d3-4173-ab1e-a61765f77d61/69d580d4-830a-4ad1-89c3-268c1b1da372"
-					(reference "#PWR053")
+					(reference "#PWR052")
 					(unit 1)
 				)
@@
 		(in_pos_files yes)
 		(dnp no)
-		(property "Reference" "#PWR056"
+		(property "Reference" "#PWR055"
 			(at 203.2 130.81 0)
 			(hide yes)
@@
 			(project "xt8086_beta"
 				(path "/8c0b3d8b-46d3-4173-ab1e-a61765f77d61/69d580d4-830a-4ad1-89c3-268c1b1da372"
-					(reference "#PWR056")
+					(reference "#PWR055")
 					(unit 1)
 				)
@@
 		(in_pos_files yes)
 		(dnp no)
-		(property "Reference" "R14"
+		(property "Reference" "R13"
 			(at 246.5578 81.28 90)
 			(show_name no)
@@
 			(project "xt8086_beta"
 				(path "/8c0b3d8b-46d3-4173-ab1e-a61765f77d61/69d580d4-830a-4ad1-89c3-268c1b1da372"
-					(reference "R14")
+					(reference "R13")
 					(unit 1)
 				)
@@
 		(in_pos_files yes)
 		(dnp no)
-		(property "Reference" "#PWR051"
+		(property "Reference" "#PWR050"
 			(at 81.28 55.88 0)
 			(hide yes)
@@
 			(project "xt8086_beta"
 				(path "/8c0b3d8b-46d3-4173-ab1e-a61765f77d61/69d580d4-830a-4ad1-89c3-268c1b1da372"
-					(reference "#PWR051")
+					(reference "#PWR050")
 					(unit 1)
 				)

Commit message: Board updates
Changed lines of the file:
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@@
 	(wire
 		(pts
-			(xy 55.88 114.3) (xy 93.98 114.3)
+			(xy 87.63 114.3) (xy 93.98 114.3)
 		)
 		(stroke
@@
 	)
 	(sheet
-		(at 43.18 111.76)
+		(at 74.93 111.76)
 		(size 12.7 5.08)
 		(exclude_from_sim no)
@@
 		)
 		(property "Sheetname" "Reset"
-			(at 43.18 111.0484 0)
+			(at 74.93 111.0484 0)
 			(show_name no)
 			(do_not_autoplace no)
@@
 		)
 		(property "Sheetfile" "reset.kicad_sch"
-			(at 43.18 117.4246 0)
+			(at 74.93 117.4246 0)
 			(hide yes)
 			(show_name no)
@@
 		)
 		(pin "RESET" input
-			(at 55.88 114.3 0)
+			(at 87.63 114.3 0)
 			(effects
 				(font

Commit message: Board updates
Parts:
- added TP1: +1V1, xt8086:TestPoint_Pad_1.0x1.0mm, symbol xt8086:TestPoint
- renumbered C8 to C12, C9 to C13, C10 to C14, C11 to C15, C12 to C16, C13 to C17, C14 to C18, C15 to C19, C16 to C20, C17 to C21, C18 to C22, C19 to C23, C20 to C24, C21 to C25, C22 to C26, C23 to C27, C24 to C28, C25 to C29, R9 to R10, R10 to R11, R11 to R12, R12 to R13, R13 to R14, R14 to R15, R8 to R9
Connections:
- net +1V1: now also TP1.1

Commit message: Board updates
Parts:
- renumbered J6 to J5, Y1 to X1
Changed lines of the file:
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@@
 		(in_pos_files yes)
 		(dnp no)
-		(property "Reference" "J6"
+		(property "Reference" "J5"
 			(at 93.218 134.366 0)
 			(show_name no)
@@
 			(project "xt8086_beta"
 				(path "/8c0b3d8b-46d3-4173-ab1e-a61765f77d61/69d580d4-830a-4ad1-89c3-268c1b1da372"
-					(reference "J6")
+					(reference "J5")
 					(unit 1)
 				)
@@
 		(dnp no)
 		(fields_autoplaced yes)
-		(property "Reference" "Y1"
+		(property "Reference" "X1"
 			(at 68.58 90.0998 0)
 			(show_name no)
@@
 			(project "xt8086_beta"
 				(path "/8c0b3d8b-46d3-4173-ab1e-a61765f77d61/69d580d4-830a-4ad1-89c3-268c1b1da372"
-					(reference "Y1")
+					(reference "X1")
 					(unit 1)
 				)

Commit message: feat: xt8086_beta gets Dino's sound and schematic changes
xt8086_beta and dino_z80 share their platform, so everything done to the
Dino schematic is carried over:

- Buzzer sheet replaced by Dino's Sound + Speaker sheets: LM358 line out,
  PAM8403 driving a CVS-2308 speaker, S2 as HDMI L/R + speaker enable,
  stereo HDMI audio (AUDIO_IN_L/R no longer tied together).
- GP46 is PWM_L, GP44 is PWM_R, exactly as on Dino; J1 (UART) is gone
  and GP45 is left unconnected.
- USB defaults to the RP2350: R3 pulls SW low, S1's common goes to +3V3,
  JP3 (USB Test) straps SW high.
- H1-H4 become 2.5 mm pad-and-via holes tied to GND.
- MS9288A footprint renamed QFN-48_6x6mm.
- Shared sheets take Dino's current versions with xt8086_beta's own
  references; SI values, X1 renamed Y2, datasheet links fixed, plus TI
  SN74LS74A and Analog Devices DS3231M links for xt-only parts.
- Libraries: PAM8403D, LM358, CVS-2308, MountingHole_Pad symbols and
  their footprints/3D models; SOT-23 pad mirror fix and SOIC-8 from Dino.

dino.kicad_sym also gains CVS-2308 and MountingHole_Pad, which Dino's
schematic had only in its symbol cache.

ERC: 0. The board is not updated yet.
Parts:
- C12, C14, C16, C17: value 4.7u -> 4.7µF
- C13, C15, C18, C19, C20, C21, C22, C23, C24, C25, C26, C27, C28, C29: value 100n -> 100nF
- J5: AliExpress https://www.aliexpress.com/item/1005007039504981.html -> (none)
- L1: value 3.3u -> 3.3µH
- R10: value 1K -> 1kΩ
- R11, R12: value 27R -> 27Ω
- R13, R14: value 10K -> 10kΩ; AliExpress https://www.vishay.com/docs/28952/mcs0402at-mct0603at-mcu08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 -> (none)
- R15: value 0R -> 0Ω
- R9: value 33R -> 33Ω
- Y2: renamed from X1; value ASE-12MHz -> 12MHz
Changed lines of the file:
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@@
 			)
 		)
-		(property "Value" "3.3u"
+		(property "Value" "3.3µH"
 			(at 63.5 58.42 0)
 			(show_name no)
@@
 			)
 		)
-		(property "Value" "4.7u"
+		(property "Value" "4.7µF"
 			(at 85.471 26.543 0)
 			(show_name no)
@@
 			)
 		)
-		(property "Value" "27R"
+		(property "Value" "27Ω"
 			(at 172.72 49.53 90)
 			(show_name no)
@@
 			)
 		)
-		(property "Value" "1K"
+		(property "Value" "1kΩ"
 			(at 73.66 69.4436 90)
 			(show_name no)
@@
 			)
 		)
-		(property "Value" "100n"
+		(property "Value" "100nF"
 			(at 230.251 36.703 0)
 			(show_name no)
@@
 			)
 		)
-		(property "Value" "100n"
+		(property "Value" "100nF"
 			(at 184.531 36.703 0)
 			(show_name no)
@@
 			)
 		)
-		(property "Value" "0R"
+		(property "Value" "0Ω"
 			(at 261.747 151.638 0)
 			(show_name no)
@@
 			)
 		)
-		(property "Value" "100n"
+		(property "Value" "100nF"
 			(at 207.391 36.703 0)
 			(show_name no)
@@
 			)
 		)
-		(property "Value" "4.7u"
+		(property "Value" "4.7µF"
 			(at 39.37 58.42 0)
 			(show_name no)
@@
 			)
 		)
-		(property "Value" "100n"
+		(property "Value" "100nF"
 			(at 218.821 36.703 0)
 			(show_name no)
@@
 			)
 		)
-		(property "Value" "100n"
+		(property "Value" "100nF"
 			(at 253.111 36.703 0)
 			(show_name no)
@@
 			)
 		)
-		(property "Value" "4.7u"
+		(property "Value" "4.7µF"
 			(at 85.09 45.72 0)
 			(show_name no)
@@
 			)
 		)
-		(property "Value" "100n"
+		(property "Value" "100nF"
 			(at 96.901 26.543 0)
 			(show_name no)
@@
 			)
 		)
-		(property "Value" "100n"
+		(property "Value" "100nF"
 			(at 195.961 36.703 0)
 			(show_name no)
@@
 			)
 		)
-		(property "Value" "100n"
+		(property "Value" "100nF"
 			(at 204.851 92.583 0)
 			(show_name no)
@@
 			)
 		)
-		(property "Value" "100n"
+		(property "Value" "100nF"
 			(at 241.681 36.703 0)
 			(show_name no)
@@
 			)
 		)
-		(property "Value" "100n"
+		(property "Value" "100nF"
 			(at 172.466 36.703 0)
 			(show_name no)
@@
 			)
 		)
-		(property "Value" "100n"
+		(property "Value" "100nF"
 			(at 264.541 36.703 0)
 			(show_name no)
@@
 			)
 		)
-		(property "Datasheet" ""
+		(property "Datasheet" "https://datasheets.raspberrypi.com/rp2350/rp2350-datasheet.pdf"
 			(at 106.68 93.98 0)
 			(hide yes)
@@
 			)
 		)
-		(property "Value" "100n"
+		(property "Value" "100nF"
 			(at 74.041 26.543 0)
 			(show_name no)
@@
 			)
 		)
-		(property "Value" "100n"
+		(property "Value" "100nF"
 			(at 192.913 127.889 0)
 			(show_name no)
@@
 			)
 		)
-		(property "Value" "27R"
+		(property "Value" "27Ω"
 			(at 172.466 54.864 90)
 			(show_name no)
@@
 			)
 		)
-		(property "Value" "4.7u"
+		(property "Value" "4.7µF"
 			(at 50.8 58.42 0)
 			(show_name no)
@@
 			)
 		)
-		(property "Value" "100n"
+		(property "Value" "100nF"
 			(at 30.48 93.9769 0)
 			(show_name no)
@@
 			)
 		)
-		(property "Datasheet" "https://www.mouser.com/datasheet/2/154/basics-us_2-54mm-125848.pdf"
+		(property "Datasheet" "https://www.jst-mfg.com/product/pdf/eng/eSH.pdf"
 			(at 82.55 128.27 0)
 			(hide yes)
@@
 			)
 		)
-		(property "AliExpress" "https://www.aliexpress.com/item/1005007039504981.html"
+		(property "AliExpress" ""
 			(at 82.55 128.27 0)
 			(hide yes)
@@
 			)
 		)
-		(property "Value" "10K"
+		(property "Value" "10kΩ"
 			(at 189.6364 147.32 90)
 			(show_name no)
@@
 			)
 		)
-		(property "Datasheet" ""
+		(property "Datasheet" "https://www.vishay.com/docs/28952/mcs0402at-mct0603at-mcu0805at-mca1206at.pdf"
 			(at 186.69 147.32 0)
 			(hide yes)
@@
 			)
 		)
-		(property "AliExpress" "https://www.vishay.com/docs/28952/mcs0402at-mct0603at-mcu0805at-mca1206at.pdf"
+		(property "AliExpress" ""
 			(at 186.69 147.32 0)
 			(hide yes)
@@
 			)
 		)
-		(property "Value" "33R"
+		(property "Value" "33Ω"
 			(at 70.993 37.592 0)
 			(show_name no)
@@
 			)
 		)
-		(property "Value" "10K"
+		(property "Value" "10kΩ"
 			(at 244.2464 81.28 90)
 			(show_name no)
@@
 			)
 		)
-		(property "Datasheet" ""
+		(property "Datasheet" "https://www.vishay.com/docs/28952/mcs0402at-mct0603at-mcu0805at-mca1206at.pdf"
 			(at 241.3 81.28 0)
 			(hide yes)
@@
 			)
 		)
-		(property "AliExpress" "https://www.vishay.com/docs/28952/mcs0402at-mct0603at-mcu0805at-mca1206at.pdf"
+		(property "AliExpress" ""
 			(at 241.3 81.28 0)
 			(hide yes)
@@
 		(dnp no)
 		(fields_autoplaced yes)
-		(property "Reference" "X1"
+		(property "Reference" "Y2"
 			(at 68.58 90.0998 0)
 			(show_name no)
@@
 			)
 		)
-		(property "Value" "ASE-12MHz"
+		(property "Value" "12MHz"
 			(at 68.58 92.6398 0)
 			(show_name no)
@@
 			)
 		)
-		(property "Datasheet" "http://www.abracon.com/Oscillators/ASV.pdf"
+		(property "Datasheet" "https://abracon.com/Oscillators/ASEseries.pdf"
 			(at 53.34 96.52 0)
 			(hide yes)
@@
 			(project "xt8086_beta"
 				(path "/8c0b3d8b-46d3-4173-ab1e-a61765f77d61/69d580d4-830a-4ad1-89c3-268c1b1da372"
-					(reference "X1")
+					(reference "Y2")
 					(unit 1)
 				)

Commit message: feat: round test points on dino_z80 and xt8086_beta
Test points use the 1.0 mm round TestPoint_Pad_D1.0mm instead of the
square pad; placement, nets and labels are unchanged. Also includes the
latest xt8086_beta edits on the power, sound and speaker sheets and board.
Parts:
- TP1: footprint xt8086:TestPoint_Pad_1.0x1.0mm -> xt8086:TestPoint_Pad_D1.0mm
Changed lines of the file:
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@@
 			)
 		)
-		(property "Footprint" "xt8086:TestPoint_Pad_1.0x1.0mm"
+		(property "Footprint" "xt8086:TestPoint_Pad_D1.0mm"
 			(at 49.53 134.62 0)
 			(hide yes)

Commit message: fix: board review round - protection, pull-ups, parts data
- MS9288A config I2C pull-ups (SCL/SDA) go to +3V3; the chip's pins
  are rated only to DVDD33 + 0.5 V, and the reference leaves them open
- MS9288A audio inputs: 0 Ohm series + 10 kOhm shunt (not fitted) ahead
  of the coupling caps, so the reference 1/2 divider can be fitted later
- HDMI +5 V pin: 0.2 A resettable fuse (F2, 0603) in series with D5
- SD card: 10 kOhm pull-ups on CMD, DAT0 and DAT3 (SPI mode)
- xt8086: U1 is a 74HCT04 buffering GP29 to a 5 V 8086 CLK; RESET gets a
  10 kOhm pull-up so the CPU is held in reset until the RP2350 drives it
- video ladder and headphone series resistors 400/800 -> 402/806 Ohm
- LCSC part numbers checked against JLC for 452 parts; wrong numbers on
  R57, the 4.7 uF caps and the USB-C connector fixed
- MS9288A symbol: pin 3 is NC, datasheet linked; CD4069 pin name fixed
- Dino board follows the schematic renumbering; label and via clean-up
Parts:
- C12, C14, C16, C17: LCSC (none) -> C19666
- C13, C15, C18, C19, C20, C21, C22, C23, C24, C25, C26, C27, C28, C29: LCSC (none) -> C14663
- J5: LCSC (none) -> C160389
- L1: LCSC (none) -> C42411119
- R10: LCSC (none) -> C21190
- R11, R12: LCSC (none) -> C2907021
- R13, R14: LCSC (none) -> C25804
- R15: LCSC (none) -> C21189
- R9: LCSC (none) -> C23140
- U6: LCSC (none) -> C42415655
- U7: LCSC (none) -> C190862
- U8: LCSC (none) -> C5333729
- Y2: LCSC (none) -> C7503129
