File: xt8086_beta/usb.kicad_sch (KiCad schematic)
At the start: 23 parts, among them J7 USB4215-03-A, J8 SS-52100-004, U10 TPS2116DRL, U11 AMS1117-3.3, U12 USBLC6-2SC6, U13 USBLC6-2SC6, U9 USBLC6-2SC6

Commit message: Board updates
Parts:
- removed U11: AMS1117-3.3, xt8086:SOT-223-3_TabPin2, symbol xt8086:AMS1117-3.3
- added C31: 100n, xt8086:C_0603_1608Metric, symbol xt8086:C
- C38: renamed from C33; footprint xt8086:C_Radial_D6.3mm_P2.50mm -> xt8086:C_1206_3216Metric; symbol xt8086:C_Polarized_Small -> xt8086:C_Small
- renumbered C26 to C30, C27 to C32, C28 to C33, C29 to C34, C30 to C35, C31 to C36, C32 to C37, C34 to C39, C35 to C40, C36 to C41, JP5 to JP1, R15 to R16, R16 to R17, R17 to R18, R18 to R19, U12 to U11, U13 to U12
Connections:
- net GND: now also C31.1
- net VBUS: no longer C32.2, C34.2, C40.1, C41.1, J8.1 (VBUS1), J8.5 (VBUS2), JP1.1 (Pin_1), R18.2, U10.3 (VIN1), U10.5 (MODE)
- net +5V_LOGIC renamed +5V_SEL
- net +5V_SEL: now also C31.2
- new net +5V_DC: C32.2, C34.2, JP1.1 (Pin_1), R18.2, U10.3 (VIN1), U10.5 (MODE)
- new net VBUS_P1: C40.1, J8.1 (VBUS1)
- new net VBUS_P2: C41.1, J8.5 (VBUS2)
- no-connect marks 8 -> 7
Other:
- added sheet 3V3 Buck (buck3v3.kicad_sch)
- added sheet USB-A Port Power (usb_a_power.kicad_sch)
- moved on the sheet: C36, C37, C39

Commit message: Board updates
Parts:
- added R54: 1M, xt8086:R_0603_1608Metric, symbol xt8086:R
- C36: footprint xt8086:C_Radial_D6.3mm_P2.50mm -> xt8086:CP_Radial_D6.3mm_P2.50mm
Connections:
- net at R18.1, R19.2, U10.4 (PR1): now also R54.2
- net ST: now reaches U10.8 (ST)
- net ST: now also R54.1
- no-connect marks 7 -> 6
Other:
- note added: "(matches frank_next R56)."
- note added: "R54: TPS2116 ST -> PR1 hysteresis"
Changed lines of the file:
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@@
 	)
 	(no_connect
-		(at 127 134.62)
-	)
-	(no_connect
 		(at 52.07 77.47)
 	)
@@
 			)
 		)
-		(property "Footprint" "xt8086:C_Radial_D6.3mm_P2.50mm"
+		(property "Footprint" "xt8086:CP_Radial_D6.3mm_P2.50mm"
 			(at 163.83 133.35 0)
 			(hide yes)
@@
 		)
 	)
+	(wire
+		(pts
+			(xy 127.0 134.62) (xy 134.62 134.62)
+		)
+		(stroke
+			(width 0)
+			(type default)
+		)
+	)
+	(label "ST"
+		(at 134.62 134.62 0)
+		(effects
+				(font
+					(size 1.27 1.27)
+				)
+				(justify left bottom)
+			)
+	)
+	(symbol
+		(lib_id "xt8086:R")
+		(at 72.39 127.0 90)
+		(unit 1)
+		(body_style 1)
+		(exclude_from_sim no)
+		(in_bom yes)
+		(on_board yes)
+		(in_pos_files yes)
+		(dnp no)
+		(property "Reference" "R54"
+			(at 72.39 121.92 90)
+			(show_name no)
+			(do_not_autoplace no)
+			(effects
+				(font
+					(size 1.27 1.27)
+				)
+			)
+		)
+		(property "Value" "1M"
+			(at 72.39 124.46 90)
+			(show_name no)
+			(do_not_autoplace no)
+			(effects
+				(font
+					(size 1.27 1.27)
+				)
+			)
+		)
+		(property "Footprint" "xt8086:R_0603_1608Metric"
+			(at 72.39 127.0 0)
+			(hide yes)
+			(show_name no)
+			(do_not_autoplace no)
+			(effects
+				(font
+					(size 1.27 1.27)
+				)
+			)
+		)
+		(property "Datasheet" ""
+			(at 72.39 127.0 0)
+			(hide yes)
+			(show_name no)
+			(do_not_autoplace no)
+			(effects
+				(font
+					(size 1.27 1.27)
+				)
+			)
+		)
+		(property "Description" "Resistor"
+			(at 72.39 127.0 0)
+			(hide yes)
+			(show_name no)
+			(do_not_autoplace no)
+			(effects
+				(font
+					(size 1.27 1.27)
+				)
+			)
+		)
+		(pin "1"
+		)
+		(pin "2"
+		)
+		(instances
+			(project "xt8086_beta"
+				(path "/8c0b3d8b-46d3-4173-ab1e-a61765f77d61/fc69669c-5428-4356-8e92-0aa932a39979"
+					(reference "R54")
+					(unit 1)
+				)
+			)
+		)
+	)
+	(wire
+		(pts
+			(xy 76.2 127.0) (xy 80.01 127.0)
+		)
+		(stroke
+			(width 0)
+			(type default)
+		)
+	)
+	(wire
+		(pts
+			(xy 68.58 127.0) (xy 63.5 127.0)
+		)
+		(stroke
+			(width 0)
+			(type default)
+		)
+	)
+	(label "ST"
+		(at 63.5 127.0 0)
+		(effects
+				(font
+					(size 1.27 1.27)
+				)
+				(justify left bottom)
+			)
+	)
+	(text "R54: TPS2116 ST -> PR1 hysteresis"
+		(exclude_from_sim no)
+		(at 55.0 146.0 0)
+		(effects
+			(font
+				(size 1.27 1.27)
+			)
+			(justify left bottom)
+		)
+	)
+	(text "(matches frank_next R56)."
+		(exclude_from_sim no)
+		(at 55.0 149.81 0)
+		(effects
+			(font
+				(size 1.27 1.27)
+			)
+			(justify left bottom)
+		)
+	)

Commit message: Board updates
Other:
- note removed: "(matches frank_next R56)."
- note removed: "R54: TPS2116 ST -> PR1 hysteresis"
Changed lines of the file:
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@@
 	(wire
 		(pts
+			(xy 127 134.62) (xy 134.62 134.62)
+		)
+		(stroke
+			(width 0)
+			(type default)
+		)
+	)
+	(wire
+		(pts
 			(xy 62.23 69.85) (xy 62.23 74.93)
 		)
@@
 	(wire
 		(pts
+			(xy 68.58 127) (xy 63.5 127)
+		)
+		(stroke
+			(width 0)
+			(type default)
+		)
+	)
+	(wire
+		(pts
 			(xy 228.6 53.34) (xy 228.6 62.23)
 		)
@@
 	(wire
 		(pts
+			(xy 76.2 127) (xy 80.01 127)
+		)
+		(stroke
+			(width 0)
+			(type default)
+		)
+	)
+	(wire
+		(pts
 			(xy 115.57 146.05) (xy 102.87 146.05)
 		)
@@
 		)
 	)
+	(label "ST"
+		(at 63.5 127 0)
+		(effects
+			(font
+				(size 1.27 1.27)
+			)
+			(justify left bottom)
+		)
+	)
 	(label "UA1M"
 		(at 256.54 72.39 180)
@@
 		)
 	)
+	(label "ST"
+		(at 134.62 134.62 0)
+		(effects
+			(font
+				(size 1.27 1.27)
+			)
+			(justify left bottom)
+		)
+	)
 	(label "UA2M"
 		(at 157.48 64.77 0)
@@
 	)
 	(symbol
+		(lib_id "xt8086:R")
+		(at 72.39 127 90)
+		(unit 1)
+		(body_style 1)
+		(exclude_from_sim no)
+		(in_bom yes)
+		(on_board yes)
+		(in_pos_files yes)
+		(dnp no)
+		(property "Reference" "R54"
+			(at 72.39 121.92 90)
+			(show_name no)
+			(do_not_autoplace no)
+			(effects
+				(font
+					(size 1.27 1.27)
+				)
+			)
+		)
+		(property "Value" "1M"
+			(at 72.39 124.46 90)
+			(show_name no)
+			(do_not_autoplace no)
+			(effects
+				(font
+					(size 1.27 1.27)
+				)
+			)
+		)
+		(property "Footprint" "xt8086:R_0603_1608Metric"
+			(at 72.39 127 0)
+			(hide yes)
+			(show_name no)
+			(do_not_autoplace no)
+			(effects
+				(font
+					(size 1.27 1.27)
+				)
+			)
+		)
+		(property "Datasheet" ""
+			(at 72.39 127 0)
+			(hide yes)
+			(show_name no)
+			(do_not_autoplace no)
+			(effects
+				(font
+					(size 1.27 1.27)
+				)
+			)
+		)
+		(property "Description" "Resistor"
+			(at 72.39 127 0)
+			(hide yes)
+			(show_name no)
+			(do_not_autoplace no)
+			(effects
+				(font
+					(size 1.27 1.27)
+				)
+			)
+		)
+		(pin "1"
+		)
+		(pin "2"
+		)
+		(instances
+			(project "xt8086_beta"
+				(path "/8c0b3d8b-46d3-4173-ab1e-a61765f77d61/fc69669c-5428-4356-8e92-0aa932a39979"
+					(reference "R54")
+					(unit 1)
+				)
+			)
+		)
+	)
+	(symbol
 		(lib_id "xt8086:Conn_01x02_Pin")
 		(at 57.15 113.03 180)
@@
 		)
 	)
-	(wire
-		(pts
-			(xy 127.0 134.62) (xy 134.62 134.62)
-		)
-		(stroke
-			(width 0)
-			(type default)
-		)
-	)
-	(label "ST"
-		(at 134.62 134.62 0)
-		(effects
-				(font
-					(size 1.27 1.27)
-				)
-				(justify left bottom)
-			)
-	)
-	(symbol
-		(lib_id "xt8086:R")
-		(at 72.39 127.0 90)
-		(unit 1)
-		(body_style 1)
-		(exclude_from_sim no)
-		(in_bom yes)
-		(on_board yes)
-		(in_pos_files yes)
-		(dnp no)
-		(property "Reference" "R54"
-			(at 72.39 121.92 90)
-			(show_name no)
-			(do_not_autoplace no)
-			(effects
-				(font
-					(size 1.27 1.27)
-				)
-			)
-		)
-		(property "Value" "1M"
-			(at 72.39 124.46 90)
-			(show_name no)
-			(do_not_autoplace no)
-			(effects
-				(font
-					(size 1.27 1.27)
-				)
-			)
-		)
-		(property "Footprint" "xt8086:R_0603_1608Metric"
-			(at 72.39 127.0 0)
-			(hide yes)
-			(show_name no)
-			(do_not_autoplace no)
-			(effects
-				(font
-					(size 1.27 1.27)
-				)
-			)
-		)
-		(property "Datasheet" ""
-			(at 72.39 127.0 0)
-			(hide yes)
-			(show_name no)
-			(do_not_autoplace no)
-			(effects
-				(font
-					(size 1.27 1.27)
-				)
-			)
-		)
-		(property "Description" "Resistor"
-			(at 72.39 127.0 0)
-			(hide yes)
-			(show_name no)
-			(do_not_autoplace no)
-			(effects
-				(font
-					(size 1.27 1.27)
-				)
-			)
-		)
-		(pin "1"
-		)
-		(pin "2"
-		)
-		(instances
-			(project "xt8086_beta"
-				(path "/8c0b3d8b-46d3-4173-ab1e-a61765f77d61/fc69669c-5428-4356-8e92-0aa932a39979"
-					(reference "R54")
-					(unit 1)
-				)
-			)
-		)
-	)
-	(wire
-		(pts
-			(xy 76.2 127.0) (xy 80.01 127.0)
-		)
-		(stroke
-			(width 0)
-			(type default)
-		)
-	)
-	(wire
-		(pts
-			(xy 68.58 127.0) (xy 63.5 127.0)
-		)
-		(stroke
-			(width 0)
-			(type default)
-		)
-	)
-	(label "ST"
-		(at 63.5 127.0 0)
-		(effects
-				(font
-					(size 1.27 1.27)
-				)
-				(justify left bottom)
-			)
-	)
-	(text "R54: TPS2116 ST -> PR1 hysteresis"
-		(exclude_from_sim no)
-		(at 55.0 146.0 0)
-		(effects
-			(font
-				(size 1.27 1.27)
-			)
-			(justify left bottom)
-		)
-	)
-	(text "(matches frank_next R56)."
-		(exclude_from_sim no)
-		(at 55.0 149.81 0)
-		(effects
-			(font
-				(size 1.27 1.27)
-			)
-			(justify left bottom)
-		)
-	)

Commit message: Board updates
Parts:
- C32, C33: value 100nF -> 100n
- C34, C35: value 10uF -> 10u
- renumbered J7 to J6, J8 to J7, R54 to R18, R18 to R19, R19 to R20
Changed lines of the file:
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@@
 		(dnp no)
 		(fields_autoplaced yes)
-		(property "Reference" "J8"
+		(property "Reference" "J7"
 			(at 204.47 54.61 0)
 			(show_name no)
@@
 			(project "xt8086_beta"
 				(path "/8c0b3d8b-46d3-4173-ab1e-a61765f77d61/fc69669c-5428-4356-8e92-0aa932a39979"
-					(reference "J8")
+					(reference "J7")
 					(unit 1)
 				)
@@
 			)
 		)
-		(property "Value" "10uF"
+		(property "Value" "10u"
 			(at 118.491 111.633 0)
 			(show_name no)
@@
 		(in_pos_files yes)
 		(dnp no)
-		(property "Reference" "J7"
+		(property "Reference" "J6"
 			(at 43.18 60.96 0)
 			(hide yes)
@@
 			(project "xt8086_beta"
 				(path "/8c0b3d8b-46d3-4173-ab1e-a61765f77d61/fc69669c-5428-4356-8e92-0aa932a39979"
-					(reference "J7")
+					(reference "J6")
 					(unit 1)
 				)
@@
 		(in_pos_files yes)
 		(dnp no)
-		(property "Reference" "R19"
+		(property "Reference" "R20"
 			(at 83.82 134.62 90)
 			(show_name no)
@@
 			(project "xt8086_beta"
 				(path "/8c0b3d8b-46d3-4173-ab1e-a61765f77d61/fc69669c-5428-4356-8e92-0aa932a39979"
-					(reference "R19")
+					(reference "R20")
 					(unit 1)
 				)
@@
 			)
 		)
-		(property "Value" "100nF"
+		(property "Value" "100n"
 			(at 105.791 111.633 0)
 			(show_name no)
@@
 		(in_pos_files yes)
 		(dnp no)
-		(property "Reference" "R54"
+		(property "Reference" "R18"
 			(at 72.39 121.92 90)
 			(show_name no)
@@
 			(project "xt8086_beta"
 				(path "/8c0b3d8b-46d3-4173-ab1e-a61765f77d61/fc69669c-5428-4356-8e92-0aa932a39979"
-					(reference "R54")
+					(reference "R18")
 					(unit 1)
 				)
@@
 			)
 		)
-		(property "Value" "10uF"
+		(property "Value" "10u"
 			(at 118.491 148.717 0)
 			(show_name no)
@@
 		(in_pos_files yes)
 		(dnp no)
-		(property "Reference" "R18"
+		(property "Reference" "R19"
 			(at 83.82 119.38 90)
 			(show_name no)
@@
 			(project "xt8086_beta"
 				(path "/8c0b3d8b-46d3-4173-ab1e-a61765f77d61/fc69669c-5428-4356-8e92-0aa932a39979"
-					(reference "R18")
+					(reference "R19")
 					(unit 1)
 				)
@@
 			)
 		)
-		(property "Value" "100nF"
+		(property "Value" "100n"
 			(at 105.791 148.717 0)
 			(show_name no)

Commit message: feat: xt8086_beta gets Dino's sound and schematic changes
xt8086_beta and dino_z80 share their platform, so everything done to the
Dino schematic is carried over:

- Buzzer sheet replaced by Dino's Sound + Speaker sheets: LM358 line out,
  PAM8403 driving a CVS-2308 speaker, S2 as HDMI L/R + speaker enable,
  stereo HDMI audio (AUDIO_IN_L/R no longer tied together).
- GP46 is PWM_L, GP44 is PWM_R, exactly as on Dino; J1 (UART) is gone
  and GP45 is left unconnected.
- USB defaults to the RP2350: R3 pulls SW low, S1's common goes to +3V3,
  JP3 (USB Test) straps SW high.
- H1-H4 become 2.5 mm pad-and-via holes tied to GND.
- MS9288A footprint renamed QFN-48_6x6mm.
- Shared sheets take Dino's current versions with xt8086_beta's own
  references; SI values, X1 renamed Y2, datasheet links fixed, plus TI
  SN74LS74A and Analog Devices DS3231M links for xt-only parts.
- Libraries: PAM8403D, LM358, CVS-2308, MountingHole_Pad symbols and
  their footprints/3D models; SOT-23 pad mirror fix and SOIC-8 from Dino.

dino.kicad_sym also gains CVS-2308 and MountingHole_Pad, which Dino's
schematic had only in its symbol cache.

ERC: 0. The board is not updated yet.
Parts:
- C30, C31, C32, C33, C37, C39: value 100n -> 100nF
- C34, C35, C40, C41: value 10u -> 10µF
- C36, C38: value 100u -> 100µF
- R16, R17: value 5.1K -> 5.1kΩ
- R18: value 1M -> 1MΩ
- R19: value 300K -> 300kΩ; AliExpress https://www.vishay.com/docs/28952/mcs0402at-mct0603at-mcu08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 -> (none)
- R20: value 100K -> 100kΩ; AliExpress https://www.vishay.com/docs/28952/mcs0402at-mct0603at-mcu08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 -> (none)
Other:
- moved on the sheet: C36, C37, C38, C39

Commit message: feat: compact rounded solder jumpers and debug jumpers across S2
- all solder jumpers use a compact rounded footprint
  (SolderJumper-2_P1.0mm_Open_RoundedPad0.7x1.0mm: 0.7x1.0 mm pads,
  0.3 mm gap), scaled from KiCad's stock RoundedPad jumper
- JP4/JP5/JP6 (Audio L, Audio R, Speaker) bridge each S2 position, on
  the back under S2, so the DIP switch can be left unfitted
- JP3 on Dino gets short tracks to its vias, which the smaller pads no
  longer cover
Parts:
- JP1: footprint xt8086:SolderJumper-2_P1.3mm_Open_Pad1.0x1.5mm -> xt8086:SolderJumper-2_P1.0mm_Open_RoundedPad0.7x1.0mm
Changed lines of the file:
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@@
 			)
 		)
-		(property "Footprint" "xt8086:SolderJumper-2_P1.3mm_Open_Pad1.0x1.5mm"
+		(property "Footprint" "xt8086:SolderJumper-2_P1.0mm_Open_RoundedPad0.7x1.0mm"
 			(at 57.15 113.03 0)
 			(hide yes)

Commit message: fix: board review round - protection, pull-ups, parts data
- MS9288A config I2C pull-ups (SCL/SDA) go to +3V3; the chip's pins
  are rated only to DVDD33 + 0.5 V, and the reference leaves them open
- MS9288A audio inputs: 0 Ohm series + 10 kOhm shunt (not fitted) ahead
  of the coupling caps, so the reference 1/2 divider can be fitted later
- HDMI +5 V pin: 0.2 A resettable fuse (F2, 0603) in series with D5
- SD card: 10 kOhm pull-ups on CMD, DAT0 and DAT3 (SPI mode)
- xt8086: U1 is a 74HCT04 buffering GP29 to a 5 V 8086 CLK; RESET gets a
  10 kOhm pull-up so the CPU is held in reset until the RP2350 drives it
- video ladder and headphone series resistors 400/800 -> 402/806 Ohm
- LCSC part numbers checked against JLC for 452 parts; wrong numbers on
  R57, the 4.7 uF caps and the USB-C connector fixed
- MS9288A symbol: pin 3 is NC, datasheet linked; CD4069 pin name fixed
- Dino board follows the schematic renumbering; label and via clean-up
Parts:
- C30, C31, C32, C33, C37, C39: LCSC (none) -> C14663
- C34, C35, C40, C41: LCSC (none) -> C19702
- C36: LCSC (none) -> C48935385
- C38: LCSC (none) -> C15008
- J6: LCSC C165948 -> C37616412
- R16, R17: LCSC (none) -> C23186
- R18: LCSC (none) -> C22935
- R19: LCSC (none) -> C23024
- R20: LCSC (none) -> C25803
- U10: LCSC (none) -> C3235557
- U11, U12, U9: LCSC (none) -> C7519
Changed lines of the file:
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@@
 			)
 		)
+		(property "LCSC" "C14663"
+			(at 212.09 132.08 0)
+			(hide yes)
+			(show_name no)
+			(do_not_autoplace no)
+			(effects
+				(font
+					(size 1.27 1.27)
+				)
+			)
+		)
 		(property "Description" "Unpolarized capacitor, small symbol"
 			(at 212.09 132.08 0)
@@
 			)
 		)
+		(property "LCSC" "C48935385"
+			(at 166.37 132.08 0)
+			(hide yes)
+			(show_name no)
+			(do_not_autoplace no)
+			(effects
+				(font
+					(size 1.27 1.27)
+				)
+			)
+		)
 		(property "Description" "Polarized capacitor, small symbol"
 			(at 166.37 132.08 0)
@@
 			)
 		)
-		(property "LCSC" ""
+		(property "LCSC" "C19702"
 			(at 115.57 110.49 0)
 			(show_name no)
@@
 			)
 		)
+		(property "LCSC" "C15008"
+			(at 204.47 132.08 0)
+			(hide yes)
+			(show_name no)
+			(do_not_autoplace no)
+			(effects
+				(font
+					(size 1.27 1.27)
+				)
+			)
+		)
 		(property "Description" "Polarized capacitor, small symbol"
 			(at 204.47 132.08 0)
@@
 			)
 		)
-		(property "LCSC" ""
+		(property "LCSC" "C19702"
 			(at 220.98 53.34 0)
 			(hide yes)
@@
 			)
 		)
-		(property "LCSC" "C165948"
+		(property "LCSC" "C37616412"
 			(at 49.53 71.12 0)
 			(hide yes)
@@
 			)
 		)
-		(property "LCSC" ""
+		(property "LCSC" "C14663"
 			(at 87.63 52.07 0)
 			(hide yes)
@@
 			)
 		)
-		(property "LCSC" ""
+		(property "LCSC" "C25803"
 			(at 83.82 129.54 0)
 			(show_name no)
@@
 			)
 		)
-		(property "LCSC" ""
+		(property "LCSC" "C14663"
 			(at 102.87 110.49 0)
 			(show_name no)
@@
 			)
 		)
+		(property "LCSC" "C22935"
+			(at 72.39 127 0)
+			(hide yes)
+			(show_name no)
+			(do_not_autoplace no)
+			(effects
+				(font
+					(size 1.27 1.27)
+				)
+			)
+		)
 		(property "Description" "Resistor"
 			(at 72.39 127 0)
@@
 			)
 		)
-		(property "LCSC" ""
+		(property "LCSC" "C19702"
 			(at 115.57 149.86 0)
 			(show_name no)
@@
 			)
 		)
-		(property "LCSC" ""
+		(property "LCSC" "C23024"
 			(at 83.82 124.46 0)
 			(show_name no)
@@
 			)
 		)
-		(property "LCSC" ""
+		(property "LCSC" "C14663"
 			(at 102.87 149.86 0)
 			(show_name no)
@@
 			)
 		)
+		(property "LCSC" "C14663"
+			(at 177.8 132.08 0)
+			(hide yes)
+			(show_name no)
+			(do_not_autoplace no)
+			(effects
+				(font
+					(size 1.27 1.27)
+				)
+			)
+		)
 		(property "Description" "Unpolarized capacitor, small symbol"
 			(at 177.8 132.08 0)
@@
 			)
 		)
-		(property "LCSC" ""
+		(property "LCSC" "C19702"
 			(at 243.84 53.34 0)
 			(hide yes)
@@
 			)
 		)
+		(property "LCSC" "C3235557"
+			(at 116.84 128.27 0)
+			(hide yes)
+			(show_name no)
+			(do_not_autoplace no)
+			(effects
+				(font
+					(size 1.27 1.27)
+				)
+			)
+		)
 		(property "Description" "2-channel power mux with manual and priority switchover, 1.6V to 5.5V, 2.5A"
 			(at 116.84 130.556 0)
@@
 			)
 		)
-		(property "LCSC" ""
+		(property "LCSC" "C23186"
 			(at 54.61 64.77 0)
 			(hide yes)
@@
 			)
 		)
-		(property "LCSC" ""
+		(property "LCSC" "C23186"
 			(at 54.61 80.01 0)
 			(hide yes)
@@
 			)
 		)
+		(property "LCSC" "C7519"
+			(at 242.57 76.835 0)
+			(hide yes)
+			(show_name no)
+			(do_not_autoplace no)
+			(effects
+				(font
+					(size 1.27 1.27)
+				)
+				(justify left)
+			)
+		)
 		(property "Description" "Very low capacitance ESD protection diode, 2 data-line, SOT-23-6"
 			(at 241.3 85.09 0)
@@
 			)
 		)
+		(property "LCSC" "C7519"
+			(at 91.44 78.105 0)
+			(hide yes)
+			(show_name no)
+			(do_not_autoplace no)
+			(effects
+				(font
+					(size 1.27 1.27)
+				)
+				(justify left)
+			)
+		)
 		(property "Description" "Very low capacitance ESD protection diode, 2 data-line, SOT-23-6"
 			(at 90.17 69.85 0)
@@
 			)
 		)
+		(property "LCSC" "C14663"
+			(at 99.06 58.42 0)
+			(hide yes)
+			(show_name no)
+			(do_not_autoplace no)
+			(effects
+				(font
+					(size 1.27 1.27)
+				)
+			)
+		)
 		(property "Description" "Unpolarized capacitor"
 			(at 99.06 58.42 0)
@@
 			(at 242.57 78.105 0)
 			(hide yes)
+			(show_name no)
+			(do_not_autoplace no)
+			(effects
+				(font
+					(size 1.27 1.27)
+				)
+				(justify left)
+			)
+		)
+		(property "LCSC" "C7519"
+			(at 242.57 78.105 0)
+			(hide yes)
