File: xt8086_beta/reset.kicad_sch (KiCad schematic)
At the start: 1 part

Commit message: Board updates
Parts:
- renumbered S5 to S4
Changed lines of the file:
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@@
 		(dnp no)
 		(fields_autoplaced yes)
-		(property "Reference" "S5"
+		(property "Reference" "S4"
 			(at 162.56 90.17 0)
 			(show_name no)
@@
 			(project "xt8086_beta"
 				(path "/8c0b3d8b-46d3-4173-ab1e-a61765f77d61/69d580d4-830a-4ad1-89c3-268c1b1da372/f116f564-09bc-474c-8ad3-3a701671535f"
-					(reference "S5")
+					(reference "S4")
 					(unit 1)
 				)
@@
 		(in_pos_files yes)
 		(dnp no)
-		(property "Reference" "#PWR093"
+		(property "Reference" "#PWR089"
 			(at 146.05 100.33 0)
 			(hide yes)
@@
 			(project "xt8086_beta"
 				(path "/8c0b3d8b-46d3-4173-ab1e-a61765f77d61/69d580d4-830a-4ad1-89c3-268c1b1da372/f116f564-09bc-474c-8ad3-3a701671535f"
-					(reference "#PWR093")
+					(reference "#PWR089")
 					(unit 1)
 				)
@@
 		(in_pos_files yes)
 		(dnp no)
-		(property "Reference" "#PWR094"
+		(property "Reference" "#PWR090"
 			(at 179.07 100.33 0)
 			(hide yes)
@@
 			(project "xt8086_beta"
 				(path "/8c0b3d8b-46d3-4173-ab1e-a61765f77d61/69d580d4-830a-4ad1-89c3-268c1b1da372/f116f564-09bc-474c-8ad3-3a701671535f"
-					(reference "#PWR094")
+					(reference "#PWR090")
 					(unit 1)
 				)

Commit message: Board updates
Parts:
- added C42: 1n, xt8086:C_0603_1608Metric, symbol xt8086:C
Connections:
- net GND: now also C42.1
- net RESET: now also C42.2
Changed lines of the file:
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@@
 	(generator_version "10.0")
 	(paper "A4")
+	(junction
+		(at 152.4 97.79)
+		(diameter 0)
+		(color 0 0 0 0)
+	)
+	(wire
+		(pts
+			(xy 152.4 97.79) (xy 152.4 90.17)
+		)
+		(stroke
+			(width 0)
+			(type default)
+		)
+	)
 	(wire
 		(pts
@@
 			)
 			(justify right)
+		)
+	)
+	(symbol
+		(lib_id "xt8086:C")
+		(at 152.4 86.36 0)
+		(unit 1)
+		(body_style 1)
+		(exclude_from_sim no)
+		(in_bom yes)
+		(on_board yes)
+		(in_pos_files yes)
+		(dnp no)
+		(property "Reference" "C42"
+			(at 154.305 85.09 0)
+			(show_name no)
+			(do_not_autoplace no)
+			(effects
+				(font
+					(size 1.27 1.27)
+				)
+				(justify left)
+			)
+		)
+		(property "Value" "1n"
+			(at 154.305 87.63 0)
+			(show_name no)
+			(do_not_autoplace no)
+			(effects
+				(font
+					(size 1.27 1.27)
+				)
+				(justify left)
+			)
+		)
+		(property "Footprint" "xt8086:C_0603_1608Metric"
+			(at 152.4 86.36 0)
+			(hide yes)
+			(show_name no)
+			(do_not_autoplace no)
+			(effects
+				(font
+					(size 1.27 1.27)
+				)
+			)
+		)
+		(property "Datasheet" ""
+			(at 152.4 86.36 0)
+			(hide yes)
+			(show_name no)
+			(do_not_autoplace no)
+			(effects
+				(font
+					(size 1.27 1.27)
+				)
+			)
+		)
+		(property "Description" "Unpolarized capacitor"
+			(at 152.4 86.36 0)
+			(hide yes)
+			(show_name no)
+			(do_not_autoplace no)
+			(effects
+				(font
+					(size 1.27 1.27)
+				)
+			)
+		)
+		(pin "1"
+		)
+		(pin "2"
+		)
+		(instances
+			(project "xt8086_beta"
+				(path "/8c0b3d8b-46d3-4173-ab1e-a61765f77d61/69d580d4-830a-4ad1-89c3-268c1b1da372/f116f564-09bc-474c-8ad3-3a701671535f"
+					(reference "C42")
+					(unit 1)
+				)
+			)
 		)
 	)
@@
 		(in_pos_files yes)
 		(dnp no)
-		(property "Reference" "#PWR088"
+		(property "Reference" "#PWR0102"
 			(at 146.05 100.33 0)
 			(hide yes)
@@
 			(project "xt8086_beta"
 				(path "/8c0b3d8b-46d3-4173-ab1e-a61765f77d61/69d580d4-830a-4ad1-89c3-268c1b1da372/f116f564-09bc-474c-8ad3-3a701671535f"
-					(reference "#PWR088")
+					(reference "#PWR0102")
 					(unit 1)
 				)
@@
 		(in_pos_files yes)
 		(dnp no)
-		(property "Reference" "#PWR089"
+		(property "Reference" "#PWR0103"
 			(at 179.07 100.33 0)
 			(hide yes)
@@
 			(project "xt8086_beta"
 				(path "/8c0b3d8b-46d3-4173-ab1e-a61765f77d61/69d580d4-830a-4ad1-89c3-268c1b1da372/f116f564-09bc-474c-8ad3-3a701671535f"
-					(reference "#PWR089")
+					(reference "#PWR0103")
 					(unit 1)
 				)
+			)
+		)
+	)
+	(symbol
+		(lib_id "xt8086:GND")
+		(at 152.4 82.55 180)
+		(unit 1)
+		(body_style 1)
+		(exclude_from_sim no)
+		(in_bom yes)
+		(on_board yes)
+		(in_pos_files no)
+		(dnp no)
+		(fields_autoplaced yes)
+		(property "Reference" "#PWR0101"
+			(at 152.4 78.74 0)
+			(hide yes)
+			(show_name no)
+			(do_not_autoplace no)
+			(effects
+				(font
+					(size 1.27 1.27)
+				)
+			)
+		)
+		(property "Value" "GND"
+			(at 152.4 78.994 0)
+			(show_name no)
+			(do_not_autoplace no)
+			(effects
+				(font
+					(size 1.27 1.27)
+				)
+			)
+		)
+		(property "Footprint" ""
+			(at 152.4 82.55 0)
+			(hide yes)
+			(show_name no)
+			(do_not_autoplace no)
+			(effects
+				(font
+					(size 1.27 1.27)
+				)
+			)
+		)
+		(property "Datasheet" ""
+			(at 152.4 82.55 0)
+			(hide yes)
+			(show_name no)
+			(do_not_autoplace no)
+			(effects
+				(font
+					(size 1.27 1.27)
+				)
+			)
+		)
+		(property "Description" "Power symbol creates a global label with name \"GND\" , ground"
+			(at 152.4 82.55 0)
+			(hide yes)
+			(show_name no)
+			(do_not_autoplace no)
+			(effects
+				(font
+					(size 1.27 1.27)
+				)
+			)
+		)
+		(pin "1"
+		)
+		(instances
+			(project "xt8086_beta"
+				(path "/8c0b3d8b-46d3-4173-ab1e-a61765f77d61/69d580d4-830a-4ad1-89c3-268c1b1da372/f116f564-09bc-474c-8ad3-3a701671535f"
+					(reference "#PWR0101")
+					(unit 1)
+				)

Commit message: feat: xt8086_beta gets Dino's sound and schematic changes
xt8086_beta and dino_z80 share their platform, so everything done to the
Dino schematic is carried over:

- Buzzer sheet replaced by Dino's Sound + Speaker sheets: LM358 line out,
  PAM8403 driving a CVS-2308 speaker, S2 as HDMI L/R + speaker enable,
  stereo HDMI audio (AUDIO_IN_L/R no longer tied together).
- GP46 is PWM_L, GP44 is PWM_R, exactly as on Dino; J1 (UART) is gone
  and GP45 is left unconnected.
- USB defaults to the RP2350: R3 pulls SW low, S1's common goes to +3V3,
  JP3 (USB Test) straps SW high.
- H1-H4 become 2.5 mm pad-and-via holes tied to GND.
- MS9288A footprint renamed QFN-48_6x6mm.
- Shared sheets take Dino's current versions with xt8086_beta's own
  references; SI values, X1 renamed Y2, datasheet links fixed, plus TI
  SN74LS74A and Analog Devices DS3231M links for xt-only parts.
- Libraries: PAM8403D, LM358, CVS-2308, MountingHole_Pad symbols and
  their footprints/3D models; SOT-23 pad mirror fix and SOIC-8 from Dino.

dino.kicad_sym also gains CVS-2308 and MountingHole_Pad, which Dino's
schematic had only in its symbol cache.

ERC: 0. The board is not updated yet.
Parts:
- C42: value 1n -> 1nF
Other:
- company: (none) -> Mikhail Matveev
- title: (none) -> ${NAME} ${MODEL}
Changed lines of the file:
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@@
 	(generator_version "10.0")
 	(paper "A4")
+	(title_block
+		(title "${NAME} ${MODEL}")
+		(date "${DATE}")
+		(rev "${VERSION}")
+		(company "Mikhail Matveev")
+		(comment 1 "https://github.com/rh1tech/frank")
+	)
 	(junction
 		(at 152.4 97.79)
@@
 			)
 		)
-		(property "Value" "1n"
+		(property "Value" "1nF"
 			(at 154.305 87.63 0)
 			(show_name no)
@@
 			)
 		)
-		(property "Datasheet" "https://componentsearchengine.com/Datasheets/1/KMR221G LFS.pdf"
+		(property "Datasheet" "https://www.littelfuse.com/assetdocs/littelfuse-ck-tactile-kmr2-series-datasheet?assetguid=f782bfc7-b600-4ab5-8c8d-a2a094a642e3"
 			(at 168.91 292.71 0)
 			(hide yes)

Commit message: fix: board review round - protection, pull-ups, parts data
- MS9288A config I2C pull-ups (SCL/SDA) go to +3V3; the chip's pins
  are rated only to DVDD33 + 0.5 V, and the reference leaves them open
- MS9288A audio inputs: 0 Ohm series + 10 kOhm shunt (not fitted) ahead
  of the coupling caps, so the reference 1/2 divider can be fitted later
- HDMI +5 V pin: 0.2 A resettable fuse (F2, 0603) in series with D5
- SD card: 10 kOhm pull-ups on CMD, DAT0 and DAT3 (SPI mode)
- xt8086: U1 is a 74HCT04 buffering GP29 to a 5 V 8086 CLK; RESET gets a
  10 kOhm pull-up so the CPU is held in reset until the RP2350 drives it
- video ladder and headphone series resistors 400/800 -> 402/806 Ohm
- LCSC part numbers checked against JLC for 452 parts; wrong numbers on
  R57, the 4.7 uF caps and the USB-C connector fixed
- MS9288A symbol: pin 3 is NC, datasheet linked; CD4069 pin name fixed
- Dino board follows the schematic renumbering; label and via clean-up
Parts:
- C42: LCSC (none) -> C1588
- S4: LCSC (none) -> C72443
Changed lines of the file:
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@@
+			)
+		)
+		(property "LCSC" "C1588"
+			(at 152.4 86.36 0)
+			(hide yes)
+			(show_name no)
+			(do_not_autoplace no)
+			(effects
+				(font
+					(size 1.27 1.27)
+				)
 			)
 		)
@@
 			(at 168.91 292.71 0)
 			(hide yes)
+			(show_name no)
+			(do_not_autoplace no)
+			(effects
+				(font
+					(size 1.27 1.27)
+				)
+				(justify left top)
+			)
+		)
+		(property "LCSC" "C72443"
+			(at 168.91 292.71 0)
+			(hide yes)

Commit message: fix: xt8086_beta 1.04 - pre-production review, TVS input, labels, release
- Power: SMAJ15A TVS D7 after the fuse (C908769, optional fit); Q1 gate
  divider R22/R23 100K/43K (Vgs within +-12 V at the TVS clamp); MP1584 UVLO
  R25/R26 300K/100K (start ~6.0 V); C44 680u 25V (C46550437); notes fixed
- Every capacitor value carries its voltage (from the LCSC part)
- Test points on all rails, on the back
- ERC: connector/hub pin types, PWR_FLAGs; 49 stale exclusions removed.
  ERC 0 errors, 0 warnings
- RP2350 exposed-pad vias tagged heatsink (no type mismatch)
- Fields: LCSC numbers removed from solder jumpers, S1/U1/U2/Y2/L1 part
  data and datasheet links corrected
- Layout: vias moved out of signal/power pads where a 45-degree escape
  exists, corners fixed, reference labels 0.7 mm bold re-placed
- Release 1.04: gerbers, schematics, assembly PDF, iBOM
  (DRC 0 violations, 0 unconnected, 0 parity)
Parts:
- C42: value 1nF -> 1n 50V
Changed lines of the file:
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@@
 			)
 		)
-		(property "Value" "1nF"
+		(property "Value" "1n 50V"
 			(at 154.305 87.63 0)
 			(show_name no)
