File: xt8086_beta/usb_a_power.kicad_sch (KiCad schematic)
At the start: 13 parts, among them U20 CH217K, U21 CH217K

Commit message: Board updates
Parts:
- C89, C92: footprint xt8086:C_Radial_D6.3mm_P2.50mm -> xt8086:CP_Radial_D6.3mm_P2.50mm
Changed lines of the file:
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@@
 			)
 		)
-		(property "Footprint" "xt8086:C_Radial_D6.3mm_P2.50mm"
+		(property "Footprint" "xt8086:CP_Radial_D6.3mm_P2.50mm"
 			(at 88.9 71.12 0)
 			(hide yes)
@@
 			)
 		)
-		(property "Footprint" "xt8086:C_Radial_D6.3mm_P2.50mm"
+		(property "Footprint" "xt8086:CP_Radial_D6.3mm_P2.50mm"
 			(at 104.14 71.12 0)
 			(hide yes)

Commit message: Board updates
Parts:
- C89, C92: value 100uF -> 100u
- renumbered LD3 to D6, R50 to R51, R51 to R52, R52 to R53, R53 to R54, U20 to U18, U21 to U19
Changed lines of the file:
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@@
 		(dnp no)
 		(fields_autoplaced yes)
-		(property "Reference" "#PWR0188"
+		(property "Reference" "#PWR0186"
 			(at 139.7 128.27 0)
 			(hide yes)
@@
 			(project "xt8086_beta"
 				(path "/8c0b3d8b-46d3-4173-ab1e-a61765f77d61/fc69669c-5428-4356-8e92-0aa932a39979/e922aa3b-a7c2-5123-b7ae-6a56da586377"
-					(reference "#PWR0188")
+					(reference "#PWR0186")
 					(unit 1)
 				)
@@
 		(dnp no)
 		(fields_autoplaced yes)
-		(property "Reference" "#PWR0181"
+		(property "Reference" "#PWR0179"
 			(at 101.6 127 0)
 			(hide yes)
@@
 			(project "xt8086_beta"
 				(path "/8c0b3d8b-46d3-4173-ab1e-a61765f77d61/fc69669c-5428-4356-8e92-0aa932a39979/e922aa3b-a7c2-5123-b7ae-6a56da586377"
-					(reference "#PWR0181")
+					(reference "#PWR0179")
 					(unit 1)
 				)
@@
 		(dnp no)
 		(fields_autoplaced yes)
-		(property "Reference" "#PWR0183"
+		(property "Reference" "#PWR0181"
 			(at 107.95 91.44 0)
 			(hide yes)
@@
 			(project "xt8086_beta"
 				(path "/8c0b3d8b-46d3-4173-ab1e-a61765f77d61/fc69669c-5428-4356-8e92-0aa932a39979/e922aa3b-a7c2-5123-b7ae-6a56da586377"
-					(reference "#PWR0183")
+					(reference "#PWR0181")
 					(unit 1)
 				)
@@
 		(dnp no)
 		(fields_autoplaced yes)
-		(property "Reference" "#PWR0185"
+		(property "Reference" "#PWR0183"
 			(at 118.11 95.25 0)
 			(hide yes)
@@
 			(project "xt8086_beta"
 				(path "/8c0b3d8b-46d3-4173-ab1e-a61765f77d61/fc69669c-5428-4356-8e92-0aa932a39979/e922aa3b-a7c2-5123-b7ae-6a56da586377"
-					(reference "#PWR0185")
+					(reference "#PWR0183")
 					(unit 1)
 				)
@@
 		(in_pos_files yes)
 		(dnp no)
-		(property "Reference" "R51"
+		(property "Reference" "R52"
 			(at 111.76 128.27 0)
 			(show_name no)
@@
 			(project "xt8086_beta"
 				(path "/8c0b3d8b-46d3-4173-ab1e-a61765f77d61/fc69669c-5428-4356-8e92-0aa932a39979/e922aa3b-a7c2-5123-b7ae-6a56da586377"
-					(reference "R51")
+					(reference "R52")
 					(unit 1)
 				)
@@
 		(dnp no)
 		(fields_autoplaced yes)
-		(property "Reference" "#PWR0186"
+		(property "Reference" "#PWR0184"
 			(at 118.11 133.35 0)
 			(hide yes)
@@
 			(project "xt8086_beta"
 				(path "/8c0b3d8b-46d3-4173-ab1e-a61765f77d61/fc69669c-5428-4356-8e92-0aa932a39979/e922aa3b-a7c2-5123-b7ae-6a56da586377"
-					(reference "#PWR0186")
+					(reference "#PWR0184")
 					(unit 1)
 				)
@@
 		(in_pos_files yes)
 		(dnp no)
-		(property "Reference" "U20"
+		(property "Reference" "U18"
 			(at 127 74.93 0)
 			(show_name no)
@@
 			(project "xt8086_beta"
 				(path "/8c0b3d8b-46d3-4173-ab1e-a61765f77d61/fc69669c-5428-4356-8e92-0aa932a39979/e922aa3b-a7c2-5123-b7ae-6a56da586377"
-					(reference "U20")
+					(reference "U18")
 					(unit 1)
 				)
@@
 		(in_pos_files no)
 		(dnp no)
-		(property "Reference" "#PWR0191"
+		(property "Reference" "#PWR0189"
 			(at 199.39 81.28 0)
 			(hide yes)
@@
 			(project "xt8086_beta"
 				(path "/8c0b3d8b-46d3-4173-ab1e-a61765f77d61/fc69669c-5428-4356-8e92-0aa932a39979/e922aa3b-a7c2-5123-b7ae-6a56da586377"
-					(reference "#PWR0191")
+					(reference "#PWR0189")
 					(unit 1)
 				)
@@
 		(in_pos_files yes)
 		(dnp no)
-		(property "Reference" "R50"
+		(property "Reference" "R51"
 			(at 110.49 90.17 0)
 			(show_name no)
@@
 			(project "xt8086_beta"
 				(path "/8c0b3d8b-46d3-4173-ab1e-a61765f77d61/fc69669c-5428-4356-8e92-0aa932a39979/e922aa3b-a7c2-5123-b7ae-6a56da586377"
-					(reference "R50")
+					(reference "R51")
 					(unit 1)
 				)
@@
 		(dnp no)
 		(fields_autoplaced yes)
-		(property "Reference" "#PWR0182"
+		(property "Reference" "#PWR0180"
 			(at 104.14 71.12 0)
 			(hide yes)
@@
 			(project "xt8086_beta"
 				(path "/8c0b3d8b-46d3-4173-ab1e-a61765f77d61/fc69669c-5428-4356-8e92-0aa932a39979/e922aa3b-a7c2-5123-b7ae-6a56da586377"
-					(reference "#PWR0182")
+					(reference "#PWR0180")
 					(unit 1)
 				)
@@
 		(in_pos_files yes)
 		(dnp no)
-		(property "Reference" "R53"
+		(property "Reference" "R54"
 			(at 215.9 86.36 90)
 			(show_name no)
@@
 			(project "xt8086_beta"
 				(path "/8c0b3d8b-46d3-4173-ab1e-a61765f77d61/fc69669c-5428-4356-8e92-0aa932a39979/e922aa3b-a7c2-5123-b7ae-6a56da586377"
-					(reference "R53")
+					(reference "R54")
 					(unit 1)
 				)
@@
 		(dnp no)
 		(fields_autoplaced yes)
-		(property "Reference" "#PWR0187"
+		(property "Reference" "#PWR0185"
 			(at 139.7 90.17 0)
 			(hide yes)
@@
 			(project "xt8086_beta"
 				(path "/8c0b3d8b-46d3-4173-ab1e-a61765f77d61/fc69669c-5428-4356-8e92-0aa932a39979/e922aa3b-a7c2-5123-b7ae-6a56da586377"
-					(reference "#PWR0187")
+					(reference "#PWR0185")
 					(unit 1)
 				)
@@
 		(in_pos_files yes)
 		(dnp no)
-		(property "Reference" "LD3"
+		(property "Reference" "D6"
 			(at 229.87 87.63 0)
 			(show_name no)
@@
 			(project "xt8086_beta"
 				(path "/8c0b3d8b-46d3-4173-ab1e-a61765f77d61/fc69669c-5428-4356-8e92-0aa932a39979/e922aa3b-a7c2-5123-b7ae-6a56da586377"
-					(reference "LD3")
+					(reference "D6")
 					(unit 1)
 				)
@@
 		(dnp no)
 		(fields_autoplaced yes)
-		(property "Reference" "#PWR0190"
+		(property "Reference" "#PWR0188"
 			(at 153.67 88.9 0)
 			(hide yes)
@@
 			(project "xt8086_beta"
 				(path "/8c0b3d8b-46d3-4173-ab1e-a61765f77d61/fc69669c-5428-4356-8e92-0aa932a39979/e922aa3b-a7c2-5123-b7ae-6a56da586377"
-					(reference "#PWR0190")
+					(reference "#PWR0188")
 					(unit 1)
 				)
@@
 		(dnp no)
 		(fields_autoplaced yes)
-		(property "Reference" "#PWR0180"
+		(property "Reference" "#PWR0178"
 			(at 95.25 88.9 0)
 			(hide yes)
@@
 			(project "xt8086_beta"
 				(path "/8c0b3d8b-46d3-4173-ab1e-a61765f77d61/fc69669c-5428-4356-8e92-0aa932a39979/e922aa3b-a7c2-5123-b7ae-6a56da586377"
-					(reference "#PWR0180")
+					(reference "#PWR0178")
 					(unit 1)
 				)
@@
 		(in_pos_files no)
 		(dnp no)
-		(property "Reference" "#PWR0178"
+		(property "Reference" "#PWR0176"
 			(at 76.2 54.61 0)
 			(hide yes)
@@
 			(project "xt8086_beta"
 				(path "/8c0b3d8b-46d3-4173-ab1e-a61765f77d61/fc69669c-5428-4356-8e92-0aa932a39979/e922aa3b-a7c2-5123-b7ae-6a56da586377"
-					(reference "#PWR0178")
+					(reference "#PWR0176")
 					(unit 1)
 				)
@@
 		(in_pos_files yes)
 		(dnp no)
-		(property "Reference" "U21"
+		(property "Reference" "U19"
 			(at 127 110.49 0)
 			(show_name no)
@@
 			(project "xt8086_beta"
 				(path "/8c0b3d8b-46d3-4173-ab1e-a61765f77d61/fc69669c-5428-4356-8e92-0aa932a39979/e922aa3b-a7c2-5123-b7ae-6a56da586377"
-					(reference "U21")
+					(reference "U19")
 					(unit 1)
 				)
@@
 			)
 		)
-		(property "Value" "100uF"
+		(property "Value" "100u"
 			(at 91.44 72.39 0)
 			(show_name no)
@@
 		(dnp no)
 		(fields_autoplaced yes)
-		(property "Reference" "#PWR0189"
+		(property "Reference" "#PWR0187"
 			(at 146.05 127 0)
 			(hide yes)
@@
 			(project "xt8086_beta"
 				(path "/8c0b3d8b-46d3-4173-ab1e-a61765f77d61/fc69669c-5428-4356-8e92-0aa932a39979/e922aa3b-a7c2-5123-b7ae-6a56da586377"
-					(reference "#PWR0189")
+					(reference "#PWR0187")
 					(unit 1)
 				)
@@
 		(dnp no)
 		(fields_autoplaced yes)
-		(property "Reference" "#PWR0184"
+		(property "Reference" "#PWR0182"
 			(at 110.49 129.54 0)
 			(hide yes)
@@
 			(project "xt8086_beta"
 				(path "/8c0b3d8b-46d3-4173-ab1e-a61765f77d61/fc69669c-5428-4356-8e92-0aa932a39979/e922aa3b-a7c2-5123-b7ae-6a56da586377"
-					(reference "#PWR0184")
+					(reference "#PWR0182")
 					(unit 1)
 				)
@@
 		(in_pos_files yes)
 		(dnp no)
-		(property "Reference" "R52"
+		(property "Reference" "R53"
 			(at 201.93 97.79 0)
 			(show_name no)
@@
 			(project "xt8086_beta"
 				(path "/8c0b3d8b-46d3-4173-ab1e-a61765f77d61/fc69669c-5428-4356-8e92-0aa932a39979/e922aa3b-a7c2-5123-b7ae-6a56da586377"
-					(reference "R52")
+					(reference "R53")
 					(unit 1)
 				)
@@
 			)
 		)
-		(property "Value" "100uF"
+		(property "Value" "100u"
 			(at 106.68 72.39 0)
 			(show_name no)
@@
 		(dnp no)
 		(fields_autoplaced yes)
-		(property "Reference" "#PWR0179"
+		(property "Reference" "#PWR0177"
 			(at 88.9 71.12 0)
 			(hide yes)
@@
 			(project "xt8086_beta"
 				(path "/8c0b3d8b-46d3-4173-ab1e-a61765f77d61/fc69669c-5428-4356-8e92-0aa932a39979/e922aa3b-a7c2-5123-b7ae-6a56da586377"
-					(reference "#PWR0179")
-					(unit 1)
-				)
+					(reference "#PWR0177")
+					(unit 1)
+				)

Commit message: feat: xt8086_beta gets Dino's sound and schematic changes
xt8086_beta and dino_z80 share their platform, so everything done to the
Dino schematic is carried over:

- Buzzer sheet replaced by Dino's Sound + Speaker sheets: LM358 line out,
  PAM8403 driving a CVS-2308 speaker, S2 as HDMI L/R + speaker enable,
  stereo HDMI audio (AUDIO_IN_L/R no longer tied together).
- GP46 is PWM_L, GP44 is PWM_R, exactly as on Dino; J1 (UART) is gone
  and GP45 is left unconnected.
- USB defaults to the RP2350: R3 pulls SW low, S1's common goes to +3V3,
  JP3 (USB Test) straps SW high.
- H1-H4 become 2.5 mm pad-and-via holes tied to GND.
- MS9288A footprint renamed QFN-48_6x6mm.
- Shared sheets take Dino's current versions with xt8086_beta's own
  references; SI values, X1 renamed Y2, datasheet links fixed, plus TI
  SN74LS74A and Analog Devices DS3231M links for xt-only parts.
- Libraries: PAM8403D, LM358, CVS-2308, MountingHole_Pad symbols and
  their footprints/3D models; SOT-23 pad mirror fix and SOIC-8 from Dino.

dino.kicad_sym also gains CVS-2308 and MountingHole_Pad, which Dino's
schematic had only in its symbol cache.

ERC: 0. The board is not updated yet.
Parts:
- C89, C92: value 100u -> 100µF
- C90, C91: value 10u -> 10µF
- C93, C94: value 100n -> 100nF
- R51, R52, R53: value 100K -> 100kΩ
- R54: value 1K -> 1kΩ
Other:
- company: (none) -> Mikhail Matveev
- title: USB-A Port Power -> ${NAME} ${MODEL}
Changed lines of the file:
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@@
 	(paper "A4")
 	(title_block
-		(title "USB-A Port Power")
+		(title "${NAME} ${MODEL}")
+		(date "${DATE}")
+		(rev "${VERSION}")
+		(company "Mikhail Matveev")
+		(comment 1 "https://github.com/rh1tech/frank")
 	)
 	(junction
@@
 			)
 		)
-		(property "Value" "100K"
+		(property "Value" "100kΩ"
 			(at 111.76 130.81 0)
 			(show_name no)
@@
 			)
 		)
-		(property "Value" "100n"
+		(property "Value" "100nF"
 			(at 156.21 90.17 0)
 			(show_name no)
@@
 			)
 		)
-		(property "Value" "100K"
+		(property "Value" "100kΩ"
 			(at 110.49 92.71 0)
 			(show_name no)
@@
 			)
 		)
-		(property "Value" "10u"
+		(property "Value" "10µF"
 			(at 104.14 128.27 0)
 			(show_name no)
@@
 			)
 		)
-		(property "Value" "1K"
+		(property "Value" "1kΩ"
 			(at 215.9 88.9 90)
 			(show_name no)
@@
 			)
 		)
-		(property "Value" "10u"
+		(property "Value" "10µF"
 			(at 97.79 90.17 0)
 			(show_name no)
@@
 			)
 		)
-		(property "Value" "100n"
+		(property "Value" "100nF"
 			(at 148.59 128.27 0)
 			(show_name no)
@@
 			)
 		)
-		(property "Value" "100u"
+		(property "Value" "100µF"
 			(at 91.44 72.39 0)
 			(show_name no)
@@
 			)
 		)
-		(property "Value" "100K"
+		(property "Value" "100kΩ"
 			(at 201.93 100.33 0)
 			(show_name no)
@@
 			)
 		)
-		(property "Value" "100u"
+		(property "Value" "100µF"
 			(at 106.68 72.39 0)
 			(show_name no)

Commit message: fix: board review round - protection, pull-ups, parts data
- MS9288A config I2C pull-ups (SCL/SDA) go to +3V3; the chip's pins
  are rated only to DVDD33 + 0.5 V, and the reference leaves them open
- MS9288A audio inputs: 0 Ohm series + 10 kOhm shunt (not fitted) ahead
  of the coupling caps, so the reference 1/2 divider can be fitted later
- HDMI +5 V pin: 0.2 A resettable fuse (F2, 0603) in series with D5
- SD card: 10 kOhm pull-ups on CMD, DAT0 and DAT3 (SPI mode)
- xt8086: U1 is a 74HCT04 buffering GP29 to a 5 V 8086 CLK; RESET gets a
  10 kOhm pull-up so the CPU is held in reset until the RP2350 drives it
- video ladder and headphone series resistors 400/800 -> 402/806 Ohm
- LCSC part numbers checked against JLC for 452 parts; wrong numbers on
  R57, the 4.7 uF caps and the USB-C connector fixed
- MS9288A symbol: pin 3 is NC, datasheet linked; CD4069 pin name fixed
- Dino board follows the schematic renumbering; label and via clean-up
Parts:
- C89, C92: LCSC (none) -> C48935385
- C90, C91: LCSC (none) -> C19702
- C93, C94: LCSC (none) -> C14663
- D6: LCSC (none) -> C84256
- R51, R52, R53: LCSC (none) -> C25803
- R54: LCSC (none) -> C21190
- U18, U19: LCSC (none) -> C7462749
Changed lines of the file:
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@@
+			)
+		)
+		(property "LCSC" "C25803"
+			(at 110.49 129.54 0)
+			(hide yes)
+			(show_name no)
+			(do_not_autoplace no)
+			(effects
+				(font
+					(size 1.27 1.27)
+				)
 			)
 		)
@@
 			)
 		)
+		(property "LCSC" "C14663"
+			(at 153.67 88.9 0)
+			(hide yes)
+			(show_name no)
+			(do_not_autoplace no)
+			(effects
+				(font
+					(size 1.27 1.27)
+				)
+			)
+		)
 		(property "Description" "Unpolarized capacitor"
 			(at 153.67 88.9 0)
@@
 			)
 		)
+		(property "LCSC" "C7462749"
+			(at 127 83.82 0)
+			(hide yes)
+			(show_name no)
+			(do_not_autoplace no)
+			(effects
+				(font
+					(size 1.27 1.27)
+				)
+			)
+		)
 		(property "Description" ""
 			(at 127 83.82 0)
@@
 			)
 		)
+		(property "LCSC" "C25803"
+			(at 107.95 91.44 0)
+			(hide yes)
+			(show_name no)
+			(do_not_autoplace no)
+			(effects
+				(font
+					(size 1.27 1.27)
+				)
+			)
+		)
 		(property "Description" "Resistor"
 			(at 107.95 91.44 0)
@@
 		)
 		(property "Datasheet" ""
+			(at 101.6 127 0)
+			(hide yes)
+			(show_name no)
+			(do_not_autoplace no)
+			(effects
+				(font
+					(size 1.27 1.27)
+				)
+			)
+		)
+		(property "LCSC" "C19702"
 			(at 101.6 127 0)
 			(hide yes)
@@
 			)
 		)
+		(property "LCSC" "C21190"
+			(at 215.9 91.44 0)
+			(hide yes)
+			(show_name no)
+			(do_not_autoplace no)
+			(effects
+				(font
+					(size 1.27 1.27)
+				)
+			)
+		)
 		(property "Description" "Resistor"
 			(at 215.9 91.44 0)
@@
 			)
 		)
+		(property "LCSC" "C19702"
+			(at 95.25 88.9 0)
+			(hide yes)
+			(show_name no)
+			(do_not_autoplace no)
+			(effects
+				(font
+					(size 1.27 1.27)
+				)
+			)
+		)
 		(property "Description" "Unpolarized capacitor"
 			(at 95.25 88.9 0)
@@
 			)
 		)
+		(property "LCSC" "C84256"
+			(at 228.6 91.44 0)
+			(hide yes)
+			(show_name no)
+			(do_not_autoplace no)
+			(effects
+				(font
+					(size 1.27 1.27)
+				)
+			)
+		)
 		(property "Description" "Light emitting diode"
 			(at 228.6 91.44 0)
@@
 		)
 		(property "Datasheet" ""
+			(at 146.05 127 0)
+			(hide yes)
+			(show_name no)
+			(do_not_autoplace no)
+			(effects
+				(font
+					(size 1.27 1.27)
+				)
+			)
+		)
+		(property "LCSC" "C14663"
 			(at 146.05 127 0)
 			(hide yes)
@@
 			)
 		)
+		(property "LCSC" "C7462749"
+			(at 127 121.92 0)
+			(hide yes)
+			(show_name no)
+			(do_not_autoplace no)
+			(effects
+				(font
+					(size 1.27 1.27)
+				)
+			)
+		)
 		(property "Description" ""
 			(at 127 121.92 0)
@@
 		)
 		(property "Datasheet" ""
+			(at 88.9 71.12 0)
+			(hide yes)
+			(show_name no)
+			(do_not_autoplace no)
+			(effects
+				(font
+					(size 1.27 1.27)
+				)
+			)
+		)
+		(property "LCSC" "C48935385"
 			(at 88.9 71.12 0)
 			(hide yes)
@@
 			)
 		)
+		(property "LCSC" "C25803"
+			(at 199.39 99.06 0)
+			(hide yes)
+			(show_name no)
+			(do_not_autoplace no)
+			(effects
+				(font
+					(size 1.27 1.27)
+				)
+			)
+		)
 		(property "Description" "Resistor"
 			(at 199.39 99.06 0)
@@
 			(at 104.14 71.12 0)
 			(hide yes)
+			(show_name no)
+			(do_not_autoplace no)
+			(effects
+				(font
+					(size 1.27 1.27)
+				)
+			)
+		)
+		(property "LCSC" "C48935385"
+			(at 104.14 71.12 0)
+			(hide yes)

Commit message: fix: xt8086_beta 1.04 - pre-production review, TVS input, labels, release
- Power: SMAJ15A TVS D7 after the fuse (C908769, optional fit); Q1 gate
  divider R22/R23 100K/43K (Vgs within +-12 V at the TVS clamp); MP1584 UVLO
  R25/R26 300K/100K (start ~6.0 V); C44 680u 25V (C46550437); notes fixed
- Every capacitor value carries its voltage (from the LCSC part)
- Test points on all rails, on the back
- ERC: connector/hub pin types, PWR_FLAGs; 49 stale exclusions removed.
  ERC 0 errors, 0 warnings
- RP2350 exposed-pad vias tagged heatsink (no type mismatch)
- Fields: LCSC numbers removed from solder jumpers, S1/U1/U2/Y2/L1 part
  data and datasheet links corrected
- Layout: vias moved out of signal/power pads where a 45-degree escape
  exists, corners fixed, reference labels 0.7 mm bold re-placed
- Release 1.04: gerbers, schematics, assembly PDF, iBOM
  (DRC 0 violations, 0 unconnected, 0 parity)
Parts:
- C89, C92: value 100µF -> 100u 25V
- C90, C91: value 10µF -> 10u 10V
- C93, C94: value 100nF -> 100n 50V
Changed lines of the file:
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@@
 			)
 		)
-		(property "Value" "100nF"
+		(property "Value" "100n 50V"
 			(at 156.21 90.17 0)
 			(show_name no)
@@
 			)
 		)
-		(property "Value" "10µF"
+		(property "Value" "10u 10V"
 			(at 104.14 128.27 0)
 			(show_name no)
@@
 			)
 		)
-		(property "Value" "10µF"
+		(property "Value" "10u 10V"
 			(at 97.79 90.17 0)
 			(show_name no)
@@
 			)
 		)
-		(property "Value" "100nF"
+		(property "Value" "100n 50V"
 			(at 148.59 128.27 0)
 			(show_name no)
@@
 			)
 		)
-		(property "Value" "100µF"
+		(property "Value" "100u 25V"
 			(at 91.44 72.39 0)
 			(show_name no)
@@
 			)
 		)
-		(property "Value" "100µF"
+		(property "Value" "100u 25V"
 			(at 106.68 72.39 0)
 			(show_name no)
