File: frank_zx/frank_zx.kicad_pcb (KiCad board)
At the start: 4 copper layers, 210 x 120.4 mm, 240 parts, among them J1 Debug, J11 USB4215-03-A, J12 676430910, J13 676430910, J14 676430910, J2 UART, J3 DC3RX19JA2, J6 104031-0811, J7 PJ-320D, J8 DF13-2P-1.25DSA, J9 PJ-320D, K00 MX, K01 MX, K02 MX, K03 MX, K04 MX, K05 MX, K06 MX, K07 MX, K08 MX, K09 MX, K10 MX, K11 MX, K12 MX, K13 MX, K14 MX, K15 MX, K16 MX, K17 MX, K18 MX, K19 MX, K20 MX, K21 MX, K22 MX, K23 MX, K24 MX, K25 MX, K26 MX, K27 MX, K28 MX, K29 MX, K30 MX, K31 MX, K32 MX, K33 MX, K34 MX, K35 MX, K36 MX, K37 MX, K38 MX, K39 MX, Q2 BC850, Q3 BC850, U1 APS6404L-3SQR-ZR, U14 TPD4S012DRYR, U16 AO3401A, U17 TS3USB221RSER, U18 SY8089AAAC, U19 CH334F, U2 W25Q128JVPIQ, U21 TPD4S012DRYR, U22 CH217K, U23 TPD4S012DRYR, U24 CH217K, U25 TPD4S012DRYR, U27 CH217K, U3 RP2350B, U7 TLV320DAC3100IRHBR, U8 XC6206P182MR-G, U9 ESP-01v090, Y1 12 MHz, Y4 12 MHz

Commit message: Board updates
Parts:
- moved C53 2.70 mm to (126.6, 47.7)
- moved C54 2.70 mm to (129.9, 50.9)
- moved R36 2.70 mm to (129.9, 56.0)
- moved R37 2.70 mm to (120.9, 56.0)
- moved R38 2.70 mm to (132.1, 53.5)
- moved R39 2.70 mm to (120.9, 52.2)
- moved U9 2.70 mm to (126.6, 58.6)
Changed lines of the file:
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@@
 	(footprint "FRANK:ESP-01S"
 		(layer "F.Cu")
-		(at 126.593039 61.26392 180)
+		(at 126.643039 58.56392 180)
 		(descr "Module, ESP-8266, ESP-01, 8 pin")
 		(tags "Module ESP-8266 ESP8266")
 		(property "Reference" "U9"
-			(at 5.1 -1.5 270)
+			(at 4.194891 -0.938944 180)
 			(layer "F.SilkS")
 			(effects
@@
 	(footprint "FRANK:R_0603_1608Metric"
 		(layer "B.Cu")
-		(at 132.093039 56.18392 90)
+		(at 132.143039 53.48392 90)
 		(descr "Resistor SMD 0603 (1608 Metric), square (rectangular) end terminal, IPC-7351 nominal, (Body size source: IPC-SM-782 page 72, https://www.pcb-3d.com/wordpress/wp-content/uploads/ipc-sm-782a_amendment_1_and_2.pdf), generated with kicad-footprint-generator")
 		(tags "resistor")
@@
 	(footprint "FRANK:C_0603_1608Metric"
 		(layer "B.Cu")
-		(at 126.593039 50.39392)
+		(at 126.643039 47.69392)
 		(descr "Capacitor SMD 0603 (1608 Metric), square (rectangular) end terminal, IPC-7351 nominal, (Body size source: IPC-SM-782 page 76, https://www.pcb-3d.com/wordpress/wp-content/uploads/ipc-sm-782a_amendment_1_and_2.pdf), generated with kicad-footprint-generator")
 		(tags "capacitor")
@@
 	(footprint "FRANK:R_0603_1608Metric"
 		(layer "B.Cu")
-		(at 120.803039 54.93392 90)
+		(at 120.853039 52.23392 90)
 		(descr "Resistor SMD 0603 (1608 Metric), square (rectangular) end terminal, IPC-7351 nominal, (Body size source: IPC-SM-782 page 72, https://www.pcb-3d.com/wordpress/wp-content/uploads/ipc-sm-782a_amendment_1_and_2.pdf), generated with kicad-footprint-generator")
 		(tags "resistor")
@@
 	(footprint "FRANK:R_0603_1608Metric"
 		(layer "B.Cu")
-		(at 129.843039 58.72392 90)
+		(at 129.893039 56.02392 90)
 		(descr "Resistor SMD 0603 (1608 Metric), square (rectangular) end terminal, IPC-7351 nominal, (Body size source: IPC-SM-782 page 72, https://www.pcb-3d.com/wordpress/wp-content/uploads/ipc-sm-782a_amendment_1_and_2.pdf), generated with kicad-footprint-generator")
 		(tags "resistor")
@@
 	(footprint "FRANK:R_0603_1608Metric"
 		(layer "B.Cu")
-		(at 120.803039 58.72392 90)
+		(at 120.853039 56.02392 90)
 		(descr "Resistor SMD 0603 (1608 Metric), square (rectangular) end terminal, IPC-7351 nominal, (Body size source: IPC-SM-782 page 72, https://www.pcb-3d.com/wordpress/wp-content/uploads/ipc-sm-782a_amendment_1_and_2.pdf), generated with kicad-footprint-generator")
 		(tags "resistor")
@@
 	(footprint "FRANK:C_0603_1608Metric"
 		(layer "B.Cu")
-		(at 129.843039 53.64392 90)
+		(at 129.893039 50.94392 90)
 		(descr "Capacitor SMD 0603 (1608 Metric), square (rectangular) end terminal, IPC-7351 nominal, (Body size source: IPC-SM-782 page 76, https://www.pcb-3d.com/wordpress/wp-content/uploads/ipc-sm-782a_amendment_1_and_2.pdf), generated with kicad-footprint-generator")
 		(tags "capacitor")
@@
 		(polygon
 			(pts
-				(xy 103.733039 50.34392) (xy 111.593039 50.34392) (xy 111.593039 64.56392) (xy 103.733039 64.56392)
+				(xy 103.783039 47.64392) (xy 111.643039 47.64392) (xy 111.643039 61.86392) (xy 103.783039 61.86392)
 			)
 		)

Commit message: FRANK ZX WIP
Parts:
- removed D3: 1N4148WS, FRANK:D_SOD-323
- removed Q2, Q3: BC850, FRANK:SOT-23
- removed R47: 10K, FRANK:R_0603_1608Metric
- removed R48: 1K, FRANK:R_0603_1608Metric
- added C102: 100nF, FRANK:C_0603_1608Metric, B.Cu at (249.8, 34.6)
- added D40: 1N5819WS, FRANK:D_SOD-323, B.Cu at (244.9, 34.6)
- added LD1: WS2812B-2020, FRANK:LED_WS2812B-2020_PLCC4_2.0x2.0mm, F.Cu at (248.4, 31.7)
- added LD2: Blue, FRANK:LED_0603_1608Metric, F.Cu at (243.0, 29.8)
- added R71: 1K, FRANK:R_0603_1608Metric, B.Cu at (243.0, 41.8)
- added R72: 330R, FRANK:R_0603_1608Metric, B.Cu at (241.0, 42.2)
- added S3: RP Boot, FRANK:Button_SMD_TS1234VW, F.Cu at (257.1, 97.7)
- added S4: RP Reset, FRANK:Button_SMD_TS1234VW, F.Cu at (257.1, 110.3)
- added S5: ESP Reset, FRANK:Button_SMD_3x4x2mm, F.Cu at (137.5, 50.5)
- added S6: ESP Flash, FRANK:Button_SMD_3x4x2mm, F.Cu at (137.5, 56.5)
- added S7: ESP Reset, FRANK:Button_SMD_TS1234VW, F.Cu at (50.9, 43.7)
- added U28: CD4069UBM, FRANK:SOIC127P600X175-14N, F.Cu at (91.3, 37.0)
- C2, C3, C4, C5, C6, C8, C86, C87, R4, R6, R9: moved to F.Cu
- R44: value 100R -> 4.7K
- R45, R46: value 10K -> 100K
- S1, S2: footprint FRANK:Button_SMD_3x4x2mm_2P -> FRANK:Button_SMD_3x4x2mm
- U1: moved to B.Cu
- moved S8 208.2 mm to (257.1, 83.8), turned to 90 degrees
- moved JP5 197.5 mm to (252.2, 80.8)
- moved LD3 118.8 mm to (170.1, 30.1)
- moved R57 118.8 mm to (170.9, 30.1)
- moved C85 31.5 mm to (173.6, 57.3)
- moved C89 30.3 mm to (180.4, 56.1), turned to 180 degrees
- moved C84 30.0 mm to (175.3, 57.3), turned to 90 degrees
- moved R16 28.8 mm to (250.5, 69.4), turned to 180 degrees
- moved Y4 28.3 mm to (180.3, 52.9), turned to -90 degrees
- moved U19 27.8 mm to (174.2, 52.7)
- moved R21 27.4 mm to (197.6, 54.7), turned to 180 degrees
- moved R18 26.8 mm to (197.6, 49.6), turned to 180 degrees
- moved C90 26.8 mm to (180.2, 49.9)
- moved S1 26.8 mm to (247.3, 37.9)
- moved C52 26.4 mm to (79.8, 63.1), turned to 180 degrees
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Connections:
- C67 pad 1: /Tape/TAPE -> Net-(C67-Pad1)
- C67 pad 2: Net-(C67-Pad2) -> /Tape/TAPE
- C68 pad 1: GND -> +3V3
- C68 pad 2: +3V3 -> GND
- R44 pad 1: /Tape/TAPE -> Net-(U28-A)
- R44 pad 2: GND -> Net-(C67-Pad1)
- R45 pad 1: Net-(C67-Pad2) -> Net-(U28-G-*A)
- R45 pad 2: Net-(D3-K) -> Net-(U28-A)
- R46 pad 1: +3V3 -> Net-(U28-B)
- R46 pad 2: Net-(D3-A) -> Net-(U28-G-*A)
- U3 pad 43: unconnected-(U3-GPIO34-Pad43) -> /RP2350B/LED
- U3 pad 44: unconnected-(U3-GPIO35-Pad44) -> /RP2350B/RGB_LED
Routing:
- net /GPIO20/COL0: track 0.00 -> 254.8 mm, vias 0 -> 3
- net /GPIO33/ROW3: track 0.00 -> 246.7 mm, vias 0 -> 1
- net VBUS: track 0.00 -> 241.6 mm, vias 0 -> 11
- net /GPIO30/ROW0: track 0.00 -> 233.2 mm, vias 0 -> 1
- net /GPIO32/ROW2: track 0.00 -> 232.8 mm, vias 0 -> 3
- net /GPIO21/COL1: track 0.00 -> 230.1 mm, vias 0 -> 3
- net /GPIO31/ROW1: track 0.00 -> 214.6 mm, vias 0 -> 3
- net /GPIO38/ESP_RST: track 0.00 -> 207.4 mm, vias 0 -> 4
- net /GPIO22/COL2: track 0.00 -> 198.0 mm, vias 0 -> 3
- net /GPIO3/SCL: track 0.00 -> 196.3 mm, vias 0 -> 3
- net /RP2350B/RUN: track 0.00 -> 196.2 mm, vias 0 -> 3
- net /GPIO2/SDA: track 0.00 -> 195.4 mm, vias 0 -> 3
- net /GPIO23/COL3: track 0.00 -> 173.4 mm, vias 0 -> 3
- net /RP2350B/GPIO44: track 0.00 -> 166.7 mm
- net /GPIO24/COL4: track 0.00 -> 152.9 mm, vias 0 -> 1
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- added copper zone on In2.Cu, net +1V1
- added copper zone on In2.Cu, net +3V3
- added copper zone on B.Cu, net GND
- added copper zone on F.Cu, net GND
Other:
- board size 210 x 120.4 mm -> 210 x 120 mm

Commit message: Board updates
Parts:
- added C103: 100nF, FRANK:C_0603_1608Metric, B.Cu at (77.5, 63.1)
- added H5: MountingHole, FRANK:MountingHole_2.5mm_Pad_Via, F.Cu at (51.9, 91.3)
- added H6: MountingHole, FRANK:MountingHole_2.5mm_Pad_Via, F.Cu at (256.2, 91.3)
- R60: value 1K -> 10K
- moved R63 17.0 mm to (196.2, 38.4)
- moved R62 17.0 mm to (197.8, 38.4)
- moved C91 16.8 mm to (194.6, 38.4)
Connections:
- net Net-(U7-~{RESET}) renamed /Audio/CODEC_RST
Routing:
- net GND: track 20.3 -> 64.0 mm, vias 35 -> 80
- net Net-(U18-FB): track 22.1 -> 5.66 mm
- net +3V3: track 53.2 -> 59.9 mm, vias 44 -> 43
- net /GPIO39/ESP_BOOT: track 110.2 -> 107.3 mm
- net /GPIO3/SCL: track 196.3 -> 193.4 mm
- net /GPIO2/SDA: track 195.4 -> 192.7 mm
- net /GPIO9/BCLK: track 143.3 -> 140.6 mm
- net /GPIO10/WCLK: track 142.0 -> 139.3 mm
- net /GPIO8/MCLK: track 144.7 -> 142.1 mm
- net /GPIO11/DIN: track 140.6 -> 138.0 mm
- net /Audio/CODEC_RST: track 4.82 -> 6.21 mm
- net Net-(C43-Pad1): track 43.6 -> 44.9 mm, vias 0 -> 2
- net /GPIO33/ROW3: track 246.7 -> 248.0 mm
- net /GPIO32/ROW2: track 232.8 -> 233.8 mm
- net /RP2350B/BOOT: track 103.3 -> 104.3 mm
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