File: frank_zx/usb.kicad_sch (KiCad schematic)
At the start: 41 parts, among them J11 USB4215-03-A, U14 TPD4S012DRYR, U16 AO3401A, U17 TS3USB221RSER, U18 SY8089AAAC, U19 CH334F, Y4 12 MHz

Commit message: Board updates
Parts:
- R60: value 1K -> 10K; LCSC C21190 -> C2906982
Changed lines of the file:
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@@
 			)
 		)
-		(property "Value" "1K"
+		(property "Value" "10K"
 			(at 161.29 83.82 90)
 			(show_name no)
@@
 			)
 		)
-		(property "LCSC" "C21190"
+		(property "LCSC" "C2906982"
 			(at 158.75 83.82 0)
 			(hide yes)

Commit message: chore: clean up frank_zx and apply review fixes
Remove leftovers copied from frank_next/frank_core2 that frank_zx never
uses: the frank_next project files and its stale gerbers, the unused
ch343p/esp8266/esp_multiplex/rp2350a_slave/rtc sheets, the sy8089_buck
drawing, and 18 footprints plus 17 3D models no footprint on the board
references. release.sh picks the first *.kicad_pro in the folder, so the
stray frank_next.kicad_pro would have made it release the wrong project.

Also included:
- JST-SH J1/J2 footprint numbered to the KiCad/JST standard (pad 1 at
  x=-1); physical pin order matches frank_next_proto (SWCLK/RX, GND,
  SWDIO/TX)
- microSD symbol pin 9 renamed DAT1 -> CD (card detect, unconnected)
- zones refilled, clearing 26 stale-fill DRC violations
- pending sheet and layout edits, case STLs for 1.00

ERC 0, DRC 0 violations, 0 unconnected, 0 schematic parity issues.
Changed lines of the file:
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@@
 	(wire
 		(pts
-			(xy 109.22 121.92) (xy 109.22 124.46)
+			(xy 105.41 121.92) (xy 105.41 124.46)
 		)
 		(stroke
@@
 	(wire
 		(pts
-			(xy 101.6 121.92) (xy 101.6 124.46)
+			(xy 95.25 121.92) (xy 95.25 124.46)
 		)
 		(stroke
@@
 	(wire
 		(pts
-			(xy 124.46 124.46) (xy 127 124.46)
-		)
-		(stroke
-			(width 0)
-			(type default)
-		)
-	)
-	(wire
-		(pts
 			(xy 66.04 29.21) (xy 66.04 33.02)
 		)
@@
 	(wire
 		(pts
+			(xy 132.08 119.38) (xy 128.27 119.38)
+		)
+		(stroke
+			(width 0)
+			(type default)
+		)
+	)
+	(wire
+		(pts
 			(xy 132.08 74.93) (xy 142.24 74.93)
 		)
@@
 	(wire
 		(pts
-			(xy 124.46 121.92) (xy 124.46 124.46)
+			(xy 128.27 124.46) (xy 128.27 119.38)
 		)
 		(stroke
@@
 	)
 	(label "+5V_BUCK"
-		(at 127 124.46 0)
+		(at 132.08 119.38 180)
 		(effects
 			(font
 				(size 1.27 1.27)
 			)
-			(justify left bottom)
+			(justify right bottom)
 		)
 	)
@@
 	(symbol
 		(lib_id "FRANK:GND")
-		(at 101.6 124.46 0)
+		(at 95.25 124.46 0)
 		(unit 1)
 		(body_style 1)
@@
 		(dnp no)
 		(property "Reference" "#PWR0300"
-			(at 101.6 126.46 0)
+			(at 95.25 126.46 0)
 			(hide yes)
 			(show_name no)
@@
 		)
 		(property "Value" "GND"
-			(at 101.6 128.27 0)
+			(at 95.25 128.27 0)
 			(show_name no)
 			(do_not_autoplace no)
@@
 		)
 		(property "Footprint" ""
-			(at 101.6 124.46 0)
+			(at 95.25 124.46 0)
 			(hide yes)
 			(show_name no)
@@
 		)
 		(property "Datasheet" ""
-			(at 101.6 124.46 0)
+			(at 95.25 124.46 0)
 			(hide yes)
 			(show_name no)
@@
 		)
 		(property "Description" ""
-			(at 101.6 124.46 0)
+			(at 95.25 124.46 0)
 			(hide yes)
 			(show_name no)
@@
 	(symbol
 		(lib_id "FRANK:PWR_FLAG")
-		(at 101.6 121.92 0)
+		(at 95.25 121.92 0)
 		(unit 1)
 		(body_style 1)
@@
 		(dnp no)
 		(property "Reference" "#FLG001"
-			(at 101.6 123.92 0)
+			(at 95.25 123.92 0)
 			(hide yes)
 			(show_name no)
@@
 		)
 		(property "Value" "PWR_FLAG"
-			(at 101.6 118.11 0)
+			(at 95.25 118.11 0)
 			(show_name no)
 			(do_not_autoplace no)
@@
 		)
 		(property "Footprint" ""
-			(at 101.6 121.92 0)
+			(at 95.25 121.92 0)
 			(hide yes)
 			(show_name no)
@@
 		)
 		(property "Datasheet" ""
-			(at 101.6 121.92 0)
+			(at 95.25 121.92 0)
 			(hide yes)
 			(show_name no)
@@
 		)
 		(property "Description" ""
-			(at 101.6 121.92 0)
+			(at 95.25 121.92 0)
 			(hide yes)
 			(show_name no)
@@
 	(symbol
 		(lib_id "FRANK:PWR_FLAG")
-		(at 109.22 124.46 180)
+		(at 105.41 124.46 180)
 		(unit 1)
 		(body_style 1)
@@
 		(dnp no)
 		(property "Reference" "#FLG002"
-			(at 109.22 126.46 0)
+			(at 105.41 126.46 0)
 			(hide yes)
 			(show_name no)
@@
 		)
 		(property "Value" "PWR_FLAG"
-			(at 109.22 128.27 0)
+			(at 105.41 128.27 0)
 			(show_name no)
 			(do_not_autoplace no)
@@
 		)
 		(property "Footprint" ""
-			(at 109.22 124.46 0)
+			(at 105.41 124.46 0)
 			(hide yes)
 			(show_name no)
@@
 		)
 		(property "Datasheet" ""
-			(at 109.22 124.46 0)
+			(at 105.41 124.46 0)
 			(hide yes)
 			(show_name no)
@@
 		)
 		(property "Description" ""
-			(at 109.22 124.46 0)
+			(at 105.41 124.46 0)
 			(hide yes)
 			(show_name no)
@@
 	(symbol
 		(lib_id "FRANK:PWR_FLAG")
-		(at 124.46 121.92 0)
+		(at 128.27 124.46 180)
 		(unit 1)
 		(body_style 1)
@@
 		(dnp no)
 		(property "Reference" "#FLG004"
-			(at 124.46 123.92 0)
+			(at 128.27 122.46 0)
 			(hide yes)
 			(show_name no)
@@
 		)
 		(property "Value" "PWR_FLAG"
-			(at 124.46 118.11 0)
+			(at 128.27 128.27 0)
 			(show_name no)
 			(do_not_autoplace no)
@@
 		)
 		(property "Footprint" ""
-			(at 124.46 121.92 0)
+			(at 128.27 124.46 0)
 			(hide yes)
 			(show_name no)
@@
 		)
 		(property "Datasheet" ""
-			(at 124.46 121.92 0)
+			(at 128.27 124.46 0)
 			(hide yes)
 			(show_name no)
@@
 		)
 		(property "Description" ""
-			(at 124.46 121.92 0)
+			(at 128.27 124.46 0)
 			(hide yes)
 			(show_name no)
@@
 	(symbol
 		(lib_id "FRANK:VBUS")
-		(at 109.22 121.92 0)
+		(at 105.41 121.92 0)
 		(unit 1)
 		(body_style 1)
@@
 		(dnp no)
 		(property "Reference" "#PWR0301"
-			(at 109.22 123.92 0)
+			(at 105.41 123.92 0)
 			(hide yes)
 			(show_name no)
@@
 		)
 		(property "Value" "VBUS"
-			(at 109.22 118.11 0)
+			(at 105.41 118.11 0)
 			(show_name no)
 			(do_not_autoplace no)
@@
 		)
 		(property "Footprint" ""
-			(at 109.22 121.92 0)
+			(at 105.41 121.92 0)
 			(hide yes)
 			(show_name no)
@@
 		)
 		(property "Datasheet" ""
-			(at 109.22 121.92 0)
+			(at 105.41 121.92 0)
 			(hide yes)
 			(show_name no)
@@
 		)
 		(property "Description" ""
-			(at 109.22 121.92 0)
+			(at 105.41 121.92 0)
 			(hide yes)
 			(show_name no)

Commit message: feat: frank_zx test points, speaker pads, power header; re-release 1.00
- 21 round test points (FRANK:TestPoint_Pad_D1.2mm, back side), one per net:
  ESP TX/RX/RST/BOOT, RUN, I2C SDA/SCL, I2S MCLK/BCLK/WCLK/DIN,
  TAPE (GPIO44), +3V3, +1V1, +1V8, VBUS, VBUS_IN, +5V_BUCK, buck LX,
  hub VDD33, +5V_SPK. The buck switch node is now labelled /USB/LX.
- J15: 2.54 mm solder pads in parallel with the J8 speaker connector
- J16 PWR: 3V3 / GND / 5V 2.54 mm header as on megafrank, fed from the
  In2 +3V3 / VBUS planes and the GND plane
- Release 1.00 regenerated (2026-09-30): gerbers, schematics, assembly
  PDF, iBOM. ERC and DRC clean, 0 unconnected, 0 parity issues; every
  footprint path matches its schematic symbol.
Parts:
- added TP15: VBUS, FRANK:TestPoint_Pad_D1.2mm, symbol FRANK:TestPoint
- added TP16: VBUS_IN, FRANK:TestPoint_Pad_D1.2mm, symbol FRANK:TestPoint
- added TP17: +5V_BUCK, FRANK:TestPoint_Pad_D1.2mm, symbol FRANK:TestPoint
- added TP18: LX, FRANK:TestPoint_Pad_D1.2mm, symbol FRANK:TestPoint
- added TP19: VDD33, FRANK:TestPoint_Pad_D1.2mm, symbol FRANK:TestPoint
Connections:
- net +5V_BUCK: now also TP17.1
- net VBUS: now also TP15.1
- net VBUS_IN: now also TP16.1
- net VDD33: now also TP19.1
- net LX: now reaches L6.2, U18.3 (LX)
- net LX: now also TP18.1
