File: dino_z80/buck3v3.kicad_sch (KiCad schematic)
At the start: 14 parts, among them U17 SY8089AAAC

Commit message: feat: round test points on dino_z80 and xt8086_beta
Test points use the 1.0 mm round TestPoint_Pad_D1.0mm instead of the
square pad; placement, nets and labels are unchanged. Also includes the
latest xt8086_beta edits on the power, sound and speaker sheets and board.
Parts:
- TP10, TP11: footprint dino:TestPoint_Pad_1.0x1.0mm -> dino:TestPoint_Pad_D1.0mm
Changed lines of the file:
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@@
 			)
 		)
-		(property "Footprint" "dino:TestPoint_Pad_1.0x1.0mm"
+		(property "Footprint" "dino:TestPoint_Pad_D1.0mm"
 			(at 60.96 96.52 0)
 			(hide yes)
@@
 			)
 		)
-		(property "Footprint" "dino:TestPoint_Pad_1.0x1.0mm"
+		(property "Footprint" "dino:TestPoint_Pad_D1.0mm"
 			(at 163.83 99.06 0)
 			(hide yes)

Commit message: fix: board review round - protection, pull-ups, parts data
- MS9288A config I2C pull-ups (SCL/SDA) go to +3V3; the chip's pins
  are rated only to DVDD33 + 0.5 V, and the reference leaves them open
- MS9288A audio inputs: 0 Ohm series + 10 kOhm shunt (not fitted) ahead
  of the coupling caps, so the reference 1/2 divider can be fitted later
- HDMI +5 V pin: 0.2 A resettable fuse (F2, 0603) in series with D5
- SD card: 10 kOhm pull-ups on CMD, DAT0 and DAT3 (SPI mode)
- xt8086: U1 is a 74HCT04 buffering GP29 to a 5 V 8086 CLK; RESET gets a
  10 kOhm pull-up so the CPU is held in reset until the RP2350 drives it
- video ladder and headphone series resistors 400/800 -> 402/806 Ohm
- LCSC part numbers checked against JLC for 452 parts; wrong numbers on
  R57, the 4.7 uF caps and the USB-C connector fixed
- MS9288A symbol: pin 3 is NC, datasheet linked; CD4069 pin name fixed
- Dino board follows the schematic renumbering; label and via clean-up
Parts:
- C100: renamed from C99; LCSC (none) -> C1653
- C94: renamed from C93; LCSC (none) -> C19702
- C95: renamed from C94; LCSC (none) -> C19702
- C96: renamed from C95; LCSC (none) -> C14663
- C97: renamed from C96; LCSC (none) -> C15008
- C98: renamed from C97; LCSC (none) -> C19702
- C99: renamed from C98; LCSC (none) -> C14663
- FB4: LCSC (none) -> C74488
- L3: LCSC (none) -> C354563
- R80: renamed from R74; LCSC (none) -> C25803
- R81: renamed from R75; LCSC (none) -> C31850
- U18: renamed from U17; LCSC (none) -> C78988

Commit message: fix: dino_z80 1.02 - pre-production review, TVS input, labels, release
- Power: SMAJ15A TVS D7 after the fuse (C908769, optional fit); Q1 gate
  divider R47/R48 100K/43K (Vgs within +-12 V at the TVS clamp); MP1584 UVLO
  R50/R51 300K/100K (start ~6.0 V); C54 680u 25V (C46550437); notes fixed
- Every capacitor value carries its voltage (from the LCSC part)
- Test points on all rails, on the back
- ERC: connector/hub pin types, PWR_FLAGs; 49 stale exclusions removed.
  ERC 0 errors, 0 warnings
- RP2350 exposed-pad vias tagged heatsink (no type mismatch)
- Fields: LCSC numbers removed from solder jumpers, S1/U1/U2/Y2/L1 part
  data and datasheet links corrected
- Layout: vias moved out of signal/power pads where a 45-degree escape
  exists, corners fixed, reference labels 0.7 mm bold re-placed
- Release 1.02: gerbers, schematics, assembly PDF, iBOM
  (DRC 0 violations, 0 unconnected, 0 parity)
Parts:
- C100: value 22pF -> 22p 50V
- C94, C95, C98: value 10µF -> 10u 10V
- C96, C99: value 100nF -> 100n 50V
- C97: value 100µF -> 100u 6.3V
Changed lines of the file:
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@@
 			)
 		)
-		(property "Value" "10µF"
+		(property "Value" "10u 10V"
 			(at 115.57 95.25 0)
 			(show_name no)
@@
 			)
 		)
-		(property "Value" "100µF"
+		(property "Value" "100u 6.3V"
 			(at 182.88 95.25 0)
 			(show_name no)
@@
 			)
 		)
-		(property "Value" "100nF"
+		(property "Value" "100n 50V"
 			(at 125.73 95.25 0)
 			(show_name no)
@@
 			)
 		)
-		(property "Value" "10µF"
+		(property "Value" "10u 10V"
 			(at 105.41 95.25 0)
 			(show_name no)
@@
 			)
 		)
-		(property "Value" "10µF"
+		(property "Value" "10u 10V"
 			(at 191.77 95.25 0)
 			(show_name no)
@@
 			)
 		)
-		(property "Value" "22pF"
+		(property "Value" "22p 50V"
 			(at 227.33 95.25 0)
 			(show_name no)
@@
 			)
 		)
-		(property "Value" "100nF"
+		(property "Value" "100n 50V"
 			(at 200.66 95.25 0)
 			(show_name no)
