File: dino_z80/speaker.kicad_sch (KiCad schematic)
At the start: 14 parts, among them U6 PAM8403D

Commit message: fix: pre-production review changes on dino_z80 and xt8086_beta
- AMS1117-1.8 output cap is a 22 uF 3528 tantalum on the top side
  (C87 on Dino, C76 on xt); the regulator needs it for stability
- speaker is the 1 W 8 Ohm 2308, not the 0.15 W CVS-2308
- micro SD socket value is Wurth 693072010801, matching its datasheet
- power sheet notes the 9-12 V input range and the >=16 V rating for
  the input capacitors
Parts:
- LS1: value CVS-2308 -> 2308 1W 8Ω
Changed lines of the file:
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@@
 			)
 		)
-		(property "Value" "CVS-2308"
+		(property "Value" "2308 1W 8Ω"
 			(at 99.303 95.25 90)
 			(show_name no)
@@
 			)
 		)
-		(property "Description" "23 mm round loudspeaker, 8Ω"
+		(property "Description" "23×6.8 mm round loudspeaker, 8Ω, 1 W"
 			(at 113.03 93.98 0)
 			(hide yes)

Commit message: fix: board review round - protection, pull-ups, parts data
- MS9288A config I2C pull-ups (SCL/SDA) go to +3V3; the chip's pins
  are rated only to DVDD33 + 0.5 V, and the reference leaves them open
- MS9288A audio inputs: 0 Ohm series + 10 kOhm shunt (not fitted) ahead
  of the coupling caps, so the reference 1/2 divider can be fitted later
- HDMI +5 V pin: 0.2 A resettable fuse (F2, 0603) in series with D5
- SD card: 10 kOhm pull-ups on CMD, DAT0 and DAT3 (SPI mode)
- xt8086: U1 is a 74HCT04 buffering GP29 to a 5 V 8086 CLK; RESET gets a
  10 kOhm pull-up so the CPU is held in reset until the RP2350 drives it
- video ladder and headphone series resistors 400/800 -> 402/806 Ohm
- LCSC part numbers checked against JLC for 452 parts; wrong numbers on
  R57, the 4.7 uF caps and the USB-C connector fixed
- MS9288A symbol: pin 3 is NC, datasheet linked; CD4069 pin name fixed
- Dino board follows the schematic renumbering; label and via clean-up
Parts:
- C15: LCSC (none) -> C1631
- C16, C17: LCSC (none) -> C15849
- C18: LCSC (none) -> C14663
- C19: LCSC (none) -> C19702
- C20: LCSC (none) -> C48935385
- R25, R26: LCSC (none) -> C31850
- R27: LCSC (none) -> C22975
- R28, R29, R30: LCSC (none) -> C25804
- U6: LCSC (none) -> C17337
Changed lines of the file:
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@@
 		(in_pos_files yes)
 		(dnp no)
-		(property "Reference" "#PWR062"
+		(property "Reference" "#PWR066"
 			(at 182.88 100.33 0)
 			(hide yes)
@@
 			(project "dino_z80"
 				(path "/8c0b3d8b-46d3-4173-ab1e-a61765f77d61/3603a3f9-aa53-493b-ae79-e24b3c1f7362/128bfa67-3568-45ab-9ac5-06e6eea36fac"
-					(reference "#PWR062")
+					(reference "#PWR066")
 					(unit 1)
 				)
@@
 		(in_pos_files yes)
 		(dnp no)
-		(property "Reference" "#PWR067"
+		(property "Reference" "#PWR070"
 			(at 194.31 114.3 0)
 			(hide yes)
@@
 			(project "dino_z80"
 				(path "/8c0b3d8b-46d3-4173-ab1e-a61765f77d61/3603a3f9-aa53-493b-ae79-e24b3c1f7362/128bfa67-3568-45ab-9ac5-06e6eea36fac"
-					(reference "#PWR067")
+					(reference "#PWR070")
 					(unit 1)
 				)
@@
 			)
 		)
+		(property "LCSC" "C22975"
+			(at 110.49 118.11 0)
+			(hide yes)
+			(show_name no)
+			(do_not_autoplace no)
+			(effects
+				(font
+					(size 1.27 1.27)
+				)
+			)
+		)
 		(pin "1"
 		)
@@
 			)
 		)
+		(property "LCSC" "C48935385"
+			(at 173.99 72.39 0)
+			(hide yes)
+			(show_name no)
+			(do_not_autoplace no)
+			(effects
+				(font
+					(size 1.27 1.27)
+				)
+			)
+		)
 		(pin "1"
 		)
@@
 			)
 		)
+		(property "LCSC" "C25804"
+			(at 194.31 97.79 0)
+			(hide yes)
+			(show_name no)
+			(do_not_autoplace no)
+			(effects
+				(font
+					(size 1.27 1.27)
+				)
+			)
+		)
 		(pin "1"
 		)
@@
 		(in_pos_files yes)
 		(dnp no)
-		(property "Reference" "#PWR061"
+		(property "Reference" "#PWR065"
 			(at 173.99 81.28 0)
 			(hide yes)
@@
 			(project "dino_z80"
 				(path "/8c0b3d8b-46d3-4173-ab1e-a61765f77d61/3603a3f9-aa53-493b-ae79-e24b3c1f7362/128bfa67-3568-45ab-9ac5-06e6eea36fac"
-					(reference "#PWR061")
+					(reference "#PWR065")
 					(unit 1)
 				)
@@
 			)
 		)
+		(property "LCSC" "C17337"
+			(at 151.13 93.98 0)
+			(hide yes)
+			(show_name no)
+			(do_not_autoplace no)
+			(effects
+				(font
+					(size 1.27 1.27)
+				)
+			)
+		)
 		(pin "1"
 		)
@@
 			)
 		)
+		(property "LCSC" "C19702"
+			(at 165.1 72.39 0)
+			(hide yes)
+			(show_name no)
+			(do_not_autoplace no)
+			(effects
+				(font
+					(size 1.27 1.27)
+				)
+			)
+		)
 		(pin "1"
 		)
@@
 			)
 		)
+		(property "LCSC" "C25804"
+			(at 184.15 116.84 0)
+			(hide yes)
+			(show_name no)
+			(do_not_autoplace no)
+			(effects
+				(font
+					(size 1.27 1.27)
+				)
+			)
+		)
 		(pin "1"
 		)
@@
 		(in_pos_files yes)
 		(dnp no)
-		(property "Reference" "#PWR065"
+		(property "Reference" "#PWR068"
 			(at 186.69 101.6 0)
 			(hide yes)
@@
 			(project "dino_z80"
 				(path "/8c0b3d8b-46d3-4173-ab1e-a61765f77d61/3603a3f9-aa53-493b-ae79-e24b3c1f7362/128bfa67-3568-45ab-9ac5-06e6eea36fac"
-					(reference "#PWR065")
+					(reference "#PWR068")
 					(unit 1)
 				)
@@
 		(in_pos_files yes)
 		(dnp no)
-		(property "Reference" "#PWR057"
+		(property "Reference" "#PWR060"
 			(at 156.21 81.28 0)
 			(hide yes)
@@
 			(project "dino_z80"
 				(path "/8c0b3d8b-46d3-4173-ab1e-a61765f77d61/3603a3f9-aa53-493b-ae79-e24b3c1f7362/128bfa67-3568-45ab-9ac5-06e6eea36fac"
-					(reference "#PWR057")
+					(reference "#PWR060")
 					(unit 1)
 				)
@@
 		(in_pos_files yes)
 		(dnp no)
-		(property "Reference" "#PWR056"
+		(property "Reference" "#PWR059"
 			(at 156.21 63.5 0)
 			(hide yes)
@@
 			(project "dino_z80"
 				(path "/8c0b3d8b-46d3-4173-ab1e-a61765f77d61/3603a3f9-aa53-493b-ae79-e24b3c1f7362/128bfa67-3568-45ab-9ac5-06e6eea36fac"
-					(reference "#PWR056")
+					(reference "#PWR059")
 					(unit 1)
 				)
@@
 			)
 		)
+		(property "LCSC" "C1631"
+			(at 120.65 118.11 0)
+			(hide yes)
+			(show_name no)
+			(do_not_autoplace no)
+			(effects
+				(font
+					(size 1.27 1.27)
+				)
+			)
+		)
 		(pin "1"
 		)
@@
 		(in_pos_files yes)
 		(dnp no)
-		(property "Reference" "#PWR066"
+		(property "Reference" "#PWR069"
 			(at 186.69 106.68 0)
 			(hide yes)
@@
 			(project "dino_z80"
 				(path "/8c0b3d8b-46d3-4173-ab1e-a61765f77d61/3603a3f9-aa53-493b-ae79-e24b3c1f7362/128bfa67-3568-45ab-9ac5-06e6eea36fac"
-					(reference "#PWR066")
+					(reference "#PWR069")
 					(unit 1)
 				)
@@
 			)
 		)
+		(property "LCSC" "C14663"
+			(at 156.21 72.39 0)
+			(hide yes)
+			(show_name no)
+			(do_not_autoplace no)
+			(effects
+				(font
+					(size 1.27 1.27)
+				)
+			)
+		)
 		(pin "1"
 		)
@@
 			)
 		)
+		(property "LCSC" "C15849"
+			(at 127 109.22 0)
+			(hide yes)
+			(show_name no)
+			(do_not_autoplace no)
+			(effects
+				(font
+					(size 1.27 1.27)
+				)
+			)
+		)
 		(pin "1"
 		)
@@
 		(in_pos_files yes)
 		(dnp no)
-		(property "Reference" "#PWR055"
+		(property "Reference" "#PWR058"
 			(at 151.13 125.73 0)
 			(hide yes)
@@
 			(project "dino_z80"
 				(path "/8c0b3d8b-46d3-4173-ab1e-a61765f77d61/3603a3f9-aa53-493b-ae79-e24b3c1f7362/128bfa67-3568-45ab-9ac5-06e6eea36fac"
-					(reference "#PWR055")
+					(reference "#PWR058")
 					(unit 1)
 				)
@@
 		(in_pos_files yes)
 		(dnp no)
-		(property "Reference" "#PWR053"
+		(property "Reference" "#PWR055"
 			(at 139.7 104.14 0)
 			(hide yes)
@@
 			(project "dino_z80"
 				(path "/8c0b3d8b-46d3-4173-ab1e-a61765f77d61/3603a3f9-aa53-493b-ae79-e24b3c1f7362/128bfa67-3568-45ab-9ac5-06e6eea36fac"
-					(reference "#PWR053")
+					(reference "#PWR055")
 					(unit 1)
 				)
@@
 			)
 		)
+		(property "LCSC" "C31850"
+			(at 102.87 109.22 0)
+			(hide yes)
+			(show_name no)
+			(do_not_autoplace no)
+			(effects
+				(font
+					(size 1.27 1.27)
+				)
+			)
+		)
 		(pin "1"
 		)
@@
 			)
 		)
+		(property "LCSC" "C31850"
+			(at 105.41 133.35 0)
+			(hide yes)
+			(show_name no)
+			(do_not_autoplace no)
+			(effects
+				(font
+					(size 1.27 1.27)
+				)
+			)
+		)
 		(pin "1"
 		)
@@
 		(in_pos_files yes)
 		(dnp no)
-		(property "Reference" "#PWR064"
+		(property "Reference" "#PWR067"
 			(at 184.15 120.65 0)
 			(hide yes)
@@
 			(project "dino_z80"
 				(path "/8c0b3d8b-46d3-4173-ab1e-a61765f77d61/3603a3f9-aa53-493b-ae79-e24b3c1f7362/128bfa67-3568-45ab-9ac5-06e6eea36fac"
-					(reference "#PWR064")
+					(reference "#PWR067")
 					(unit 1)
 				)
@@
 			)
 		)
+		(property "LCSC" "C15849"
+			(at 151.13 116.84 0)
+			(hide yes)
+			(show_name no)
+			(do_not_autoplace no)
+			(effects
+				(font
+					(size 1.27 1.27)
+				)
+			)
+		)
 		(pin "1"
 		)
@@
 		(in_pos_files yes)
 		(dnp no)
-		(property "Reference" "#PWR054"
+		(property "Reference" "#PWR056"
 			(at 151.13 100.33 0)
 			(hide yes)
@@
 			(project "dino_z80"
 				(path "/8c0b3d8b-46d3-4173-ab1e-a61765f77d61/3603a3f9-aa53-493b-ae79-e24b3c1f7362/128bfa67-3568-45ab-9ac5-06e6eea36fac"
-					(reference "#PWR054")
+					(reference "#PWR056")
 					(unit 1)
 				)
@@
 		(in_pos_files yes)
 		(dnp no)
-		(property "Reference" "#PWR059"
+		(property "Reference" "#PWR062"
 			(at 165.1 81.28 0)
 			(hide yes)
@@
 			(project "dino_z80"
 				(path "/8c0b3d8b-46d3-4173-ab1e-a61765f77d61/3603a3f9-aa53-493b-ae79-e24b3c1f7362/128bfa67-3568-45ab-9ac5-06e6eea36fac"
-					(reference "#PWR059")
+					(reference "#PWR062")
 					(unit 1)
 				)
@@
 		(in_pos_files yes)
 		(dnp no)
-		(property "Reference" "#PWR051"
+		(property "Reference" "#PWR053"
 			(at 110.49 127 0)
 			(hide yes)
@@
 			(project "dino_z80"
 				(path "/8c0b3d8b-46d3-4173-ab1e-a61765f77d61/3603a3f9-aa53-493b-ae79-e24b3c1f7362/128bfa67-3568-45ab-9ac5-06e6eea36fac"
-					(reference "#PWR051")
+					(reference "#PWR053")
 					(unit 1)
 				)
@@
 		(in_pos_files yes)
 		(dnp no)
-		(property "Reference" "#PWR052"
+		(property "Reference" "#PWR054"
 			(at 120.65 127 0)
 			(hide yes)
@@
 			(project "dino_z80"
 				(path "/8c0b3d8b-46d3-4173-ab1e-a61765f77d61/3603a3f9-aa53-493b-ae79-e24b3c1f7362/128bfa67-3568-45ab-9ac5-06e6eea36fac"
-					(reference "#PWR052")
+					(reference "#PWR054")
 					(unit 1)
 				)
@@
 			)
 		)
+		(property "LCSC" "C25804"
+			(at 144.78 109.22 0)
+			(hide yes)
+			(show_name no)
+			(do_not_autoplace no)
+			(effects
+				(font
+					(size 1.27 1.27)
+				)
+			)
+		)
 		(pin "1"
 		)
@@
 		(in_pos_files yes)
 		(dnp no)
-		(property "Reference" "#PWR058"
+		(property "Reference" "#PWR061"
 			(at 165.1 63.5 0)
 			(hide yes)
@@
 			(project "dino_z80"
 				(path "/8c0b3d8b-46d3-4173-ab1e-a61765f77d61/3603a3f9-aa53-493b-ae79-e24b3c1f7362/128bfa67-3568-45ab-9ac5-06e6eea36fac"
-					(reference "#PWR058")
+					(reference "#PWR061")
 					(unit 1)
 				)
@@
 		(in_pos_files yes)
 		(dnp no)
-		(property "Reference" "#PWR060"
+		(property "Reference" "#PWR064"
 			(at 173.99 63.5 0)
 			(hide yes)
@@
 			(project "dino_z80"
 				(path "/8c0b3d8b-46d3-4173-ab1e-a61765f77d61/3603a3f9-aa53-493b-ae79-e24b3c1f7362/128bfa67-3568-45ab-9ac5-06e6eea36fac"
-					(reference "#PWR060")
-					(unit 1)
-				)
+					(reference "#PWR064")
+					(unit 1)
+				)

Commit message: fix: dino_z80 1.02 - pre-production review, TVS input, labels, release
- Power: SMAJ15A TVS D7 after the fuse (C908769, optional fit); Q1 gate
  divider R47/R48 100K/43K (Vgs within +-12 V at the TVS clamp); MP1584 UVLO
  R50/R51 300K/100K (start ~6.0 V); C54 680u 25V (C46550437); notes fixed
- Every capacitor value carries its voltage (from the LCSC part)
- Test points on all rails, on the back
- ERC: connector/hub pin types, PWR_FLAGs; 49 stale exclusions removed.
  ERC 0 errors, 0 warnings
- RP2350 exposed-pad vias tagged heatsink (no type mismatch)
- Fields: LCSC numbers removed from solder jumpers, S1/U1/U2/Y2/L1 part
  data and datasheet links corrected
- Layout: vias moved out of signal/power pads where a 45-degree escape
  exists, corners fixed, reference labels 0.7 mm bold re-placed
- Release 1.02: gerbers, schematics, assembly PDF, iBOM
  (DRC 0 violations, 0 unconnected, 0 parity)
Parts:
- C15: value 6.8nF -> 6.8n 50V
- C16, C17: value 1µF -> 1u 50V
- C18: value 100nF -> 100n 50V
- C19: value 10µF -> 10u 10V
- C20: value 100µF -> 100u 25V
Changed lines of the file:
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@@
 			)
 		)
-		(property "Value" "100µF"
+		(property "Value" "100u 25V"
 			(at 176.53 72.39 90)
 			(show_name no)
@@
 			)
 		)
-		(property "Value" "10µF"
+		(property "Value" "10u 10V"
 			(at 167.64 72.39 90)
 			(show_name no)
@@
 			)
 		)
-		(property "Value" "6.8nF"
+		(property "Value" "6.8n 50V"
 			(at 123.19 118.11 90)
 			(show_name no)
@@
 			)
 		)
-		(property "Value" "100nF"
+		(property "Value" "100n 50V"
 			(at 158.75 72.39 90)
 			(show_name no)
@@
 			)
 		)
-		(property "Value" "1µF"
+		(property "Value" "1u 50V"
 			(at 127 111.76 270)
 			(show_name no)
@@
 			)
 		)
-		(property "Value" "1µF"
+		(property "Value" "1u 50V"
 			(at 153.67 116.84 90)
 			(show_name no)
